File: boards/pq-register/P1.kicad_sch (KiCad schematic)
At the start: 84 parts, among them Q1 MMBT5401, Q10 MMBT5401, Q102 MMBT5401, Q103 MMBT5401, Q11 MMBT5401, Q2 MMBT5401, Q3 MMBT5401, Q4 MMBT5401, Q5 MMBT5401, Q6 MMBT5401, Q7 MMBT5401, Q8 MMBT5401, Q9 MMBT5401

Commit message: Better PCI footprint, more layout.
Connections:
- net CP renamed CP_{1}
Changed lines of the file:
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@@
 		(property "Intersheetrefs" "${INTERSHEET_REFS}"
 			(at 29.1277 105.41 0)
-			(hide yes)
 			(show_name no)
 			(do_not_autoplace no)
@@
 		(property "Intersheetrefs" "${INTERSHEET_REFS}"
 			(at 132.9048 130.81 0)
-			(hide yes)
 			(show_name no)
 			(do_not_autoplace no)
@@
 		(property "Intersheetrefs" "${INTERSHEET_REFS}"
 			(at 133.57 99.06 0)
-			(hide yes)
 			(show_name no)
 			(do_not_autoplace no)
@@
 		(property "Intersheetrefs" "${INTERSHEET_REFS}"
 			(at 30.0348 41.91 0)
-			(hide yes)
 			(show_name no)
 			(do_not_autoplace no)
@@
 		(property "Intersheetrefs" "${INTERSHEET_REFS}"
 			(at 258.1947 43.18 0)
-			(hide yes)
 			(show_name no)
 			(do_not_autoplace no)
@@
 		(property "Intersheetrefs" "${INTERSHEET_REFS}"
 			(at 80.8348 172.72 0)
-			(hide yes)
 			(show_name no)
 			(do_not_autoplace no)
@@
 		(property "Intersheetrefs" "${INTERSHEET_REFS}"
 			(at 133.57 135.89 0)
-			(hide yes)
 			(show_name no)
 			(do_not_autoplace no)
@@
 		(property "Intersheetrefs" "${INTERSHEET_REFS}"
 			(at 28.8253 115.57 0)
-			(hide yes)
 			(show_name no)
 			(do_not_autoplace no)
@@
 		(property "Intersheetrefs" "${INTERSHEET_REFS}"
 			(at 29.9743 110.49 0)
-			(hide yes)
 			(show_name no)
 			(do_not_autoplace no)
@@
 		(property "Intersheetrefs" "${INTERSHEET_REFS}"
 			(at 29.8534 31.75 0)
-			(hide yes)
 			(show_name no)
 			(do_not_autoplace no)
@@
 		(property "Intersheetrefs" "${INTERSHEET_REFS}"
 			(at 78.4763 167.64 0)
-			(hide yes)
 			(show_name no)
 			(do_not_autoplace no)
@@
 		(property "Intersheetrefs" "${INTERSHEET_REFS}"
 			(at 79.9277 130.81 0)
-			(hide yes)
 			(show_name no)
 			(do_not_autoplace no)
@@
 		(property "Intersheetrefs" "${INTERSHEET_REFS}"
 			(at 80.7743 135.89 0)
-			(hide yes)
 			(show_name no)
 			(do_not_autoplace no)
@@
 		(property "Intersheetrefs" "${INTERSHEET_REFS}"
 			(at 78.5367 66.04 0)
-			(hide yes)
 			(show_name no)
 			(do_not_autoplace no)
@@
 		(property "Intersheetrefs" "${INTERSHEET_REFS}"
 			(at 79.6253 177.8 0)
-			(hide yes)
 			(show_name no)
 			(do_not_autoplace no)
@@
 		(property "Intersheetrefs" "${INTERSHEET_REFS}"
 			(at 30.7 36.83 0)
-			(hide yes)
 			(show_name no)
 			(do_not_autoplace no)
@@
 		(property "Intersheetrefs" "${INTERSHEET_REFS}"
 			(at 30.7 73.66 0)
-			(hide yes)
 			(show_name no)
 			(do_not_autoplace no)
@@
 		(property "Intersheetrefs" "${INTERSHEET_REFS}"
 			(at 182.6163 167.64 0)
-			(hide yes)
 			(show_name no)
 			(do_not_autoplace no)
@@
 		(property "Intersheetrefs" "${INTERSHEET_REFS}"
 			(at 30.0348 68.58 0)
-			(hide yes)
 			(show_name no)
 			(do_not_autoplace no)
@@
 		(property "Intersheetrefs" "${INTERSHEET_REFS}"
 			(at 30.2162 78.74 0)
-			(hide yes)
 			(show_name no)
 			(do_not_autoplace no)
@@
 		(property "Intersheetrefs" "${INTERSHEET_REFS}"
 			(at 132.7234 104.14 0)
-			(hide yes)
-			(show_name no)
-			(do_not_autoplace no)
-			(effects
-				(font
-					(size 1.27 1.27)
-				)
-				(justify right)
-			)
-		)
-	)
-	(global_label "CP"
+			(show_name no)
+			(do_not_autoplace no)
+			(effects
+				(font
+					(size 1.27 1.27)
+				)
+				(justify right)
+			)
+		)
+	)
+	(global_label "CP_{1}"
 		(shape input)
 		(at 166.37 69.85 270)
@@
 		)
 		(property "Intersheetrefs" "${INTERSHEET_REFS}"
-			(at 166.37 75.3752 90)
-			(hide yes)
+			(at 166.37 76.3936 90)
 			(show_name no)
 			(do_not_autoplace no)
@@
 		(property "Intersheetrefs" "${INTERSHEET_REFS}"
 			(at 79.6253 140.97 0)
-			(hide yes)
 			(show_name no)
 			(do_not_autoplace no)
@@
 		(property "Intersheetrefs" "${INTERSHEET_REFS}"
 			(at 258.1947 88.9 0)
-			(hide yes)
 			(show_name no)
 			(do_not_autoplace no)
@@
 		(property "Intersheetrefs" "${INTERSHEET_REFS}"
 			(at 133.0862 140.97 0)
-			(hide yes)
 			(show_name no)
 			(do_not_autoplace no)
@@
 		(property "Intersheetrefs" "${INTERSHEET_REFS}"
 			(at 132.9048 93.98 0)
-			(hide yes)
 			(show_name no)
 			(do_not_autoplace no)
@@
 		(property "Intersheetrefs" "${INTERSHEET_REFS}"
 			(at 79.9277 182.88 0)
-			(hide yes)
-			(show_name no)
-			(do_not_autoplace no)
+			(show_name no)
+			(do_not_autoplace no)

Commit message: Start updating 2k4 resistors to 0603, melt some traces.
Parts:
- R10, R12, R14, R16, R18, R2, R4, R6, R8: value 2k 500mW -> 2k ½W
- R65, R84, R85, R86: value 2k4 -> 2k4 ¼W; footprint Resistor_SMD:R_0402_1005Metric -> Resistor_SMD:R_0603_1608Metric
Changed lines of the file:
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@@
 			)
 		)
-		(property "Value" "2k 500mW"
+		(property "Value" "2k ½W"
 			(at 161.544 128.27 0)
 			(show_name no)
@@
 			)
 		)
-		(property "Value" "2k4"
+		(property "Value" "2k4 ¼W"
 			(at 151.13 43.688 90)
 			(show_name no)
@@
 			)
 		)
-		(property "Footprint" "Resistor_SMD:R_0402_1005Metric"
+		(property "Footprint" "Resistor_SMD:R_0603_1608Metric"
 			(at 151.384 46.736 90)
 			(hide yes)
@@
 			)
 		)
-		(property "Value" "2k 500mW"
+		(property "Value" "2k ½W"
 			(at 109.474 128.27 0)
 			(show_name no)
@@
 			)
 		)
-		(property "Value" "2k 500mW"
+		(property "Value" "2k ½W"
 			(at 109.474 63.5 0)
 			(show_name no)
@@
 			)
 		)
-		(property "Value" "2k4"
+		(property "Value" "2k4 ¼W"
 			(at 181.61 43.688 90)
 			(show_name no)
@@
 			)
 		)
-		(property "Footprint" "Resistor_SMD:R_0402_1005Metric"
+		(property "Footprint" "Resistor_SMD:R_0603_1608Metric"
 			(at 181.864 46.736 90)
 			(hide yes)
@@
 			)
 		)
-		(property "Value" "2k4"
+		(property "Value" "2k4 ¼W"
 			(at 142.24 65.278 90)
 			(show_name no)
@@
 			)
 		)
-		(property "Footprint" "Resistor_SMD:R_0402_1005Metric"
+		(property "Footprint" "Resistor_SMD:R_0603_1608Metric"
 			(at 142.494 68.326 90)
 			(hide yes)
@@
 			)
 		)
-		(property "Value" "2k 500mW"
+		(property "Value" "2k ½W"
 			(at 58.674 66.04 0)
 			(show_name no)
@@
 			)
 		)
-		(property "Value" "2k 500mW"
+		(property "Value" "2k ½W"
 			(at 161.544 91.44 0)
 			(show_name no)
@@
 			)
 		)
-		(property "Value" "2k 500mW"
+		(property "Value" "2k ½W"
 			(at 58.674 102.87 0)
 			(show_name no)
@@
 			)
 		)
-		(property "Value" "2k4"
+		(property "Value" "2k4 ¼W"
 			(at 190.5 65.278 90)
 			(show_name no)
@@
 			)
 		)
-		(property "Footprint" "Resistor_SMD:R_0402_1005Metric"
+		(property "Footprint" "Resistor_SMD:R_0603_1608Metric"
 			(at 190.754 68.326 90)
 			(hide yes)
@@
 			)
 		)
-		(property "Value" "2k 500mW"
+		(property "Value" "2k ½W"
 			(at 213.614 144.78 0)
 			(show_name no)
@@
 			)
 		)
-		(property "Value" "2k 500mW"
+		(property "Value" "2k ½W"
 			(at 109.474 165.1 0)
 			(show_name no)
@@
 			)
 		)
-		(property "Value" "2k 500mW"
+		(property "Value" "2k ½W"
 			(at 58.674 29.21 0)
 			(show_name no)

Commit message: Clean up sheet frames.
Other:
- company: © 1962 General Precision; redrawn by Sam Hanes -> © 2026 Sam Hanes, licensed CERN-OHL-W v2
- title: LGP-21 P & Q Register Board -> LGP-21 Mini - P&Q Register
Changed lines of the file:
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@@
 	(generator "eeschema")
 	(generator_version "10.0")
-	(paper "A")
+	(paper "USLetter")
 	(title_block
-		(title "LGP-21 P & Q Register Board")
-		(date "2026-06-15")
-		(rev "ESD 1060")
-		(company "© 1962 General Precision; redrawn by Sam Hanes")
-		(comment 1 "https://github.com/Elemecca/lgp21-docs")
+		(title "LGP-21 Mini - P&Q Register")
+		(date "2026-06-28")
+		(rev "A")
+		(company "© 2026 Sam Hanes, licensed CERN-OHL-W v2")
+		(comment 1 "https://github.com/Elemecca/lgp21-mini")
 	)
 	(text "P1"
