File: boards/pq-register/P1.kicad_sch (KiCad schematic)
At the start: 84 parts, among them Q1 MMBT5401, Q10 MMBT5401, Q102 MMBT5401, Q103 MMBT5401, Q11 MMBT5401, Q2 MMBT5401, Q3 MMBT5401, Q4 MMBT5401, Q5 MMBT5401, Q6 MMBT5401, Q7 MMBT5401, Q8 MMBT5401, Q9 MMBT5401

Commit message: Route resistors in the second column.
Parts:
- R65, R84: value 2k4 ¼W -> 2k4; footprint Resistor_SMD:R_0603_1608Metric -> Resistor_SMD:R_0402_1005Metric
Changed lines of the file:
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@@
 			)
 		)
-		(property "Value" "2k4 ¼W"
+		(property "Value" "2k4"
 			(at 142.24 65.278 90)
 			(show_name no)
@@
 			)
 		)
-		(property "Footprint" "Resistor_SMD:R_0603_1608Metric"
+		(property "Footprint" "Resistor_SMD:R_0402_1005Metric"
 			(at 142.494 68.326 90)
 			(hide yes)
@@
 			)
 		)
-		(property "Value" "2k4 ¼W"
+		(property "Value" "2k4"
 			(at 190.5 65.278 90)
 			(show_name no)
@@
 			)
 		)
-		(property "Footprint" "Resistor_SMD:R_0603_1608Metric"
+		(property "Footprint" "Resistor_SMD:R_0402_1005Metric"
 			(at 190.754 68.326 90)
 			(hide yes)

Commit message: Add script to export production files.
Parts:
- C1, C4: BOM Value (none) -> 120pF
- C2, C3: BOM Value (none) -> 680pF
- CR1, CR2, CR24, CR25, CR26, CR27, CR28, CR29: value 1N5819WS -> 1N4148WS; BOM Value (none) -> 1N4148WS; LCSC (none) -> C2128
- Q1, Q10, Q102, Q103, Q11, Q2, Q3, Q4, Q5, Q6, Q7, Q8, Q9: BOM Value (none) -> MMBT5401; LCSC (none) -> C8326
- R1, R11, R13, R15, R17, R3, R5, R504, R505, R7, R9: BOM Value (none) -> 56kΩ
- R10, R12, R14, R16, R18, R2, R4, R6, R8: BOM Value (none) -> 2kΩ 500mW
- R131, R132: BOM Value (none) -> 300Ω 3W
- R19, R20: BOM Value (none) -> 33kΩ
- R51, R52, R53, R54, R55, R56, R57, R58, R59, R60, R61, R62, R63, R66, R67, R68, R69, R70, R71, R72, R73, R74, R75, R76, R77, R78, R79, R80, R81, R82, R83: BOM Value (none) -> 15kΩ
- R65, R84: BOM Value (none) -> 2.4kΩ
- R85, R86: BOM Value (none) -> 2.4kΩ 250mW
