File: boards/pq-register/P2.kicad_sch (KiCad schematic)
At the start: 36 parts, among them Q12 MMBT5401, Q13 MMBT5401, Q14 MMBT5401, Q15 MMBT5401, Q16 MMBT5401, Q17 MMBT5401

Commit message: Route resistors in the second column.
Parts:
- R91, R96: value 2k4 ¼W -> 2k4; footprint Resistor_SMD:R_0603_1608Metric -> Resistor_SMD:R_0402_1005Metric
Changed lines of the file:
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@@
 			)
 		)
-		(property "Value" "2k4 ¼W"
+		(property "Value" "2k4"
 			(at 153.67 107.188 90)
 			(show_name no)
@@
 			)
 		)
-		(property "Footprint" "Resistor_SMD:R_0603_1608Metric"
+		(property "Footprint" "Resistor_SMD:R_0402_1005Metric"
 			(at 153.924 110.236 90)
 			(hide yes)
@@
 			)
 		)
-		(property "Value" "2k4 ¼W"
+		(property "Value" "2k4"
 			(at 201.93 107.188 90)
 			(show_name no)
@@
 			)
 		)
-		(property "Footprint" "Resistor_SMD:R_0603_1608Metric"
+		(property "Footprint" "Resistor_SMD:R_0402_1005Metric"
 			(at 202.184 110.236 90)
 			(hide yes)

Commit message: Add script to export production files.
Parts:
- C5, C8: BOM Value (none) -> 120pF
- C6, C7: BOM Value (none) -> 680pF
- CR3, CR4: value 1N5819WS -> 1N4148WS; BOM Value (none) -> 1N4148WS; LCSC (none) -> C2128
- Q12, Q13, Q14, Q15, Q16, Q17: BOM Value (none) -> MMBT5401; LCSC (none) -> C8326
- R127, R129: BOM Value (none) -> 300Ω 3W
- R21, R23, R25, R27: BOM Value (none) -> 56kΩ
- R22, R24, R26, R28: BOM Value (none) -> 2kΩ 500mW
- R29, R30: BOM Value (none) -> 33kΩ
- R87, R88, R89, R90, R92, R93, R94, R95: BOM Value (none) -> 15kΩ
- R91, R96: BOM Value (none) -> 2.4kΩ
- R97, R98: BOM Value (none) -> 2.4kΩ 250mW
