File: boards/pq-register/P3.kicad_sch (KiCad schematic)
At the start: 36 parts, among them Q18 MMBT5401, Q19 MMBT5401, Q20 MMBT5401, Q21 MMBT5401, Q22 MMBT5401, Q23 MMBT5401

Commit message: Route resistors in the second column.
Parts:
- R103, R108: value 2k4 ¼W -> 2k4; footprint Resistor_SMD:R_0603_1608Metric -> Resistor_SMD:R_0402_1005Metric
Changed lines of the file:
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@@
 			)
 		)
-		(property "Value" "2k4 ¼W"
+		(property "Value" "2k4"
 			(at 201.93 107.188 90)
 			(show_name no)
@@
 			)
 		)
-		(property "Footprint" "Resistor_SMD:R_0603_1608Metric"
+		(property "Footprint" "Resistor_SMD:R_0402_1005Metric"
 			(at 202.184 110.236 90)
 			(hide yes)
@@
 			)
 		)
-		(property "Value" "2k4 ¼W"
+		(property "Value" "2k4"
 			(at 153.67 107.188 90)
 			(show_name no)
@@
 			)
 		)
-		(property "Footprint" "Resistor_SMD:R_0603_1608Metric"
+		(property "Footprint" "Resistor_SMD:R_0402_1005Metric"
 			(at 153.924 110.236 90)
 			(hide yes)

Commit message: Add script to export production files.
Parts:
- C10, C11: BOM Value (none) -> 680pF
- C12, C9: BOM Value (none) -> 120pF
- CR5, CR6: value 1N5819WS -> 1N4148WS; BOM Value (none) -> 1N4148WS; LCSC (none) -> C2128
- Q18, Q19, Q20, Q21, Q22, Q23: BOM Value (none) -> MMBT5401; LCSC (none) -> C8326
- R100, R101, R102, R104, R105, R106, R107, R99: BOM Value (none) -> 15kΩ
- R103, R108: BOM Value (none) -> 2.4kΩ
- R109, R110: BOM Value (none) -> 2.4kΩ 250mW
- R125, R126: BOM Value (none) -> 300Ω 3W
- R31, R33, R35, R37: BOM Value (none) -> 56kΩ
- R32, R34, R36, R38: BOM Value (none) -> 2kΩ 500mW
- R39, R40: BOM Value (none) -> 33kΩ
