File: boards/pq-register/P4.kicad_sch (KiCad schematic)
At the start: 36 parts, among them Q24 MMBT5401, Q25 MMBT5401, Q26 MMBT5401, Q27 MMBT5401, Q28 MMBT5401, Q29 MMBT5401

Commit message: Route resistors in the second column.
Parts:
- R115, R120: value 2k4 ¼W -> 2k4; footprint Resistor_SMD:R_0603_1608Metric -> Resistor_SMD:R_0402_1005Metric
Changed lines of the file:
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@@
 			)
 		)
-		(property "Value" "2k4 ¼W"
+		(property "Value" "2k4"
 			(at 153.67 107.188 90)
 			(show_name no)
@@
 			)
 		)
-		(property "Footprint" "Resistor_SMD:R_0603_1608Metric"
+		(property "Footprint" "Resistor_SMD:R_0402_1005Metric"
 			(at 153.924 110.236 90)
 			(hide yes)
@@
 			)
 		)
-		(property "Value" "2k4 ¼W"
+		(property "Value" "2k4"
 			(at 201.93 107.188 90)
 			(show_name no)
@@
 			)
 		)
-		(property "Footprint" "Resistor_SMD:R_0603_1608Metric"
+		(property "Footprint" "Resistor_SMD:R_0402_1005Metric"
 			(at 202.184 110.236 90)
 			(hide yes)

Commit message: Add script to export production files.
Parts:
- C13, C16: BOM Value (none) -> 120pF
- C14, C15: BOM Value (none) -> 680pF
- CR7, CR8: value 1N5819WS -> 1N4148WS; BOM Value (none) -> 1N4148WS; LCSC (none) -> C2128
- Q24, Q25, Q26, Q27, Q28, Q29: BOM Value (none) -> MMBT5401; LCSC (none) -> C8326
- R111, R112, R113, R114, R116, R117, R118, R119: BOM Value (none) -> 15kΩ
- R115, R120: BOM Value (none) -> 2.4kΩ
- R121, R122: BOM Value (none) -> 2.4kΩ 250mW
- R123, R124: BOM Value (none) -> 300Ω 3W
- R41, R43, R45, R47: BOM Value (none) -> 56kΩ
- R42, R44, R46, R48: BOM Value (none) -> 2kΩ 500mW
- R49, R50: BOM Value (none) -> 33kΩ
