File: boards/pq-register/P5.kicad_sch (KiCad schematic)
At the start: 64 parts, among them Q30 MMBT5401, Q31 MMBT5401, Q32 MMBT5401, Q33 MMBT5401, Q34 MMBT5401, Q35 MMBT5401, Q36 MMBT5401, Q37 MMBT5401, Q50 MMBT5401

Commit message: Better PCI footprint, more layout.
Connections:
- net CP renamed CP_{1}
Changed lines of the file:
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@@
 		(property "Intersheetrefs" "${INTERSHEET_REFS}"
 			(at 124.3777 132.08 0)
-			(hide yes)
 			(show_name no)
 			(do_not_autoplace no)
@@
 		(property "Intersheetrefs" "${INTERSHEET_REFS}"
 			(at 36.3848 41.91 0)
-			(hide yes)
 			(show_name no)
 			(do_not_autoplace no)
@@
 		(property "Intersheetrefs" "${INTERSHEET_REFS}"
 			(at 35.1753 125.73 0)
-			(hide yes)
 			(show_name no)
 			(do_not_autoplace no)
@@
 		(property "Intersheetrefs" "${INTERSHEET_REFS}"
 			(at 35.1753 52.07 0)
-			(hide yes)
 			(show_name no)
 			(do_not_autoplace no)
@@
 		(property "Intersheetrefs" "${INTERSHEET_REFS}"
 			(at 36.3848 57.15 0)
-			(hide yes)
 			(show_name no)
 			(do_not_autoplace no)
@@
 		(property "Intersheetrefs" "${INTERSHEET_REFS}"
 			(at 34.0263 93.98 0)
-			(hide yes)
 			(show_name no)
 			(do_not_autoplace no)
@@
 		(property "Intersheetrefs" "${INTERSHEET_REFS}"
 			(at 35.1148 36.83 0)
-			(hide yes)
 			(show_name no)
 			(do_not_autoplace no)
@@
 		(property "Intersheetrefs" "${INTERSHEET_REFS}"
 			(at 89.9667 69.85 0)
-			(hide yes)
 			(show_name no)
 			(do_not_autoplace no)
@@
 		(property "Intersheetrefs" "${INTERSHEET_REFS}"
 			(at 36.5662 73.66 0)
-			(hide yes)
 			(show_name no)
 			(do_not_autoplace no)
@@
 		(property "Intersheetrefs" "${INTERSHEET_REFS}"
 			(at 124.0753 110.49 0)
-			(hide yes)
 			(show_name no)
 			(do_not_autoplace no)
@@
 		(property "Intersheetrefs" "${INTERSHEET_REFS}"
 			(at 36.3848 78.74 0)
-			(hide yes)
 			(show_name no)
 			(do_not_autoplace no)
@@
 		(property "Intersheetrefs" "${INTERSHEET_REFS}"
 			(at 94.2437 43.18 0)
-			(hide yes)
 			(show_name no)
 			(do_not_autoplace no)
@@
 		(property "Intersheetrefs" "${INTERSHEET_REFS}"
 			(at 178.8063 111.76 0)
-			(hide yes)
-			(show_name no)
-			(do_not_autoplace no)
-			(effects
-				(font
-					(size 1.27 1.27)
-				)
-				(justify right)
-			)
-		)
-	)
-	(global_label "CP"
+			(show_name no)
+			(do_not_autoplace no)
+			(effects
+				(font
+					(size 1.27 1.27)
+				)
+				(justify right)
+			)
+		)
+	)
+	(global_label "CP_{1}"
 		(shape input)
 		(at 177.8 73.66 270)
@@
 		)
 		(property "Intersheetrefs" "${INTERSHEET_REFS}"
-			(at 177.8 79.1852 90)
-			(hide yes)
+			(at 177.8 80.2036 90)
 			(show_name no)
 			(do_not_autoplace no)
@@
 		(property "Intersheetrefs" "${INTERSHEET_REFS}"
 			(at 223.9047 25.4 0)
-			(hide yes)
 			(show_name no)
 			(do_not_autoplace no)
@@
 		(property "Intersheetrefs" "${INTERSHEET_REFS}"
 			(at 36.5662 46.99 0)
-			(hide yes)
 			(show_name no)
 			(do_not_autoplace no)
@@
 		(property "Intersheetrefs" "${INTERSHEET_REFS}"
 			(at 125.95 105.41 0)
-			(hide yes)
 			(show_name no)
 			(do_not_autoplace no)
@@
 		(property "Intersheetrefs" "${INTERSHEET_REFS}"
 			(at 223.9047 46.99 0)
-			(hide yes)
 			(show_name no)
 			(do_not_autoplace no)
@@
 		(property "Intersheetrefs" "${INTERSHEET_REFS}"
 			(at 122.9263 142.24 0)
-			(hide yes)
 			(show_name no)
 			(do_not_autoplace no)
@@
 		(property "Intersheetrefs" "${INTERSHEET_REFS}"
 			(at 35.4777 83.82 0)
-			(hide yes)
 			(show_name no)
 			(do_not_autoplace no)
@@
 		(property "Intersheetrefs" "${INTERSHEET_REFS}"
 			(at 34.6915 62.23 0)
-			(hide yes)
 			(show_name no)
 			(do_not_autoplace no)
@@
 		(property "Intersheetrefs" "${INTERSHEET_REFS}"
 			(at 125.2243 137.16 0)
-			(hide yes)
 			(show_name no)
 			(do_not_autoplace no)
@@
 		(property "Intersheetrefs" "${INTERSHEET_REFS}"
 			(at 125.4662 152.4 0)
-			(hide yes)
 			(show_name no)
 			(do_not_autoplace no)
@@
 		(property "Intersheetrefs" "${INTERSHEET_REFS}"
 			(at 125.2848 147.32 0)
-			(hide yes)
 			(show_name no)
 			(do_not_autoplace no)
@@
 		(property "Intersheetrefs" "${INTERSHEET_REFS}"
 			(at 36.3243 88.9 0)
-			(hide yes)
 			(show_name no)
 			(do_not_autoplace no)
@@
 		(property "Intersheetrefs" "${INTERSHEET_REFS}"
 			(at 37.05 120.65 0)
-			(hide yes)
-			(show_name no)
-			(do_not_autoplace no)
+			(show_name no)
+			(do_not_autoplace no)

Commit message: Start updating 2k4 resistors to 0603, melt some traces.
Parts:
- R144, R155, R156, R157: value 2k4 -> 2k4 ¼W; footprint Resistor_SMD:R_0402_1005Metric -> Resistor_SMD:R_0603_1608Metric
- R222, R224, R226, R228, R230, R232, R258: value 2k 500mW -> 2k ½W
Changed lines of the file:
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@@
 			)
 		)
-		(property "Value" "2k4"
+		(property "Value" "2k4 ¼W"
 			(at 201.93 69.088 90)
 			(show_name no)
@@
 			)
 		)
-		(property "Footprint" "Resistor_SMD:R_0402_1005Metric"
+		(property "Footprint" "Resistor_SMD:R_0603_1608Metric"
 			(at 202.184 72.136 90)
 			(hide yes)
@@
 			)
 		)
-		(property "Value" "2k 500mW"
+		(property "Value" "2k ½W"
 			(at 153.924 134.62 0)
 			(show_name no)
@@
 			)
 		)
-		(property "Value" "2k4"
+		(property "Value" "2k4 ¼W"
 			(at 162.56 47.498 90)
 			(show_name no)
@@
 			)
 		)
-		(property "Footprint" "Resistor_SMD:R_0402_1005Metric"
+		(property "Footprint" "Resistor_SMD:R_0603_1608Metric"
 			(at 162.814 50.546 90)
 			(hide yes)
@@
 			)
 		)
-		(property "Value" "2k4"
+		(property "Value" "2k4 ¼W"
 			(at 193.04 47.498 90)
 			(show_name no)
@@
 			)
 		)
-		(property "Footprint" "Resistor_SMD:R_0402_1005Metric"
+		(property "Footprint" "Resistor_SMD:R_0603_1608Metric"
 			(at 193.294 50.546 90)
 			(hide yes)
@@
 			)
 		)
-		(property "Value" "2k4"
+		(property "Value" "2k4 ¼W"
 			(at 153.67 69.088 90)
 			(show_name no)
@@
 			)
 		)
-		(property "Footprint" "Resistor_SMD:R_0402_1005Metric"
+		(property "Footprint" "Resistor_SMD:R_0603_1608Metric"
 			(at 153.924 72.136 90)
 			(hide yes)
@@
 			)
 		)
-		(property "Value" "2k 500mW"
+		(property "Value" "2k ½W"
 			(at 65.024 39.37 0)
 			(show_name no)
@@
 			)
 		)
-		(property "Value" "2k 500mW"
+		(property "Value" "2k ½W"
 			(at 153.924 97.79 0)
 			(show_name no)
@@
 			)
 		)
-		(property "Value" "2k 500mW"
+		(property "Value" "2k ½W"
 			(at 120.904 67.31 0)
 			(show_name no)
@@
 			)
 		)
-		(property "Value" "2k 500mW"
+		(property "Value" "2k ½W"
 			(at 65.024 113.03 0)
 			(show_name no)
@@
 			)
 		)
-		(property "Value" "2k 500mW"
+		(property "Value" "2k ½W"
 			(at 209.804 99.06 0)
 			(show_name no)
@@
 			)
 		)
-		(property "Value" "2k 500mW"
+		(property "Value" "2k ½W"
 			(at 65.024 76.2 0)
 			(show_name no)

Commit message: Clean up sheet frames.
Other:
- company: © 1962 General Precision; redrawn by Sam Hanes -> © 2026 Sam Hanes, licensed CERN-OHL-W v2
- title: LGP-21 P & Q Register Board -> LGP-21 Mini - P&Q Register
Changed lines of the file:
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@@
 	(generator "eeschema")
 	(generator_version "10.0")
-	(paper "A")
+	(paper "USLetter")
 	(title_block
-		(title "LGP-21 P & Q Register Board")
-		(date "2026-06-15")
-		(rev "ESD 1060")
-		(company "© 1962 General Precision; redrawn by Sam Hanes")
-		(comment 1 "https://github.com/Elemecca/lgp21-docs")
+		(title "LGP-21 Mini - P&Q Register")
+		(date "2026-06-28")
+		(rev "A")
+		(company "© 2026 Sam Hanes, licensed CERN-OHL-W v2")
+		(comment 1 "https://github.com/Elemecca/lgp21-mini")
 	)
 	(text "P5"
