File: boards/pq-register/P5.kicad_sch (KiCad schematic)
At the start: 64 parts, among them Q30 MMBT5401, Q31 MMBT5401, Q32 MMBT5401, Q33 MMBT5401, Q34 MMBT5401, Q35 MMBT5401, Q36 MMBT5401, Q37 MMBT5401, Q50 MMBT5401

Commit message: Route resistors in the second column.
Parts:
- R144, R155: value 2k4 ¼W -> 2k4; footprint Resistor_SMD:R_0603_1608Metric -> Resistor_SMD:R_0402_1005Metric
Changed lines of the file:
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@@
 			)
 		)
-		(property "Value" "2k4 ¼W"
+		(property "Value" "2k4"
 			(at 201.93 69.088 90)
 			(show_name no)
@@
 			)
 		)
-		(property "Footprint" "Resistor_SMD:R_0603_1608Metric"
+		(property "Footprint" "Resistor_SMD:R_0402_1005Metric"
 			(at 202.184 72.136 90)
 			(hide yes)
@@
 			)
 		)
-		(property "Value" "2k4 ¼W"
+		(property "Value" "2k4"
 			(at 153.67 69.088 90)
 			(show_name no)
@@
 			)
 		)
-		(property "Footprint" "Resistor_SMD:R_0603_1608Metric"
+		(property "Footprint" "Resistor_SMD:R_0402_1005Metric"
 			(at 153.924 72.136 90)
 			(hide yes)

Commit message: Route passives in the rightmost column.
Parts:
- R900: renamed from R256; now fitted
Changed lines of the file:
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@@
 		(on_board yes)
 		(in_pos_files yes)
-		(dnp yes)
-		(property "Reference" "R256"
+		(dnp no)
+		(property "Reference" "R900"
 			(at 44.45 49.784 90)
 			(show_name no)
@@
 			(project "pq-register"
 				(path "/d5da316c-1ec9-4d99-8330-1c4a3f6c3ba4/57c22bd7-5c59-41f0-a879-47621ba4147d"
-					(reference "R256")
+					(reference "R900")
 					(unit 1)
 				)

Commit message: Rough route the left column.
Connections:
- net β5 renamed ~{β5}
Changed lines of the file:
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@@
 		)
 	)
-	(global_label "β5"
+	(global_label "~{β5}"
 		(shape output)
 		(at 88.9 43.18 0)

Commit message: Add script to export production files.
Parts:
- C17, C20: BOM Value (none) -> 120pF
- C18, C19: BOM Value (none) -> 680pF
- CR10, CR9: value 1N5819WS -> 1N4148WS; BOM Value (none) -> 1N4148WS; LCSC (none) -> C2128
- Q30, Q31, Q32, Q33, Q34, Q35, Q36, Q37, Q50: BOM Value (none) -> MMBT5401; LCSC (none) -> C8326
- R128, R130: BOM Value (none) -> 300Ω 3W
- R133, R134, R135, R136, R137, R138, R139, R140, R141, R142, R143, R145, R146, R147, R148, R149, R150, R151, R152, R153, R154, R209, R210, R211, R212, R213, R900: BOM Value (none) -> 15kΩ
- R144, R155: BOM Value (none) -> 2.4kΩ
- R156, R157: BOM Value (none) -> 2.4kΩ 250mW
- R221, R223, R225, R227, R229, R231, R257: BOM Value (none) -> 56kΩ
- R222, R224, R226, R228, R230, R232, R258: BOM Value (none) -> 2kΩ 500mW
- R233, R234: BOM Value (none) -> 33kΩ
