File: boards/pq-register/P6.kicad_sch (KiCad schematic)
At the start: 93 parts, among them Q38 MMBT5401, Q39 MMBT5401, Q40 MMBT5401, Q41 MMBT5401, Q42 MMBT5401, Q43 MMBT5401, Q44 MMBT5401, Q45 MMBT5401, Q46 MMBT5401, Q47 MMBT5401, Q48 MMBT5401, Q49 MMBT5401

Commit message: Better PCI footprint, more layout.
Connections:
- net CP renamed CP_{1}
Changed lines of the file:
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@@
 		(property "Intersheetrefs" "${INTERSHEET_REFS}"
 			(at 143.1253 151.13 0)
-			(hide yes)
 			(show_name no)
 			(do_not_autoplace no)
@@
 		(property "Intersheetrefs" "${INTERSHEET_REFS}"
 			(at 95.47 111.76 0)
-			(hide yes)
 			(show_name no)
 			(do_not_autoplace no)
@@
 		(property "Intersheetrefs" "${INTERSHEET_REFS}"
 			(at 144.3348 109.22 0)
-			(hide yes)
 			(show_name no)
 			(do_not_autoplace no)
@@
 		(property "Intersheetrefs" "${INTERSHEET_REFS}"
 			(at 144.5162 114.3 0)
-			(hide yes)
 			(show_name no)
 			(do_not_autoplace no)
@@
 		(property "Intersheetrefs" "${INTERSHEET_REFS}"
 			(at 35.1148 41.91 0)
-			(hide yes)
 			(show_name no)
 			(do_not_autoplace no)
@@
 		(property "Intersheetrefs" "${INTERSHEET_REFS}"
 			(at 93.5953 106.68 0)
-			(hide yes)
 			(show_name no)
 			(do_not_autoplace no)
@@
 		(property "Intersheetrefs" "${INTERSHEET_REFS}"
 			(at 225.1747 24.13 0)
-			(hide yes)
 			(show_name no)
 			(do_not_autoplace no)
@@
 		(property "Intersheetrefs" "${INTERSHEET_REFS}"
 			(at 35.4777 83.82 0)
-			(hide yes)
 			(show_name no)
 			(do_not_autoplace no)
@@
 		(property "Intersheetrefs" "${INTERSHEET_REFS}"
 			(at 36.5662 78.74 0)
-			(hide yes)
 			(show_name no)
 			(do_not_autoplace no)
@@
 		(property "Intersheetrefs" "${INTERSHEET_REFS}"
 			(at 93.5348 172.72 0)
-			(hide yes)
 			(show_name no)
 			(do_not_autoplace no)
@@
 		(property "Intersheetrefs" "${INTERSHEET_REFS}"
 			(at 144.5162 124.46 0)
-			(hide yes)
 			(show_name no)
 			(do_not_autoplace no)
@@
 		(property "Intersheetrefs" "${INTERSHEET_REFS}"
 			(at 94.7443 167.64 0)
-			(hide yes)
 			(show_name no)
 			(do_not_autoplace no)
@@
 		(property "Intersheetrefs" "${INTERSHEET_REFS}"
 			(at 225.1747 41.91 0)
-			(hide yes)
 			(show_name no)
 			(do_not_autoplace no)
@@
 		(property "Intersheetrefs" "${INTERSHEET_REFS}"
 			(at 144.2743 161.29 0)
-			(hide yes)
 			(show_name no)
 			(do_not_autoplace no)
@@
 		(property "Intersheetrefs" "${INTERSHEET_REFS}"
 			(at 35.4777 26.67 0)
-			(hide yes)
 			(show_name no)
 			(do_not_autoplace no)
@@
 		(property "Intersheetrefs" "${INTERSHEET_REFS}"
 			(at 143.0648 156.21 0)
-			(hide yes)
 			(show_name no)
 			(do_not_autoplace no)
@@
 		(property "Intersheetrefs" "${INTERSHEET_REFS}"
 			(at 93.8977 187.96 0)
-			(hide yes)
 			(show_name no)
 			(do_not_autoplace no)
@@
 		(property "Intersheetrefs" "${INTERSHEET_REFS}"
 			(at 36.3243 120.65 0)
-			(hide yes)
 			(show_name no)
 			(do_not_autoplace no)
@@
 		(property "Intersheetrefs" "${INTERSHEET_REFS}"
 			(at 36.5662 100.33 0)
-			(hide yes)
-			(show_name no)
-			(do_not_autoplace no)
-			(effects
-				(font
-					(size 1.27 1.27)
-				)
-				(justify right)
-			)
-		)
-	)
-	(global_label "CP"
+			(show_name no)
+			(do_not_autoplace no)
+			(effects
+				(font
+					(size 1.27 1.27)
+				)
+				(justify right)
+			)
+		)
+	)
+	(global_label "CP_{1}"
 		(shape input)
 		(at 177.8 68.58 270)
@@
 		)
 		(property "Intersheetrefs" "${INTERSHEET_REFS}"
-			(at 177.8 74.1052 90)
-			(hide yes)
+			(at 177.8 75.1236 90)
 			(show_name no)
 			(do_not_autoplace no)
@@
 		(property "Intersheetrefs" "${INTERSHEET_REFS}"
 			(at 35.4777 105.41 0)
-			(hide yes)
 			(show_name no)
 			(do_not_autoplace no)
@@
 		(property "Intersheetrefs" "${INTERSHEET_REFS}"
 			(at 144.2743 104.14 0)
-			(hide yes)
 			(show_name no)
 			(do_not_autoplace no)
@@
 		(property "Intersheetrefs" "${INTERSHEET_REFS}"
 			(at 143.4277 140.97 0)
-			(hide yes)
 			(show_name no)
 			(do_not_autoplace no)
@@
 		(property "Intersheetrefs" "${INTERSHEET_REFS}"
 			(at 196.5863 130.81 0)
-			(hide yes)
 			(show_name no)
 			(do_not_autoplace no)
@@
 		(property "Intersheetrefs" "${INTERSHEET_REFS}"
 			(at 195.3163 125.73 0)
-			(hide yes)
 			(show_name no)
 			(do_not_autoplace no)
@@
 		(property "Intersheetrefs" "${INTERSHEET_REFS}"
 			(at 35.1753 36.83 0)
-			(hide yes)
 			(show_name no)
 			(do_not_autoplace no)
@@
 		(property "Intersheetrefs" "${INTERSHEET_REFS}"
 			(at 36.3243 46.99 0)
-			(hide yes)
 			(show_name no)
 			(do_not_autoplace no)
@@
 		(property "Intersheetrefs" "${INTERSHEET_REFS}"
 			(at 35.5986 31.75 0)
-			(hide yes)
 			(show_name no)
 			(do_not_autoplace no)
@@
 		(property "Intersheetrefs" "${INTERSHEET_REFS}"
 			(at 35.1753 73.66 0)
-			(hide yes)
 			(show_name no)
 			(do_not_autoplace no)
@@
 		(property "Intersheetrefs" "${INTERSHEET_REFS}"
 			(at 143.4277 129.54 0)
-			(hide yes)
 			(show_name no)
 			(do_not_autoplace no)
@@
 		(property "Intersheetrefs" "${INTERSHEET_REFS}"
 			(at 93.5953 177.8 0)
-			(hide yes)
 			(show_name no)
 			(do_not_autoplace no)
@@
 		(property "Intersheetrefs" "${INTERSHEET_REFS}"
 			(at 36.3243 63.5 0)
-			(hide yes)
 			(show_name no)
 			(do_not_autoplace no)
@@
 		(property "Intersheetrefs" "${INTERSHEET_REFS}"
 			(at 35.1753 152.4 0)
-			(hide yes)
 			(show_name no)
 			(do_not_autoplace no)
@@
 		(property "Intersheetrefs" "${INTERSHEET_REFS}"
 			(at 34.0263 125.73 0)
-			(hide yes)
 			(show_name no)
 			(do_not_autoplace no)
@@
 		(property "Intersheetrefs" "${INTERSHEET_REFS}"
 			(at 141.9763 119.38 0)
-			(hide yes)
 			(show_name no)
 			(do_not_autoplace no)
@@
 		(property "Intersheetrefs" "${INTERSHEET_REFS}"
 			(at 35.1148 68.58 0)
-			(hide yes)
 			(show_name no)
 			(do_not_autoplace no)
@@
 		(property "Intersheetrefs" "${INTERSHEET_REFS}"
 			(at 37.05 147.32 0)
-			(hide yes)
 			(show_name no)
 			(do_not_autoplace no)
@@
 		(property "Intersheetrefs" "${INTERSHEET_REFS}"
 			(at 36.5662 110.49 0)
-			(hide yes)
 			(show_name no)
 			(do_not_autoplace no)
@@
 		(property "Intersheetrefs" "${INTERSHEET_REFS}"
 			(at 94.0186 182.88 0)
-			(hide yes)
 			(show_name no)
 			(do_not_autoplace no)
@@
 		(property "Intersheetrefs" "${INTERSHEET_REFS}"
 			(at 144.5162 146.05 0)
-			(hide yes)
 			(show_name no)
 			(do_not_autoplace no)
@@
 		(property "Intersheetrefs" "${INTERSHEET_REFS}"
 			(at 36.3848 115.57 0)
-			(hide yes)
 			(show_name no)
 			(do_not_autoplace no)
@@
 		(property "Intersheetrefs" "${INTERSHEET_REFS}"
 			(at 87.4267 59.69 0)
-			(hide yes)
-			(show_name no)
-			(do_not_autoplace no)
+			(show_name no)
+			(do_not_autoplace no)

Commit message: Start updating 2k4 resistors to 0603, melt some traces.
Parts:
- R181, R206, R207, R208: value 2k4 -> 2k4 ¼W; footprint Resistor_SMD:R_0402_1005Metric -> Resistor_SMD:R_0603_1608Metric
- R236, R238, R240, R242, R244, R246, R248, R250, R252, R254: value 2k 500mW -> 2k ½W
Changed lines of the file:
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@@
 			)
 		)
-		(property "Value" "2k 500mW"
+		(property "Value" "2k ½W"
 			(at 65.024 139.7 0)
 			(show_name no)
@@
 			)
 		)
-		(property "Value" "2k 500mW"
+		(property "Value" "2k ½W"
 			(at 65.024 29.21 0)
 			(show_name no)
@@
 			)
 		)
-		(property "Value" "2k 500mW"
+		(property "Value" "2k ½W"
 			(at 65.024 102.87 0)
 			(show_name no)
@@
 			)
 		)
-		(property "Value" "2k4"
+		(property "Value" "2k4 ¼W"
 			(at 201.93 64.008 90)
 			(show_name no)
@@
 			)
 		)
-		(property "Footprint" "Resistor_SMD:R_0402_1005Metric"
+		(property "Footprint" "Resistor_SMD:R_0603_1608Metric"
 			(at 202.184 67.056 90)
 			(hide yes)
@@
 			)
 		)
-		(property "Value" "2k 500mW"
+		(property "Value" "2k ½W"
 			(at 172.974 143.51 0)
 			(show_name no)
@@
 			)
 		)
-		(property "Value" "2k4"
+		(property "Value" "2k4 ¼W"
 			(at 193.04 42.418 90)
 			(show_name no)
@@
 			)
 		)
-		(property "Footprint" "Resistor_SMD:R_0402_1005Metric"
+		(property "Footprint" "Resistor_SMD:R_0603_1608Metric"
 			(at 193.294 45.466 90)
 			(hide yes)
@@
 			)
 		)
-		(property "Value" "2k 500mW"
+		(property "Value" "2k ½W"
 			(at 123.444 170.18 0)
 			(show_name no)
@@
 			)
 		)
-		(property "Value" "2k 500mW"
+		(property "Value" "2k ½W"
 			(at 65.024 66.04 0)
 			(show_name no)
@@
 			)
 		)
-		(property "Value" "2k 500mW"
+		(property "Value" "2k ½W"
 			(at 172.974 106.68 0)
 			(show_name no)
@@
 			)
 		)
-		(property "Value" "2k4"
+		(property "Value" "2k4 ¼W"
 			(at 162.56 42.418 90)
 			(show_name no)
@@
 			)
 		)
-		(property "Footprint" "Resistor_SMD:R_0402_1005Metric"
+		(property "Footprint" "Resistor_SMD:R_0603_1608Metric"
 			(at 162.814 45.466 90)
 			(hide yes)
@@
 			)
 		)
-		(property "Value" "2k 500mW"
+		(property "Value" "2k ½W"
 			(at 123.444 99.06 0)
 			(show_name no)
@@
 			)
 		)
-		(property "Value" "2k 500mW"
+		(property "Value" "2k ½W"
 			(at 226.314 107.95 0)
 			(show_name no)
@@
 			)
 		)
-		(property "Value" "2k4"
+		(property "Value" "2k4 ¼W"
 			(at 153.67 64.008 90)
 			(show_name no)
@@
 			)
 		)
-		(property "Footprint" "Resistor_SMD:R_0402_1005Metric"
+		(property "Footprint" "Resistor_SMD:R_0603_1608Metric"
 			(at 153.924 67.056 90)
 			(hide yes)
@@
 			)
 		)
-		(property "Value" "2k 500mW"
+		(property "Value" "2k ½W"
 			(at 118.364 62.23 0)
 			(show_name no)

Commit message: Clean up sheet frames.
Other:
- company: © 1962 General Precision; redrawn by Sam Hanes -> © 2026 Sam Hanes, licensed CERN-OHL-W v2
- title: LGP-21 P & Q Register Board -> LGP-21 Mini - P&Q Register
Changed lines of the file:
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@@
 	(generator "eeschema")
 	(generator_version "10.0")
-	(paper "A")
+	(paper "USLetter")
 	(title_block
-		(title "LGP-21 P & Q Register Board")
-		(date "2026-06-15")
-		(rev "ESD 1060")
-		(company "© 1962 General Precision; redrawn by Sam Hanes")
-		(comment 1 "https://github.com/Elemecca/lgp21-docs")
+		(title "LGP-21 Mini - P&Q Register")
+		(date "2026-06-28")
+		(rev "A")
+		(company "© 2026 Sam Hanes, licensed CERN-OHL-W v2")
+		(comment 1 "https://github.com/Elemecca/lgp21-mini")
 	)
 	(text "P6"
