File: boards/pq-register/P6.kicad_sch (KiCad schematic)
At the start: 93 parts, among them Q38 MMBT5401, Q39 MMBT5401, Q40 MMBT5401, Q41 MMBT5401, Q42 MMBT5401, Q43 MMBT5401, Q44 MMBT5401, Q45 MMBT5401, Q46 MMBT5401, Q47 MMBT5401, Q48 MMBT5401, Q49 MMBT5401

Commit message: Route resistors in the second column.
Parts:
- R181, R206: value 2k4 ¼W -> 2k4; footprint Resistor_SMD:R_0603_1608Metric -> Resistor_SMD:R_0402_1005Metric
Changed lines of the file:
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@@
 			)
 		)
-		(property "Value" "2k4 ¼W"
+		(property "Value" "2k4"
 			(at 201.93 64.008 90)
 			(show_name no)
@@
 			)
 		)
-		(property "Footprint" "Resistor_SMD:R_0603_1608Metric"
+		(property "Footprint" "Resistor_SMD:R_0402_1005Metric"
 			(at 202.184 67.056 90)
 			(hide yes)
@@
 			)
 		)
-		(property "Value" "2k4 ¼W"
+		(property "Value" "2k4"
 			(at 153.67 64.008 90)
 			(show_name no)
@@
 			)
 		)
-		(property "Footprint" "Resistor_SMD:R_0603_1608Metric"
+		(property "Footprint" "Resistor_SMD:R_0402_1005Metric"
 			(at 153.924 67.056 90)
 			(hide yes)

Commit message: Add script to export production files.
Parts:
- C21, C24: BOM Value (none) -> 120pF
- C22, C23: BOM Value (none) -> 680pF
- CR11, CR12: value 1N5819WS -> 1N4148WS; BOM Value (none) -> 1N4148WS; LCSC (none) -> C2128
- Q38, Q39, Q40, Q41, Q42, Q43, Q44, Q45, Q46, Q47, Q48, Q49: BOM Value (none) -> MMBT5401; LCSC (none) -> C8326
- R158, R159, R160, R161, R162, R163, R164, R165, R166, R167, R168, R169, R170, R171, R172, R173, R174, R175, R176, R177, R178, R179, R180, R182, R183, R184, R185, R186, R187, R188, R189, R190, R191, R192, R193, R194, R195, R196, R197, R198, R199, R200, R201, R202, R203, R204, R205: BOM Value (none) -> 15kΩ
- R181, R206: BOM Value (none) -> 2.4kΩ
- R207, R208: BOM Value (none) -> 2.4kΩ 250mW
- R235, R237, R239, R241, R243, R245, R247, R249, R251, R253: BOM Value (none) -> 56kΩ
- R236, R238, R240, R242, R244, R246, R248, R250, R252, R254: BOM Value (none) -> 2kΩ 500mW
- R280, R64: BOM Value (none) -> 300Ω 3W
- R512, R513: BOM Value (none) -> 33kΩ
