File: boards/pq-register/Q3.kicad_sch (KiCad schematic)
At the start: 51 parts, among them Q101 MMBT5401, Q63 MMBT5401, Q83 MMBT5401, Q84 MMBT5401, Q85 MMBT5401, Q86 MMBT5401, Q87 MMBT5401, Q88 MMBT5401

Commit message: Better PCI footprint, more layout.
Connections:
- net ~{Q3_{S}}: now reaches C35.2, Q101.1 (B), Q88.3 (C), R411.1, R500.2
- net CP renamed CP_{2}
Other:
- moved on the sheet: Q85, R406, R407, R471, R472

Commit message: Start updating 2k4 resistors to 0603, melt some traces.
Parts:
- R282, R468, R470, R472, R474: value 2k 500mW -> 2k ½W
- R405, R410, R411, R412: value 2k4 -> 2k4 ¼W; footprint Resistor_SMD:R_0402_1005Metric -> Resistor_SMD:R_0603_1608Metric
Changed lines of the file:
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@@
 			)
 		)
-		(property "Value" "2k4"
+		(property "Value" "2k4 ¼W"
 			(at 143.51 90.678 90)
 			(show_name no)
@@
 			)
 		)
-		(property "Footprint" "Resistor_SMD:R_0402_1005Metric"
+		(property "Footprint" "Resistor_SMD:R_0603_1608Metric"
 			(at 143.764 93.726 90)
 			(hide yes)
@@
 			)
 		)
-		(property "Value" "2k4"
+		(property "Value" "2k4 ¼W"
 			(at 191.77 90.678 90)
 			(show_name no)
@@
 			)
 		)
-		(property "Footprint" "Resistor_SMD:R_0402_1005Metric"
+		(property "Footprint" "Resistor_SMD:R_0603_1608Metric"
 			(at 192.024 93.726 90)
 			(hide yes)
@@
 			)
 		)
-		(property "Value" "2k 500mW"
+		(property "Value" "2k ½W"
 			(at 183.134 116.84 0)
 			(show_name no)
@@
 			)
 		)
-		(property "Value" "2k 500mW"
+		(property "Value" "2k ½W"
 			(at 134.874 120.65 0)
 			(show_name no)
@@
 			)
 		)
-		(property "Value" "2k4"
+		(property "Value" "2k4 ¼W"
 			(at 182.88 69.088 90)
 			(show_name no)
@@
 			)
 		)
-		(property "Footprint" "Resistor_SMD:R_0402_1005Metric"
+		(property "Footprint" "Resistor_SMD:R_0603_1608Metric"
 			(at 183.134 72.136 90)
 			(hide yes)
@@
 			)
 		)
-		(property "Value" "2k4"
+		(property "Value" "2k4 ¼W"
 			(at 152.4 69.088 90)
 			(show_name no)
@@
 			)
 		)
-		(property "Footprint" "Resistor_SMD:R_0402_1005Metric"
+		(property "Footprint" "Resistor_SMD:R_0603_1608Metric"
 			(at 152.654 72.136 90)
 			(hide yes)
@@
 			)
 		)
-		(property "Value" "2k 500mW"
+		(property "Value" "2k ½W"
 			(at 57.404 129.54 0)
 			(show_name no)
@@
 			)
 		)
-		(property "Value" "2k 500mW"
+		(property "Value" "2k ½W"
 			(at 95.504 88.9 0)
 			(show_name no)
@@
 			)
 		)
-		(property "Value" "2k 500mW"
+		(property "Value" "2k ½W"
 			(at 57.404 92.71 0)
 			(show_name no)

Commit message: Clean up sheet frames.
Other:
- company: © 1962 General Precision; redrawn by Sam Hanes -> © 2026 Sam Hanes, licensed CERN-OHL-W v2
- title: LGP-21 P & Q Register Board -> LGP-21 Mini - P&Q Register
Changed lines of the file:
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@@
 	(generator "eeschema")
 	(generator_version "10.0")
-	(paper "A")
+	(paper "USLetter")
 	(title_block
-		(title "LGP-21 P & Q Register Board")
-		(date "2026-06-15")
-		(rev "ESD 1060")
-		(company "© 1962 General Precision; redrawn by Sam Hanes")
-		(comment 1 "https://github.com/Elemecca/lgp21-docs")
+		(title "LGP-21 Mini - P&Q Register")
+		(date "2026-06-28")
+		(rev "A")
+		(company "© 2026 Sam Hanes, licensed CERN-OHL-W v2")
+		(comment 1 "https://github.com/Elemecca/lgp21-mini")
 	)
 	(text "Q3"
