File: boards/pq-register/Q3.kicad_sch (KiCad schematic)
At the start: 51 parts, among them Q101 MMBT5401, Q63 MMBT5401, Q83 MMBT5401, Q84 MMBT5401, Q85 MMBT5401, Q86 MMBT5401, Q87 MMBT5401, Q88 MMBT5401

Commit message: Route resistors in the second column.
Parts:
- R405, R410: value 2k4 ¼W -> 2k4; footprint Resistor_SMD:R_0603_1608Metric -> Resistor_SMD:R_0402_1005Metric
Changed lines of the file:
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@@
 			)
 		)
-		(property "Value" "2k4 ¼W"
+		(property "Value" "2k4"
 			(at 143.51 90.678 90)
 			(show_name no)
@@
 			)
 		)
-		(property "Footprint" "Resistor_SMD:R_0603_1608Metric"
+		(property "Footprint" "Resistor_SMD:R_0402_1005Metric"
 			(at 143.764 93.726 90)
 			(hide yes)
@@
 			)
 		)
-		(property "Value" "2k4 ¼W"
+		(property "Value" "2k4"
 			(at 191.77 90.678 90)
 			(show_name no)
@@
 			)
 		)
-		(property "Footprint" "Resistor_SMD:R_0603_1608Metric"
+		(property "Footprint" "Resistor_SMD:R_0402_1005Metric"
 			(at 192.024 93.726 90)
 			(hide yes)

Commit message: Route passives in the rightmost column.
Parts:
- R905: renamed from R511; now fitted
Connections:
- net B1: now reaches R905.1
- no-connect marks 1 -> 0
Changed lines of the file:
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@@
 		(color 0 0 0 0)
 	)
-	(no_connect
-		(at 33.02 115.57)
-	)
 	(wire
 		(pts
@@
 		)
 	)
+	(global_label "B1"
+		(shape input)
+		(at 33.02 115.57 180)
+		(fields_autoplaced yes)
+		(effects
+			(font
+				(size 1.27 1.27)
+			)
+			(justify right)
+		)
+		(property "Intersheetrefs" "${INTERSHEET_REFS}"
+			(at 27.5553 115.57 0)
+			(show_name no)
+			(do_not_autoplace no)
+			(effects
+				(font
+					(size 1.27 1.27)
+				)
+				(justify right)
+			)
+		)
+	)
 	(global_label "~{bq}"
 		(shape input)
@@
 		(on_board yes)
 		(in_pos_files yes)
-		(dnp yes)
-		(property "Reference" "R511"
+		(dnp no)
+		(property "Reference" "R905"
 			(at 36.83 113.284 90)
 			(show_name no)
@@
 			(project "pq-register"
 				(path "/d5da316c-1ec9-4d99-8330-1c4a3f6c3ba4/f1bfd5ae-8a8b-41b5-a3d1-70c5dff4adf1"
-					(reference "R511")
+					(reference "R905")
 					(unit 1)
 				)
@@
 		)
 	)
+	(group ""
+		(lib_id "Project:emitter-follower")
+		(members "1c2f65ec-bd52-4802-9d12-0c55807f1893" "29c78692-4cf8-4ed1-b3da-35a81dfd88b1"
+			"2b814adf-5036-466c-9e1d-53c2fd4f132a" "4ca50ffc-425b-4cff-9f89-0e66fef23dba"
+			"573b71fa-b508-4e68-b3f7-4c7eadc2a910" "6022987c-3010-41c4-a58d-13afa00b75f8"
+			"6b943d04-fd8f-40dc-a871-057e5a463f8b" "6d92eac0-67d6-4156-a4f2-5769c16a6f9a"
+			"7af3b50b-a788-4f84-bef8-71831ecb5b6a" "849244a5-e7a4-4b7e-9585-d1d1ebfb1b42"
+			"89977826-6dad-4e67-9ed1-5c7cd6d16374" "8ca0d968-3556-47bf-89b2-3c7fba821f5a"
+			"e038cc43-45da-4725-b628-e01793e83dbb" "e31192bb-dc70-42be-bae2-c27a337a47d5"
+			"e92237c1-927e-437e-b534-37bf132dad79" "eb00264a-098f-4e65-bec8-02a59b7474b0"
+		)
+	)

Commit message: Assorted cleanup and silkscreen.
Parts:
- renumbered R905 to R901
Changed lines of the file:
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@@
 		(in_pos_files yes)
 		(dnp no)
-		(property "Reference" "R905"
+		(property "Reference" "R901"
 			(at 36.83 113.284 90)
 			(show_name no)
@@
 			(project "pq-register"
 				(path "/d5da316c-1ec9-4d99-8330-1c4a3f6c3ba4/f1bfd5ae-8a8b-41b5-a3d1-70c5dff4adf1"
-					(reference "R905")
+					(reference "R901")
 					(unit 1)
 				)

Commit message: Add script to export production files.
Parts:
- C35, C38: BOM Value (none) -> 120pF
- C36, C37: BOM Value (none) -> 680pF
- CR17, CR18, CR21, CR22, CR23: value 1N5819WS -> 1N4148WS; BOM Value (none) -> 1N4148WS; LCSC (none) -> C2128
- Q101, Q63, Q83, Q84, Q85, Q86, Q87, Q88: BOM Value (none) -> MMBT5401; LCSC (none) -> C8326
- R281, R467, R469, R471, R473, R499: BOM Value (none) -> 56kΩ
- R282, R468, R470, R472, R474: BOM Value (none) -> 2kΩ 500mW
- R334, R335, R336, R337, R338, R339, R400, R401, R402, R403, R406, R407, R408, R409, R901: BOM Value (none) -> 15kΩ
- R383, R500: BOM Value (none) -> 300Ω 3W
- R405, R410: BOM Value (none) -> 2.4kΩ
- R411, R412: BOM Value (none) -> 2.4kΩ 250mW
- R475, R476: BOM Value (none) -> 33kΩ
