File: boards/pq-register/Q4.kicad_sch (KiCad schematic)
At the start: 54 parts, among them Q89 MMBT5401, Q90 MMBT5401, Q91 MMBT5401, Q92 MMBT5401, Q93 MMBT5401, Q94 MMBT5401, Q95 MMBT5401, Q96 MMBT5401

Commit message: Better PCI footprint, more layout.
Connections:
- net CP renamed CP_{2}
Changed lines of the file:
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@@
 		(property "Intersheetrefs" "${INTERSHEET_REFS}"
 			(at 83.3748 148.59 0)
-			(hide yes)
 			(show_name no)
 			(do_not_autoplace no)
@@
 		(property "Intersheetrefs" "${INTERSHEET_REFS}"
 			(at 83.3748 172.72 0)
-			(hide yes)
 			(show_name no)
 			(do_not_autoplace no)
@@
 		(property "Intersheetrefs" "${INTERSHEET_REFS}"
 			(at 83.3748 193.04 0)
-			(hide yes)
 			(show_name no)
 			(do_not_autoplace no)
@@
 		(property "Intersheetrefs" "${INTERSHEET_REFS}"
 			(at 83.7377 182.88 0)
-			(hide yes)
 			(show_name no)
 			(do_not_autoplace no)
@@
 		(property "Intersheetrefs" "${INTERSHEET_REFS}"
 			(at 83.8586 187.96 0)
-			(hide yes)
 			(show_name no)
 			(do_not_autoplace no)
@@
 		(property "Intersheetrefs" "${INTERSHEET_REFS}"
 			(at 84.6448 177.8 0)
-			(hide yes)
 			(show_name no)
 			(do_not_autoplace no)
@@
 		(property "Intersheetrefs" "${INTERSHEET_REFS}"
 			(at 41.5858 59.69 0)
-			(hide yes)
 			(show_name no)
 			(do_not_autoplace no)
@@
 		(property "Intersheetrefs" "${INTERSHEET_REFS}"
 			(at 84.8262 133.35 0)
-			(hide yes)
 			(show_name no)
 			(do_not_autoplace no)
@@
 		(property "Intersheetrefs" "${INTERSHEET_REFS}"
 			(at 42.7348 64.77 0)
-			(hide yes)
 			(show_name no)
 			(do_not_autoplace no)
@@
 		(property "Intersheetrefs" "${INTERSHEET_REFS}"
 			(at 83.3748 143.51 0)
-			(hide yes)
 			(show_name no)
 			(do_not_autoplace no)
@@
 		(property "Intersheetrefs" "${INTERSHEET_REFS}"
 			(at 83.3748 167.64 0)
-			(hide yes)
 			(show_name no)
 			(do_not_autoplace no)
@@
 		(property "Intersheetrefs" "${INTERSHEET_REFS}"
 			(at 226.5052 43.18 0)
-			(hide yes)
 			(show_name no)
 			(do_not_autoplace no)
@@
 		(property "Intersheetrefs" "${INTERSHEET_REFS}"
 			(at 83.3748 99.06 0)
-			(hide yes)
 			(show_name no)
 			(do_not_autoplace no)
@@
 		(property "Intersheetrefs" "${INTERSHEET_REFS}"
 			(at 143.3068 110.49 0)
-			(hide yes)
 			(show_name no)
 			(do_not_autoplace no)
@@
 		(property "Intersheetrefs" "${INTERSHEET_REFS}"
 			(at 226.5052 25.4 0)
-			(hide yes)
 			(show_name no)
 			(do_not_autoplace no)
@@
 		(property "Intersheetrefs" "${INTERSHEET_REFS}"
 			(at 82.2258 104.14 0)
-			(hide yes)
 			(show_name no)
 			(do_not_autoplace no)
@@
 		(property "Intersheetrefs" "${INTERSHEET_REFS}"
 			(at 83.3748 138.43 0)
-			(hide yes)
-			(show_name no)
-			(do_not_autoplace no)
-			(effects
-				(font
-					(size 1.27 1.27)
-				)
-				(justify right)
-			)
-		)
-	)
-	(global_label "CP"
+			(show_name no)
+			(do_not_autoplace no)
+			(effects
+				(font
+					(size 1.27 1.27)
+				)
+				(justify right)
+			)
+		)
+	)
+	(global_label "CP_{2}"
 		(shape input)
 		(at 179.07 69.85 270)
@@
 		)
 		(property "Intersheetrefs" "${INTERSHEET_REFS}"
-			(at 179.07 75.3752 90)
-			(hide yes)
+			(at 179.07 76.3936 90)
 			(show_name no)
 			(do_not_autoplace no)
@@
 		(property "Intersheetrefs" "${INTERSHEET_REFS}"
 			(at 83.7377 128.27 0)
-			(hide yes)
-			(show_name no)
-			(do_not_autoplace no)
+			(show_name no)
+			(do_not_autoplace no)

Commit message: Start updating 2k4 resistors to 0603, melt some traces.
Parts:
- R416, R434, R435, R436: value 2k4 -> 2k4 ¼W; footprint Resistor_SMD:R_0402_1005Metric -> Resistor_SMD:R_0603_1608Metric
- R478, R480, R482, R484, R486, R488: value 2k 500mW -> 2k ½W
Changed lines of the file:
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@@
 			)
 		)
-		(property "Value" "2k4"
+		(property "Value" "2k4 ¼W"
 			(at 194.31 43.688 90)
 			(show_name no)
@@
 			)
 		)
-		(property "Footprint" "Resistor_SMD:R_0402_1005Metric"
+		(property "Footprint" "Resistor_SMD:R_0603_1608Metric"
 			(at 194.564 46.736 90)
 			(hide yes)
@@
 			)
 		)
-		(property "Value" "2k 500mW"
+		(property "Value" "2k ½W"
 			(at 72.644 52.07 0)
 			(show_name no)
@@
 			)
 		)
-		(property "Value" "2k 500mW"
+		(property "Value" "2k ½W"
 			(at 113.284 45.72 0)
 			(show_name no)
@@
 			)
 		)
-		(property "Value" "2k 500mW"
+		(property "Value" "2k ½W"
 			(at 113.284 130.81 0)
 			(show_name no)
@@
 			)
 		)
-		(property "Value" "2k4"
+		(property "Value" "2k4 ¼W"
 			(at 154.94 65.278 90)
 			(show_name no)
@@
 			)
 		)
-		(property "Footprint" "Resistor_SMD:R_0402_1005Metric"
+		(property "Footprint" "Resistor_SMD:R_0603_1608Metric"
 			(at 155.194 68.326 90)
 			(hide yes)
@@
 			)
 		)
-		(property "Value" "2k 500mW"
+		(property "Value" "2k ½W"
 			(at 172.974 92.71 0)
 			(show_name no)
@@
 			)
 		)
-		(property "Value" "2k 500mW"
+		(property "Value" "2k ½W"
 			(at 113.284 91.44 0)
 			(show_name no)
@@
 			)
 		)
-		(property "Value" "2k4"
+		(property "Value" "2k4 ¼W"
 			(at 203.2 65.278 90)
 			(show_name no)
@@
 			)
 		)
-		(property "Footprint" "Resistor_SMD:R_0402_1005Metric"
+		(property "Footprint" "Resistor_SMD:R_0603_1608Metric"
 			(at 203.454 68.326 90)
 			(hide yes)
@@
 			)
 		)
-		(property "Value" "2k 500mW"
+		(property "Value" "2k ½W"
 			(at 113.284 170.18 0)
 			(show_name no)
@@
 			)
 		)
-		(property "Value" "2k4"
+		(property "Value" "2k4 ¼W"
 			(at 163.83 43.688 90)
 			(show_name no)
@@
 			)
 		)
-		(property "Footprint" "Resistor_SMD:R_0402_1005Metric"
+		(property "Footprint" "Resistor_SMD:R_0603_1608Metric"
 			(at 164.084 46.736 90)
 			(hide yes)

Commit message: Clean up sheet frames.
Other:
- company: © 1962 General Precision; redrawn by Sam Hanes -> © 2026 Sam Hanes, licensed CERN-OHL-W v2
- title: LGP-21 P & Q Register Board -> LGP-21 Mini - P&Q Register
Changed lines of the file:
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@@
 	(generator "eeschema")
 	(generator_version "10.0")
-	(paper "A")
+	(paper "USLetter")
 	(title_block
-		(title "LGP-21 P & Q Register Board")
-		(date "2026-06-15")
-		(rev "ESD 1060")
-		(company "© 1962 General Precision; redrawn by Sam Hanes")
-		(comment 1 "https://github.com/Elemecca/lgp21-docs")
+		(title "LGP-21 Mini - P&Q Register")
+		(date "2026-06-28")
+		(rev "A")
+		(company "© 2026 Sam Hanes, licensed CERN-OHL-W v2")
+		(comment 1 "https://github.com/Elemecca/lgp21-mini")
 	)
 	(text "Q4"
