File: boards/pq-register/Q4.kicad_sch (KiCad schematic)
At the start: 54 parts, among them Q89 MMBT5401, Q90 MMBT5401, Q91 MMBT5401, Q92 MMBT5401, Q93 MMBT5401, Q94 MMBT5401, Q95 MMBT5401, Q96 MMBT5401

Commit message: Route resistors in the second column.
Parts:
- R416, R434: value 2k4 ¼W -> 2k4; footprint Resistor_SMD:R_0603_1608Metric -> Resistor_SMD:R_0402_1005Metric
Changed lines of the file:
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@@
 			)
 		)
-		(property "Value" "2k4 ¼W"
+		(property "Value" "2k4"
 			(at 154.94 65.278 90)
 			(show_name no)
@@
 			)
 		)
-		(property "Footprint" "Resistor_SMD:R_0603_1608Metric"
+		(property "Footprint" "Resistor_SMD:R_0402_1005Metric"
 			(at 155.194 68.326 90)
 			(hide yes)
@@
 			)
 		)
-		(property "Value" "2k4 ¼W"
+		(property "Value" "2k4"
 			(at 203.2 65.278 90)
 			(show_name no)
@@
 			)
 		)
-		(property "Footprint" "Resistor_SMD:R_0603_1608Metric"
+		(property "Footprint" "Resistor_SMD:R_0402_1005Metric"
 			(at 203.454 68.326 90)
 			(hide yes)

Commit message: Add script to export production files.
Parts:
- C39, C42: BOM Value (none) -> 120pF
- C40, C41: BOM Value (none) -> 680pF
- CR19, CR20: value 1N5819WS -> 1N4148WS; BOM Value (none) -> 1N4148WS; LCSC (none) -> C2128
- Q89, Q90, Q91, Q92, Q93, Q94, Q95, Q96: BOM Value (none) -> MMBT5401; LCSC (none) -> C8326
- R404, R503: BOM Value (none) -> 300Ω 3W
- R413, R414, R415, R417, R418, R419, R420, R421, R422, R423, R424, R425, R426, R427, R428, R429, R430, R431, R432, R433: BOM Value (none) -> 15kΩ
- R416, R434: BOM Value (none) -> 2.4kΩ
- R435, R436: BOM Value (none) -> 2.4kΩ 250mW
- R477, R479, R481, R483, R485, R487: BOM Value (none) -> 56kΩ
- R478, R480, R482, R484, R486, R488: BOM Value (none) -> 2kΩ 500mW
- R489, R490: BOM Value (none) -> 33kΩ
