File: boards/pq-register/pq-register.kicad_sch (KiCad schematic)
At the start: 48 parts, among them P1 Card Edge, Q51 MMBT5401, Q52 MMBT5401, Q53 MMBT5401, Q54 MMBT5401, Q55 MMBT5401, Q56 MMBT5401, Q97 MMBT5401, Q98 MMBT5401, Q99 MMBT5401

Commit message: Better PCI footprint, more layout.
Parts:
- P1: footprint Connector_PCBEdge:BUS_PCI -> Project:Bus_PCI_5V_32bit
Connections:
- net +15V: now also P1.A2 (+15V); no longer P1.A61 (+15V)
- net -15V: now also P1.A4 (-15V); no longer P1.A59 (-15V)
- net -20V: now also P1.A1 (-20V); no longer P1.A62 (-20V)
- net -20V_{D}: now also P1.A61 (-20V_{D}); no longer P1.A2 (-20V_{D})
- net A: now also P1.B16 (A); no longer P1.B45 (A)
- net A*: now also P1.B14 (A*); no longer P1.B47 (A*)
- net B1: now also P1.B39 (Bl); no longer P1.B22 (Bl)
- net F: now also P1.B25 (F); no longer P1.B36 (F)
- net Faf: now also P1.B40 (Faf); no longer P1.B21 (Faf)
- net G: now also P1.A6 (G); no longer P1.A57 (G)
- net GND: now also P1.A62 (GND); no longer P1.A1 (GND)
- net H: now also P1.B2 (H); no longer P1.B61 (H)
- net K: now also P1.B34 (K); no longer P1.B27 (K)
- net O1: now also P1.A44 (O1); no longer P1.A17 (O1)
- net P1: now also P1.A5 (P1); no longer P1.A58 (P1)
- net P2: now also P1.B29 (P2); no longer P1.B32 (P2)
- net P3: now also P1.B32 (P3); no longer P1.B29 (P3)
- net P4: now also P1.B31 (P4); no longer P1.B30 (P4)
- net P5: now also P1.B19 (P5); no longer P1.B42 (P5)
- net P5a: now also P1.A21 (P5a); no longer P1.A40 (P5a)
- net P6: now also P1.B28 (P6); no longer P1.B33 (P6)
- net P6a: now also P1.A25 (P6a); no longer P1.A36 (P6a)
- net Q1: now also P1.A57 (Q1); no longer P1.A6 (Q1)
- net Q1b: now also P1.A38 (Q1b); no longer P1.A23 (Q1b)
- net Q2: now also P1.B44 (Q2); no longer P1.B17 (Q2)
- net Q2a: now also P1.A40 (Q2a); no longer P1.A21 (Q2a)
- net Q3: now also P1.A58 (Q3); no longer P1.A5 (Q3)
- net Q4: now also P1.B43 (Q4); no longer P1.B18 (Q4)
- net R: now also P1.B42 (R); no longer P1.B19 (R)
- net S2: now also P1.A27 (S2); no longer P1.A34 (S2)
- net S3: now also P1.A30 (S3); no longer P1.A31 (S3)
- net T3: now also P1.A29 (T3); no longer P1.A32 (T3)
- net Tc: now also P1.A36 (Tc); no longer P1.A25 (Tc)
- net V: now also P1.A19 (V); no longer P1.A42 (V)
- net bs: now also P1.B30 (bs); no longer P1.B31 (bs)
- net ia: now also P1.A28 (ia); no longer P1.A33 (ia)
- net rl: now also P1.A8 (r1); no longer P1.A55 (r1)
- net ~{A*}: now also P1.B15 (~{A*}); no longer P1.B46 (~{A*})
- net ~{A}: now also P1.B13 (~{A}); no longer P1.B48 (~{A})
- net ~{C}: now also P1.B37 (~{C}); no longer P1.B24 (~{C})
- net ~{Faf}: now also P1.B48 (~{Faf}); no longer P1.B13 (~{Faf})
- net ~{F}: now also P1.B26 (~{F}); no longer P1.B35 (~{F})
- net ~{G}: now also P1.A7 (~{G}); no longer P1.A56 (~{G})
- net ~{H'}: now also P1.B46 (~{H'}); no longer P1.B15 (~{H'})
- net ~{H}: now also P1.A47 (~{H}); no longer P1.A14 (~{H})
- net ~{O1}: now also P1.A41 (~{O1}); no longer P1.A20 (~{O1})
- net ~{P1c}: now also P1.A9 (~{P1c}); no longer P1.A54 (~{P1c})
- net ~{P1d}: now also P1.A11 (~{P1d}); no longer P1.A52 (~{P1d})
- net ~{P1}: now also P1.A3 (~{P1}); no longer P1.A60 (~{P1})
- net ~{P2c}: now also P1.A12 (~{P2c}); no longer P1.A49 (~{P2c})
- net ~{P2d}: now also P1.A13 (~{P2d}); no longer P1.A48 (~{P2d})
- net ~{P2}: now also P1.A48 (~{P2}); no longer P1.A13 (~{P2})
- net ~{P3c}: now also P1.A14 (~{P3c}); no longer P1.A47 (~{P3c})
- net ~{P3d}: now also P1.A15 (~{P3d}); no longer P1.A46 (~{P3d})
- net ~{P3}: now also P1.A49 (~{P3}); no longer P1.A12 (~{P3})
- net ~{P4c}: now also P1.A16 (~{P4c}); no longer P1.A45 (~{P4c})
- net ~{P4d}: now also P1.A17 (~{P4d}); no longer P1.A44 (~{P4d})
- net ~{P4}: now also P1.A52 (~{P4}); no longer P1.A11 (~{P4})
- net ~{P5c}: now also P1.A20 (~{P5c}); no longer P1.A41 (~{P5c})
- net ~{P5d}: now also P1.A23 (~{P5d}); no longer P1.A38 (~{P5d})
- net ~{P5}: now also P1.A55 (~{P5}); no longer P1.A8 (~{P5})
- net ~{P6c}: now also P1.A24 (~{P6c}); no longer P1.A37 (~{P6c})
- net ~{P6d}: now also P1.A26 (~{P6d}); no longer P1.A35 (~{P6d})
- net ~{P6}: now also P1.B45 (~{P6}); no longer P1.B16 (~{P6})
- net ~{Q1d}: now also P1.A39 (~{Q1d}); no longer P1.A22 (~{Q1d})
- net ~{Q1}: now also P1.B61 (~{Q1}); no longer P1.B2 (~{Q1})
- net ~{Q2c}: now also P1.A43 (~{Q2c}); no longer P1.A18 (~{Q2c})
- net ~{Q2d}: now also P1.A45 (~{Q2d}); no longer P1.A16 (~{Q2d})
- net ~{Q2}: now also P1.B60 (~{Q2}); no longer P1.B3 (~{Q2})
- net ~{Q3}: now also P1.A59 (~{Q3}); no longer P1.A4 (~{Q3})
- net ~{Q4}: now also P1.B62 (~{Q4}); no longer P1.B1 (~{Q4})
- net ~{R}: now also P1.B41 (~{R}); no longer P1.B20 (~{R})
- net ~{S1}: now also P1.A46 (~{S1}); no longer P1.A15 (~{S1})
- net ~{S2}: now also P1.A54 (~{S2}); no longer P1.A9 (~{S2})
- net ~{Tb1}: now also P1.A32 (~{Tb1}); no longer P1.A29 (~{Tb1})
- net ~{Tb2}: now also P1.A31 (~{Tb2}); no longer P1.A30 (~{Tb2})
- net ~{Tb3}: now also P1.A34 (~{Tb3}); no longer P1.A27 (~{Tb3})
- net ~{Tb4}: now also P1.A35 (~{Tb4}); no longer P1.A26 (~{Tb4})
- net ~{To}: now also P1.B49 (~{To}); no longer P1.B12 (~{To})
- net ~{V}: now also P1.A22 (~{V}); no longer P1.A39 (~{V})
- net ~{bq}: now also P1.A53 (~{bq}); no longer P1.A10 (~{bq})
- net ~{ic}: now also P1.A33 (~{ic}); no longer P1.A28 (~{ic})
- net ~{rl}: now also P1.A10 (~{r1}); no longer P1.A53 (~{r1})
- net α9: now also P1.B47 (α9); no longer P1.B14 (α9)
- net Cp renamed CP
- net CP: now also P1.B27 (CP); no longer P1.B34 (CP)
- new net P1b: P1.B1 (P1b)
- no-connect marks 32 -> 31

Commit message: Start updating 2k4 resistors to 0603, melt some traces.
Parts:
- R260, R267, R492, R494, R496: value 2k 500mW -> 2k ½W
Changed lines of the file:
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@@
 			)
 		)
-		(property "Value" "2k 500mW"
+		(property "Value" "2k ½W"
 			(at 142.494 67.31 0)
 			(show_name no)
@@
 			)
 		)
-		(property "Value" "2k 500mW"
+		(property "Value" "2k ½W"
 			(at 142.494 114.3 0)
 			(show_name no)
@@
 			)
 		)
-		(property "Value" "2k 500mW"
+		(property "Value" "2k ½W"
 			(at 142.494 154.94 0)
 			(show_name no)
@@
 			)
 		)
-		(property "Value" "2k 500mW"
+		(property "Value" "2k ½W"
 			(at 180.594 66.04 0)
 			(show_name no)
@@
 			)
 		)
-		(property "Value" "2k 500mW"
+		(property "Value" "2k ½W"
 			(at 180.594 107.95 0)
 			(show_name no)

Commit message: Clean up sheet frames.
Other:
- company: © 1962 General Precision; redrawn by Sam Hanes -> © 2026 Sam Hanes, licensed CERN-OHL-W v2
- title: LGP-21 P & Q Register Board -> LGP-21 Mini - P&Q Register
Changed lines of the file:
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@@
 	(generator "eeschema")
 	(generator_version "10.0")
-	(paper "A")
+	(paper "USLetter")
 	(title_block
-		(title "LGP-21 P & Q Register Board")
-		(date "2026-06-15")
-		(rev "ESD 1060")
-		(company "© 1962 General Precision; redrawn by Sam Hanes")
-		(comment 1 "https://github.com/Elemecca/lgp21-docs")
+		(title "LGP-21 Mini - P&Q Register")
+		(date "2026-06-28")
+		(rev "A")
+		(company "© 2026 Sam Hanes, licensed CERN-OHL-W v2")
+		(comment 1 "https://github.com/Elemecca/lgp21-mini")
 	)
 	(rectangle
