File: boards/pq-register/Q1.kicad_sch (KiCad schematic)
At the start: 92 parts, among them Q57 MMBT5401, Q58 MMBT5401, Q59 MMBT5401, Q60 MMBT5401, Q61 MMBT5401, Q62 MMBT5401, Q64 MMBT5401, Q66 MMBT5401, Q67 MMBT5401, Q68 MMBT5401, Q69 MMBT5401, Q70 MMBT5401, Q71 MMBT5401, Q72 MMBT5401

Commit message: Route resistors in the second column.
Parts:
- R350, R362: value 2k4 ¼W -> 2k4; footprint Resistor_SMD:R_0603_1608Metric -> Resistor_SMD:R_0402_1005Metric
Changed lines of the file:
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@@
 			)
 		)
-		(property "Value" "2k4 ¼W"
+		(property "Value" "2k4"
 			(at 241.3 60.198 90)
 			(show_name no)
@@
 			)
 		)
-		(property "Footprint" "Resistor_SMD:R_0603_1608Metric"
+		(property "Footprint" "Resistor_SMD:R_0402_1005Metric"
 			(at 241.554 63.246 90)
 			(hide yes)
@@
 			)
 		)
-		(property "Value" "2k4 ¼W"
+		(property "Value" "2k4"
 			(at 193.04 60.198 90)
 			(show_name no)
@@
 			)
 		)
-		(property "Footprint" "Resistor_SMD:R_0603_1608Metric"
+		(property "Footprint" "Resistor_SMD:R_0402_1005Metric"
 			(at 193.294 63.246 90)
 			(hide yes)

Commit message: Route passives in the rightmost column.
Parts:
- R901: renamed from R447; now fitted
- R902: renamed from R506; now fitted
Changed lines of the file:
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@@
 		(on_board yes)
 		(in_pos_files yes)
-		(dnp yes)
-		(property "Reference" "R506"
+		(dnp no)
+		(property "Reference" "R902"
 			(at 142.24 147.574 90)
 			(show_name no)
@@
 			(project "pq-register"
 				(path "/d5da316c-1ec9-4d99-8330-1c4a3f6c3ba4/f5a3ee66-2980-4c4b-9db6-5c1c30d0ba91"
-					(reference "R506")
+					(reference "R902")
 					(unit 1)
 				)
@@
 		(on_board yes)
 		(in_pos_files yes)
-		(dnp yes)
-		(property "Reference" "R447"
+		(dnp no)
+		(property "Reference" "R901"
 			(at 90.17 183.134 90)
 			(show_name no)
@@
 			(project "pq-register"
 				(path "/d5da316c-1ec9-4d99-8330-1c4a3f6c3ba4/f5a3ee66-2980-4c4b-9db6-5c1c30d0ba91"
-					(reference "R447")
+					(reference "R901")
 					(unit 1)
 				)

Commit message: Assorted cleanup and silkscreen.
Parts:
- renumbered R901 to R903, R902 to R904
Changed lines of the file:
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@@
 		(in_pos_files yes)
 		(dnp no)
-		(property "Reference" "R902"
+		(property "Reference" "R904"
 			(at 142.24 147.574 90)
 			(show_name no)
@@
 			(project "pq-register"
 				(path "/d5da316c-1ec9-4d99-8330-1c4a3f6c3ba4/f5a3ee66-2980-4c4b-9db6-5c1c30d0ba91"
-					(reference "R902")
+					(reference "R904")
 					(unit 1)
 				)
@@
 		(in_pos_files yes)
 		(dnp no)
-		(property "Reference" "R901"
+		(property "Reference" "R903"
 			(at 90.17 183.134 90)
 			(show_name no)
@@
 			(project "pq-register"
 				(path "/d5da316c-1ec9-4d99-8330-1c4a3f6c3ba4/f5a3ee66-2980-4c4b-9db6-5c1c30d0ba91"
-					(reference "R901")
+					(reference "R903")
 					(unit 1)
 				)

Commit message: Add script to export production files.
Parts:
- C27, C30: BOM Value (none) -> 120pF
- C28, C29: BOM Value (none) -> 680pF
- CR13, CR14: value 1N5819WS -> 1N4148WS; BOM Value (none) -> 1N4148WS; LCSC (none) -> C2128
- Q57, Q58, Q59, Q60, Q61, Q62, Q64, Q66, Q67, Q68, Q69, Q70, Q71, Q72: BOM Value (none) -> MMBT5401; LCSC (none) -> C8326
- R268, R270, R272, R274, R276, R278, R283, R287, R289, R291, R293, R295: BOM Value (none) -> 56kΩ
- R269, R271, R273, R275, R277, R279, R284, R288, R290, R292, R294, R296: BOM Value (none) -> 2kΩ 500mW
- R297, R298: BOM Value (none) -> 33kΩ
- R310, R311, R312, R313, R314, R315, R316, R317, R318, R319, R320, R321, R322, R323, R324, R325, R326, R327, R328, R329, R330, R331, R332, R333, R340, R341, R342, R351, R352, R353, R354, R355, R356, R357, R358, R359, R360, R361, R903, R904: BOM Value (none) -> 15kΩ
- R350, R362: BOM Value (none) -> 2.4kΩ
- R363, R364: BOM Value (none) -> 2.4kΩ 250mW
- R382, R502: BOM Value (none) -> 300Ω 3W
