File: boards/card-template/card-template.kicad_pcb (KiCad board)
At the start: 2 copper layers, 114.3 x 118.7 mm, 6 parts, among them P1 Card Edge

Commit message: Add script to export production files.
Connections:
- P1 pad A10: ~{rl} -> unconnected-(P1-~{r1}-PadA10)
- P1 pad A11: ~{P1d} -> unconnected-(P1-~{P1d}-PadA11)
- P1 pad A12: ~{P2c} -> unconnected-(P1-~{P2c}-PadA12)
- P1 pad A13: ~{P2d} -> unconnected-(P1-~{P2d}-PadA13)
- P1 pad A14: ~{P3c} -> unconnected-(P1-~{P3c}-PadA14)
- P1 pad A15: ~{P3d} -> unconnected-(P1-~{P3d}-PadA15)
- P1 pad A16: ~{P4c} -> unconnected-(P1-~{P4c}-PadA16)
- P1 pad A17: ~{P4d} -> unconnected-(P1-~{P4d}-PadA17)
- P1 pad A19: V -> unconnected-(P1-V-PadA19)
- P1 pad A20: ~{P5c} -> unconnected-(P1-~{P5c}-PadA20)
- P1 pad A21: P5a -> unconnected-(P1-P5a-PadA21)
- P1 pad A22: ~{V} -> unconnected-(P1-~{V}-PadA22)
- P1 pad A23: ~{P5d} -> unconnected-(P1-~{P5d}-PadA23)
- P1 pad A24: ~{P6c} -> unconnected-(P1-~{P6c}-PadA24)
- P1 pad A25: P6a -> unconnected-(P1-P6a-PadA25)
- P1 pad A26: ~{P6d} -> unconnected-(P1-~{P6d}-PadA26)
- P1 pad A27: S2 -> unconnected-(P1-S2-PadA27)
- P1 pad A28: ia -> unconnected-(P1-ia-PadA28)
- P1 pad A29: T3 -> unconnected-(P1-T3-PadA29)
- P1 pad A3: ~{P1} -> unconnected-(P1-~{P1}-PadA3)
- P1 pad A30: S3 -> unconnected-(P1-S3-PadA30)
- P1 pad A31: ~{Tb2} -> unconnected-(P1-~{Tb2}-PadA31)
- P1 pad A32: ~{Tb1} -> unconnected-(P1-~{Tb1}-PadA32)
- P1 pad A33: ~{ic} -> unconnected-(P1-~{ic}-PadA33)
- P1 pad A34: ~{Tb3} -> unconnected-(P1-~{Tb3}-PadA34)
- P1 pad A35: ~{Tb4} -> unconnected-(P1-~{Tb4}-PadA35)
- P1 pad A36: Tc -> unconnected-(P1-Tc-PadA36)
- P1 pad A38: Q1b -> unconnected-(P1-Q1b-PadA38)
- P1 pad A39: ~{Q1d} -> unconnected-(P1-~{Q1d}-PadA39)
- P1 pad A40: ~{Q2a} -> unconnected-(P1-Q2a-PadA40)
- P1 pad A41: ~{O1} -> unconnected-(P1-~{O1}-PadA41)
- P1 pad A43: ~{Q2c} -> unconnected-(P1-~{Q2c}-PadA43)
- P1 pad A44: O1 -> unconnected-(P1-O1-PadA44)
- P1 pad A45: ~{Q2d} -> unconnected-(P1-~{Q2d}-PadA45)
- P1 pad A46: ~{S1} -> unconnected-(P1-~{S1}-PadA46)
- P1 pad A47: ~{H} -> unconnected-(P1-~{H}-PadA47)
- P1 pad A48: ~{P2} -> unconnected-(P1-~{P2}-PadA48)
- P1 pad A49: ~{P3} -> unconnected-(P1-~{P3}-PadA49)
- P1 pad A5: P1 -> unconnected-(P1-P1-PadA5)
- P1 pad A52: ~{P4} -> unconnected-(P1-~{P4}-PadA52)
- P1 pad A53: ~{bq} -> unconnected-(P1-~{bq}-PadA53)
- P1 pad A54: ~{S2} -> unconnected-(P1-~{S2}-PadA54)
- P1 pad A55: ~{P5} -> unconnected-(P1-~{P5}-PadA55)
- P1 pad A57: Q1 -> unconnected-(P1-Q1-PadA57)
- P1 pad A58: Q3 -> unconnected-(P1-Q3-PadA58)
- P1 pad A59: ~{Q3} -> unconnected-(P1-~{Q3}-PadA59)
- P1 pad A6: G -> unconnected-(P1-G-PadA6)
- P1 pad A7: ~{G} -> unconnected-(P1-~{G}-PadA7)
- P1 pad A8: rl -> unconnected-(P1-r1-PadA8)
- P1 pad A9: ~{P1c} -> unconnected-(P1-~{P1c}-PadA9)
- P1 pad B1: P1b -> unconnected-(P1-P1b-PadB1)
- P1 pad B13: ~{A} -> unconnected-(P1-~{A}-PadB13)
- P1 pad B14: A* -> unconnected-(P1-A*-PadB14)
- P1 pad B15: ~{A*} -> unconnected-(P1-~{A*}-PadB15)
- P1 pad B16: A -> unconnected-(P1-A-PadB16)
- P1 pad B19: P5 -> unconnected-(P1-P5-PadB19)
- P1 pad B2: H -> unconnected-(P1-H-PadB2)
- P1 pad B25: F -> unconnected-(P1-F-PadB25)
- P1 pad B26: ~{F} -> unconnected-(P1-~{F}-PadB26)
- P1 pad B27: CP -> unconnected-(P1-CP-PadB27)
- P1 pad B28: P6 -> unconnected-(P1-P6-PadB28)
- P1 pad B29: P2 -> unconnected-(P1-P2-PadB29)
- P1 pad B30: bs -> unconnected-(P1-bs-PadB30)
- P1 pad B31: P4 -> unconnected-(P1-P4-PadB31)
- P1 pad B32: P3 -> unconnected-(P1-P3-PadB32)
- P1 pad B34: K -> unconnected-(P1-K-PadB34)
- P1 pad B37: ~{C} -> unconnected-(P1-~{C}-PadB37)
- P1 pad B39: B1 -> unconnected-(P1-Bl-PadB39)
- P1 pad B40: Faf -> unconnected-(P1-Faf-PadB40)
- P1 pad B41: ~{R} -> unconnected-(P1-~{R}-PadB41)
- P1 pad B42: R -> unconnected-(P1-R-PadB42)
- P1 pad B43: Q4 -> unconnected-(P1-Q4-PadB43)
- P1 pad B44: Q2 -> unconnected-(P1-Q2-PadB44)
- P1 pad B45: ~{P6} -> unconnected-(P1-~{P6}-PadB45)
- P1 pad B46: ~{H'} -> unconnected-(P1-~{H'}-PadB46)
- P1 pad B47: α9 -> unconnected-(P1-α9-PadB47)
- P1 pad B48: ~{Faf} -> unconnected-(P1-~{Faf}-PadB48)
- P1 pad B49: ~{To} -> unconnected-(P1-~{To}-PadB49)
- P1 pad B60: ~{Q2} -> unconnected-(P1-~{Q2}-PadB60)
- P1 pad B61: ~{Q1} -> unconnected-(P1-~{Q1}-PadB61)
- P1 pad B62: ~{Q4} -> unconnected-(P1-~{Q4}-PadB62)
