File: boards/phase-control/F-flop.kicad_sch (KiCad schematic)
At the start: 86 parts, among them Q1 MMBT5401, Q10 MMBT5401, Q11 MMBT5401, Q12 MMBT5401, Q2 MMBT5401, Q3 MMBT5401, Q4 MMBT5401, Q5 MMBT5401, Q6 MMBT5401, Q7 MMBT5401, Q8 MMBT5401, Q9 MMBT5401

Commit message: Start the Phase Control board.
Parts:
- Q1, Q10, Q11, Q12, Q2, Q3, Q4, Q5, Q6, Q7, Q8, Q9: symbol Transistor_BJT:Q_PNP_EBC -> Transistor_BJT:Q_PNP_BEC
Connections:
- net GND: now also Q1.2 (E), Q10.2 (E), Q2.2 (E), Q3.2 (E), Q4.2 (E), Q5.2 (E), Q6.2 (E), Q7.2 (E), Q8.2 (E), Q9.2 (E); no longer Q1.1 (E), Q10.1 (E), Q2.1 (E), Q3.1 (E), Q4.1 (E), Q5.1 (E), Q6.1 (E), Q7.1 (E), Q8.1 (E), Q9.1 (E)
- net at R43.2, R44.2, R45.2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: now also Q3.1 (B); no longer Q3.2 (B)
- net at C1.2, Q10.3 (C), R385.2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: now also Q11.1 (B); no longer Q11.2 (B)
- net at C4.1, CR2.1 (K), R18.1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: now also Q10.1 (B); no longer Q10.2 (B)
- net at C4.2, Q9.3 (C), R21.2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: now also Q12.1 (B); no longer Q12.2 (B)
- net at R1.1, R33.2, R34.2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: now also Q1.1 (B); no longer Q1.2 (B)
- net at R51.2, R52.2, R53.2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: now also Q5.1 (B); no longer Q5.2 (B)
- net at C1.1, CR1.1 (K), R17.1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: now also Q9.1 (B); no longer Q9.2 (B)
- net at CR5.1 (K): now also Q11.2 (E); no longer Q11.1 (E)
- net at R15.1, R56.2, R62.2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: now also Q8.1 (B); no longer Q8.2 (B)
- net at R13.1, R63.2, R64.2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: now also Q7.1 (B); no longer Q7.2 (B)
- net at R11.1, R57.2, R58.2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: now also Q6.1 (B); no longer Q6.2 (B)
- net at R3.1, R40.2, R41.2: now also Q2.1 (B); no longer Q2.2 (B)
- net at CR8.1 (K): now also Q12.2 (E); no longer Q12.1 (E)
- net at R39.2, R42.2, R48.2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: now also Q4.1 (B); no longer Q4.2 (B)
Changed lines of the file:
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@@
 	)
 	(symbol
-		(lib_id "Transistor_BJT:Q_PNP_EBC")
+		(lib_id "Transistor_BJT:Q_PNP_BEC")
 		(at 52.07 107.95 0)
 		(unit 1)
@@
 			)
 		)
-		(property "Description" "Germanium PNP Transistor"
+		(property "Description" "PNP BJT"
 			(at 52.07 107.95 0)
 			(hide yes)
@@
 			)
 		)
-		(property "Sim.Pins" "1=E 2=B 3=C"
+		(property "Sim.Pins" "1=B 2=E 3=C"
 			(at 52.07 107.95 0)
 			(hide yes)
@@
 	)
 	(symbol
-		(lib_id "Transistor_BJT:Q_PNP_EBC")
+		(lib_id "Transistor_BJT:Q_PNP_BEC")
 		(at 237.49 49.53 0)
 		(unit 1)
@@
 			)
 		)
-		(property "Description" "Germanium PNP Transistor"
+		(property "Description" "PNP BJT"
 			(at 237.49 49.53 0)
 			(hide yes)
@@
 			)
 		)
-		(property "Sim.Pins" "1=E 2=B 3=C"
+		(property "Sim.Pins" "1=B 2=E 3=C"
 			(at 237.49 49.53 0)
 			(hide yes)
@@
 	)
 	(symbol
-		(lib_id "Transistor_BJT:Q_PNP_EBC")
+		(lib_id "Transistor_BJT:Q_PNP_BEC")
 		(at 113.03 184.15 0)
 		(unit 1)
@@
 			)
 		)
-		(property "Description" "Germanium PNP Transistor"
+		(property "Description" "PNP BJT"
 			(at 113.03 184.15 0)
 			(hide yes)
@@
 			)
 		)
-		(property "Sim.Pins" "1=E 2=B 3=C"
+		(property "Sim.Pins" "1=B 2=E 3=C"
 			(at 113.03 184.15 0)
 			(hide yes)
@@
 	)
 	(symbol
-		(lib_id "Transistor_BJT:Q_PNP_EBC")
+		(lib_id "Transistor_BJT:Q_PNP_BEC")
 		(at 52.07 36.83 0)
 		(unit 1)
@@
 			)
 		)
-		(property "Description" "Germanium PNP Transistor"
+		(property "Description" "PNP BJT"
 			(at 52.07 36.83 0)
 			(hide yes)
@@
 			)
 		)
-		(property "Sim.Pins" "1=E 2=B 3=C"
+		(property "Sim.Pins" "1=B 2=E 3=C"
 			(at 52.07 36.83 0)
 			(hide yes)
@@
 	)
 	(symbol
-		(lib_id "Transistor_BJT:Q_PNP_EBC")
+		(lib_id "Transistor_BJT:Q_PNP_BEC")
 		(at 160.02 144.78 0)
 		(unit 1)
@@
 			)
 		)
-		(property "Description" "Germanium PNP Transistor"
+		(property "Description" "PNP BJT"
 			(at 160.02 144.78 0)
 			(hide yes)
@@
 			)
 		)
-		(property "Sim.Pins" "1=E 2=B 3=C"
+		(property "Sim.Pins" "1=B 2=E 3=C"
 			(at 160.02 144.78 0)
 			(hide yes)
@@
 	)
 	(symbol
-		(lib_id "Transistor_BJT:Q_PNP_EBC")
+		(lib_id "Transistor_BJT:Q_PNP_BEC")
 		(at 50.8 184.15 0)
 		(unit 1)
@@
 			)
 		)
-		(property "Description" "Germanium PNP Transistor"
+		(property "Description" "PNP BJT"
 			(at 50.8 184.15 0)
 			(hide yes)
@@
 			)
 		)
-		(property "Sim.Pins" "1=E 2=B 3=C"
+		(property "Sim.Pins" "1=B 2=E 3=C"
 			(at 50.8 184.15 0)
 			(hide yes)
@@
 	)
 	(symbol
-		(lib_id "Transistor_BJT:Q_PNP_EBC")
+		(lib_id "Transistor_BJT:Q_PNP_BEC")
 		(at 160.02 76.2 0)
 		(mirror y)
@@
 			)
 		)
-		(property "Description" "Germanium PNP Transistor"
+		(property "Description" "PNP BJT"
 			(at 160.02 76.2 0)
 			(hide yes)
@@
 			)
 		)
-		(property "Sim.Pins" "1=E 2=B 3=C"
+		(property "Sim.Pins" "1=B 2=E 3=C"
 			(at 160.02 76.2 0)
 			(hide yes)
@@
 	)
 	(symbol
-		(lib_id "Transistor_BJT:Q_PNP_EBC")
+		(lib_id "Transistor_BJT:Q_PNP_BEC")
 		(at 128.27 99.06 0)
 		(unit 1)
@@
 			)
 		)
-		(property "Description" "Germanium PNP Transistor"
+		(property "Description" "PNP BJT"
 			(at 128.27 99.06 0)
 			(hide yes)
@@
 			)
 		)
-		(property "Sim.Pins" "1=E 2=B 3=C"
+		(property "Sim.Pins" "1=B 2=E 3=C"
 			(at 128.27 99.06 0)
 			(hide yes)
@@
 	)
 	(symbol
-		(lib_id "Transistor_BJT:Q_PNP_EBC")
+		(lib_id "Transistor_BJT:Q_PNP_BEC")
 		(at 237.49 95.25 0)
 		(unit 1)
@@
 			)
 		)
-		(property "Description" "Germanium PNP Transistor"
+		(property "Description" "PNP BJT"
 			(at 237.49 95.25 0)
 			(hide yes)
@@
 			)
 		)
-		(property "Sim.Pins" "1=E 2=B 3=C"
+		(property "Sim.Pins" "1=B 2=E 3=C"
 			(at 237.49 95.25 0)
 			(hide yes)
@@
 	)
 	(symbol
-		(lib_id "Transistor_BJT:Q_PNP_EBC")
+		(lib_id "Transistor_BJT:Q_PNP_BEC")
 		(at 52.07 72.39 0)
 		(unit 1)
@@
 			)
 		)
-		(property "Description" "Germanium PNP Transistor"
+		(property "Description" "PNP BJT"
 			(at 52.07 72.39 0)
 			(hide yes)
@@
 			)
 		)
-		(property "Sim.Pins" "1=E 2=B 3=C"
+		(property "Sim.Pins" "1=B 2=E 3=C"
 			(at 52.07 72.39 0)
 			(hide yes)
@@
 	)
 	(symbol
-		(lib_id "Transistor_BJT:Q_PNP_EBC")
+		(lib_id "Transistor_BJT:Q_PNP_BEC")
 		(at 52.07 148.59 0)
 		(unit 1)
@@
 			)
 		)
-		(property "Description" "Germanium PNP Transistor"
+		(property "Description" "PNP BJT"
 			(at 52.07 148.59 0)
 			(hide yes)
@@
 			)
 		)
-		(property "Sim.Pins" "1=E 2=B 3=C"
+		(property "Sim.Pins" "1=B 2=E 3=C"
 			(at 52.07 148.59 0)
 			(hide yes)
@@
 	)
 	(symbol
-		(lib_id "Transistor_BJT:Q_PNP_EBC")
+		(lib_id "Transistor_BJT:Q_PNP_BEC")
 		(at 205.74 76.2 0)
 		(unit 1)
@@
 			)
 		)
-		(property "Description" "Germanium PNP Transistor"
+		(property "Description" "PNP BJT"
 			(at 205.74 76.2 0)
 			(hide yes)
@@
 			)
 		)
-		(property "Sim.Pins" "1=E 2=B 3=C"
+		(property "Sim.Pins" "1=B 2=E 3=C"
 			(at 205.74 76.2 0)
 			(hide yes)
@@
 			"296c9191-3a04-4018-adbe-9fc2ff6d5d85" "2a68b6ea-1537-4dfc-a559-75fc21579301"
 			"3155e888-fee3-4f59-ae21-a8450436d383" "33277c7b-9cc9-4254-83bd-9bc477c0bc0d"
-			"33fb5f43-4ed0-49e1-8840-16713d85b204" "3a270356-1cf0-40e7-9c4c-8f8e80f3de0f"
-			"3cdb720d-84e6-4e7b-9dbb-1cf6bc12e4c3" "41d6d1a4-e4c2-4e95-bbad-e65b77a7693e"
-			"464b3f71-0413-4f79-9ca7-6b10ccbd1ec2" "52722a16-757b-472b-8581-0d11b3ab7d6e"
-			"52cc9cf1-92a9-437b-b441-f07ecdc6467c" "53e1f588-310c-41d1-8dee-be2299699407"
-			"54b3538b-23a3-4262-ab9a-63bbb7655327" "564b8596-f6fd-44d7-a820-f923c5e28f64"
-			"60f778d9-b976-4f8e-8048-0e301e3a7106" "63ca2f4d-a5db-428b-8618-b0b00964f39c"
+			"33fb5f43-4ed0-49e1-8840-16713d85b204" "3cdb720d-84e6-4e7b-9dbb-1cf6bc12e4c3"
+			"41d6d1a4-e4c2-4e95-bbad-e65b77a7693e" "464b3f71-0413-4f79-9ca7-6b10ccbd1ec2"
+			"52722a16-757b-472b-8581-0d11b3ab7d6e" "52cc9cf1-92a9-437b-b441-f07ecdc6467c"
+			"53e1f588-310c-41d1-8dee-be2299699407" "54b3538b-23a3-4262-ab9a-63bbb7655327"
+			"564b8596-f6fd-44d7-a820-f923c5e28f64" "60f778d9-b976-4f8e-8048-0e301e3a7106"
 			"672a20fe-e0be-4626-9476-3e58685c3999" "6b6ddc89-6359-4478-bddb-63de80467452"
 			"6e11d458-4e77-4517-b05e-3486af400c3c" "6e15cffc-e068-4390-b115-4d3ebfd86938"

Commit message: Add script to export production files.
Parts:
- C1, C4: BOM Value (none) -> 120pF
- C2, C3: BOM Value (none) -> 680pF
- CR1, CR2, CR3, CR4, CR5, CR6, CR7, CR8: value 1N5819WS -> 1N4148WS; BOM Value (none) -> 1N4148WS; LCSC (none) -> C2128
- Q1, Q10, Q11, Q12, Q2, Q3, Q4, Q5, Q6, Q7, Q8, Q9: BOM Value (none) -> MMBT5401; LCSC (none) -> C8326
- R1, R11, R13, R15, R19, R20, R3, R5, R7, R9: BOM Value (none) -> 56kΩ
- R10, R12, R14, R16, R2, R4, R6, R8: BOM Value (none) -> 2kΩ 500mW
- R17, R18: BOM Value (none) -> 33kΩ
- R21, R385: BOM Value (none) -> 300Ω 3W
- R33, R34, R35, R36, R37, R38, R39, R40, R41, R42, R43, R44, R45, R46, R47, R48, R49, R51, R52, R53, R54, R55, R56, R57, R58, R59, R60, R61, R62, R63, R64, R65, R66, R67, R68, R69: BOM Value (none) -> 15kΩ
- R50, R70: BOM Value (none) -> 2.4kΩ
- R71, R72: BOM Value (none) -> 2.4kΩ 250mW

Commit message: Rough layout for Phase Control.
Connections:
- net ~{F_{S}}: now reaches C1.2, Q10.3 (C), Q11.1 (B), R385.2, R71.1
- net F_{S}: now reaches C4.2, Q12.1 (B), Q9.3 (C), R21.2, R72.2
Changed lines of the file:
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@@
+		)
+	)
+	(label "~{F_{S}}"
+		(at 143.51 49.53 0)
+		(effects
+			(font
+				(size 1.27 1.27)
+			)
+			(justify left bottom)
+		)
+	)
+	(label "F_{S}"
+		(at 223.52 68.58 180)
+		(effects
+			(font
+				(size 1.27 1.27)
+			)
+			(justify right bottom)
 		)
 	)
