File: boards/phase-control/G-flop.kicad_sch (KiCad schematic)
At the start: 136 parts, among them Q13 MMBT5401, Q14 MMBT5401, Q15 MMBT5401, Q16 MMBT5401, Q17 MMBT5401, Q18 MMBT5401, Q19 MMBT5401, Q20 MMBT5401, Q21 MMBT5401, Q22 MMBT5401, Q23 MMBT5401, Q24 MMBT5401, Q25 MMBT5401, Q26 MMBT5401, Q27 MMBT5401

Commit message: Start the Phase Control board.
Parts:
- Q13, Q14, Q15, Q16, Q17, Q18, Q19, Q20, Q21, Q22, Q23, Q24, Q25, Q26, Q27: symbol Transistor_BJT:Q_PNP_EBC -> Transistor_BJT:Q_PNP_BEC
Connections:
- net GND: now also Q13.2 (E), Q14.2 (E), Q15.2 (E), Q16.2 (E), Q17.2 (E), Q18.2 (E), Q19.2 (E), Q20.2 (E), Q21.2 (E), Q22.2 (E), Q23.2 (E), Q24.2 (E), Q25.2 (E); no longer Q13.1 (E), Q14.1 (E), Q15.1 (E), Q16.1 (E), Q17.1 (E), Q18.1 (E), Q19.1 (E), Q20.1 (E), Q21.1 (E), Q22.1 (E), Q23.1 (E), Q24.1 (E), Q25.1 (E)
- net at R101.2, R110.2, R118.2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: now also Q19.1 (B); no longer Q19.2 (B)
- net at R102.2, R103.2, R104.2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: now also Q16.1 (B); no longer Q16.2 (B)
- net at C5.1, CR9.1 (K), R146.2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: now also Q24.1 (B); no longer Q24.2 (B)
- net at R24.1, R84.2, R85.2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: now also Q14.1 (B); no longer Q14.2 (B)
- net at R22.1, R73.2, R74.2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: now also Q13.1 (B); no longer Q13.2 (B)
- net at R111.2, R112.2, R113.2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: now also Q17.1 (B); no longer Q17.2 (B)
- net at R100.2, R26.1, R94.2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: now also Q15.1 (B); no longer Q15.2 (B)
- net at R133.2, R137.2, R143.2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: now also Q23.1 (B); no longer Q23.2 (B)
- net at R138.2, R139.2, R140.2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: now also Q22.1 (B); no longer Q22.2 (B)
- net at C5.2, Q25.3 (C), R146.1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: now also Q26.1 (B); no longer Q26.2 (B)
- net at R134.2, R135.2, R136.2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: now also Q21.1 (B); no longer Q21.2 (B)
- net at R129.2, R130.2, R131.2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: now also Q20.1 (B); no longer Q20.2 (B)
- net at R119.2, R120.2, R121.2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: now also Q18.1 (B); no longer Q18.2 (B)
- net at C8.1, CR10.1 (K), R147.1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: now also Q25.1 (B); no longer Q25.2 (B)
- net at C8.2, Q24.3 (C), R147.2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: now also Q27.1 (B); no longer Q27.2 (B)
- net at CR16.1 (K): now also Q27.2 (E); no longer Q27.1 (E)
- net at CR13.1 (K): now also Q26.2 (E); no longer Q26.1 (E)
Changed lines of the file:
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@@
 	)
 	(symbol
-		(lib_id "Transistor_BJT:Q_PNP_EBC")
+		(lib_id "Transistor_BJT:Q_PNP_BEC")
 		(at 180.34 147.32 0)
 		(unit 1)
@@
 			)
 		)
-		(property "Description" "Germanium PNP Transistor"
+		(property "Description" "PNP BJT"
 			(at 180.34 147.32 0)
 			(hide yes)
@@
 			)
 		)
-		(property "Sim.Pins" "1=E 2=B 3=C"
+		(property "Sim.Pins" "1=B 2=E 3=C"
 			(at 180.34 147.32 0)
 			(hide yes)
@@
 	)
 	(symbol
-		(lib_id "Transistor_BJT:Q_PNP_EBC")
+		(lib_id "Transistor_BJT:Q_PNP_BEC")
 		(at 238.76 73.66 0)
 		(unit 1)
@@
 			)
 		)
-		(property "Description" "Germanium PNP Transistor"
+		(property "Description" "PNP BJT"
 			(at 238.76 73.66 0)
 			(hide yes)
@@
 			)
 		)
-		(property "Sim.Pins" "1=E 2=B 3=C"
+		(property "Sim.Pins" "1=B 2=E 3=C"
 			(at 238.76 73.66 0)
 			(hide yes)
@@
 	)
 	(symbol
-		(lib_id "Transistor_BJT:Q_PNP_EBC")
+		(lib_id "Transistor_BJT:Q_PNP_BEC")
 		(at 238.76 27.94 0)
 		(unit 1)
@@
 			)
 		)
-		(property "Description" "Germanium PNP Transistor"
+		(property "Description" "PNP BJT"
 			(at 238.76 27.94 0)
 			(hide yes)
@@
 			)
 		)
-		(property "Sim.Pins" "1=E 2=B 3=C"
+		(property "Sim.Pins" "1=B 2=E 3=C"
 			(at 238.76 27.94 0)
 			(hide yes)
@@
 	)
 	(symbol
-		(lib_id "Transistor_BJT:Q_PNP_EBC")
+		(lib_id "Transistor_BJT:Q_PNP_BEC")
 		(at 53.34 140.97 0)
 		(unit 1)
@@
 			)
 		)
-		(property "Description" "Germanium PNP Transistor"
+		(property "Description" "PNP BJT"
 			(at 53.34 140.97 0)
 			(hide yes)
@@
 			)
 		)
-		(property "Sim.Pins" "1=E 2=B 3=C"
+		(property "Sim.Pins" "1=B 2=E 3=C"
 			(at 53.34 140.97 0)
 			(hide yes)
@@
 	)
 	(symbol
-		(lib_id "Transistor_BJT:Q_PNP_EBC")
+		(lib_id "Transistor_BJT:Q_PNP_BEC")
 		(at 161.29 54.61 0)
 		(mirror y)
@@
 			)
 		)
-		(property "Description" "Germanium PNP Transistor"
+		(property "Description" "PNP BJT"
 			(at 161.29 54.61 0)
 			(hide yes)
@@
 			)
 		)
-		(property "Sim.Pins" "1=E 2=B 3=C"
+		(property "Sim.Pins" "1=B 2=E 3=C"
 			(at 161.29 54.61 0)
 			(hide yes)
@@
 	)
 	(symbol
-		(lib_id "Transistor_BJT:Q_PNP_EBC")
+		(lib_id "Transistor_BJT:Q_PNP_BEC")
 		(at 238.76 143.51 0)
 		(unit 1)
@@
 			)
 		)
-		(property "Description" "Germanium PNP Transistor"
+		(property "Description" "PNP BJT"
 			(at 238.76 143.51 0)
 			(hide yes)
@@
 			)
 		)
-		(property "Sim.Pins" "1=E 2=B 3=C"
+		(property "Sim.Pins" "1=B 2=E 3=C"
 			(at 238.76 143.51 0)
 			(hide yes)
@@
 	)
 	(symbol
-		(lib_id "Transistor_BJT:Q_PNP_EBC")
+		(lib_id "Transistor_BJT:Q_PNP_BEC")
 		(at 207.01 54.61 0)
 		(unit 1)
@@
 			)
 		)
-		(property "Description" "Germanium PNP Transistor"
+		(property "Description" "PNP BJT"
 			(at 207.01 54.61 0)
 			(hide yes)
@@
 			)
 		)
-		(property "Sim.Pins" "1=E 2=B 3=C"
+		(property "Sim.Pins" "1=B 2=E 3=C"
 			(at 207.01 54.61 0)
 			(hide yes)
@@
 	)
 	(symbol
-		(lib_id "Transistor_BJT:Q_PNP_EBC")
+		(lib_id "Transistor_BJT:Q_PNP_BEC")
 		(at 53.34 96.52 0)
 		(unit 1)
@@
 			)
 		)
-		(property "Description" "Germanium PNP Transistor"
+		(property "Description" "PNP BJT"
 			(at 53.34 96.52 0)
 			(hide yes)
@@
 			)
 		)
-		(property "Sim.Pins" "1=E 2=B 3=C"
+		(property "Sim.Pins" "1=B 2=E 3=C"
 			(at 53.34 96.52 0)
 			(hide yes)
@@
 	)
 	(symbol
-		(lib_id "Transistor_BJT:Q_PNP_EBC")
+		(lib_id "Transistor_BJT:Q_PNP_BEC")
 		(at 53.34 180.34 0)
 		(unit 1)
@@
 			)
 		)
-		(property "Description" "Germanium PNP Transistor"
+		(property "Description" "PNP BJT"
 			(at 53.34 180.34 0)
 			(hide yes)
@@
 			)
 		)
-		(property "Sim.Pins" "1=E 2=B 3=C"
+		(property "Sim.Pins" "1=B 2=E 3=C"
 			(at 53.34 180.34 0)
 			(hide yes)
@@
 	)
 	(symbol
-		(lib_id "Transistor_BJT:Q_PNP_EBC")
+		(lib_id "Transistor_BJT:Q_PNP_BEC")
 		(at 180.34 182.88 0)
 		(unit 1)
@@
 			)
 		)
-		(property "Description" "Germanium PNP Transistor"
+		(property "Description" "PNP BJT"
 			(at 180.34 182.88 0)
 			(hide yes)
@@
 			)
 		)
-		(property "Sim.Pins" "1=E 2=B 3=C"
+		(property "Sim.Pins" "1=B 2=E 3=C"
 			(at 180.34 182.88 0)
 			(hide yes)
@@
 	)
 	(symbol
-		(lib_id "Transistor_BJT:Q_PNP_EBC")
+		(lib_id "Transistor_BJT:Q_PNP_BEC")
 		(at 135.89 77.47 0)
 		(unit 1)
@@
 			)
 		)
-		(property "Description" "Germanium PNP Transistor"
+		(property "Description" "PNP BJT"
 			(at 135.89 77.47 0)
 			(hide yes)
@@
 			)
 		)
-		(property "Sim.Pins" "1=E 2=B 3=C"
+		(property "Sim.Pins" "1=B 2=E 3=C"
 			(at 135.89 77.47 0)
 			(hide yes)
@@
 	)
 	(symbol
-		(lib_id "Transistor_BJT:Q_PNP_EBC")
+		(lib_id "Transistor_BJT:Q_PNP_BEC")
 		(at 116.84 137.16 0)
 		(unit 1)
@@
 			)
 		)
-		(property "Description" "Germanium PNP Transistor"
+		(property "Description" "PNP BJT"
 			(at 116.84 137.16 0)
 			(hide yes)
@@
 			)
 		)
-		(property "Sim.Pins" "1=E 2=B 3=C"
+		(property "Sim.Pins" "1=B 2=E 3=C"
 			(at 116.84 137.16 0)
 			(hide yes)
@@
 	)
 	(symbol
-		(lib_id "Transistor_BJT:Q_PNP_EBC")
+		(lib_id "Transistor_BJT:Q_PNP_BEC")
 		(at 116.84 176.53 0)
 		(unit 1)
@@
 			)
 		)
-		(property "Description" "Germanium PNP Transistor"
+		(property "Description" "PNP BJT"
 			(at 116.84 176.53 0)
 			(hide yes)
@@
 			)
 		)
-		(property "Sim.Pins" "1=E 2=B 3=C"
+		(property "Sim.Pins" "1=B 2=E 3=C"
 			(at 116.84 176.53 0)
 			(hide yes)
@@
 	)
 	(symbol
-		(lib_id "Transistor_BJT:Q_PNP_EBC")
+		(lib_id "Transistor_BJT:Q_PNP_BEC")
 		(at 180.34 111.76 0)
 		(unit 1)
@@
 			)
 		)
-		(property "Description" "Germanium PNP Transistor"
+		(property "Description" "PNP BJT"
 			(at 180.34 111.76 0)
 			(hide yes)
@@
 			)
 		)
-		(property "Sim.Pins" "1=E 2=B 3=C"
+		(property "Sim.Pins" "1=B 2=E 3=C"
 			(at 180.34 111.76 0)
 			(hide yes)
@@
 	)
 	(symbol
-		(lib_id "Transistor_BJT:Q_PNP_EBC")
+		(lib_id "Transistor_BJT:Q_PNP_BEC")
 		(at 53.34 41.91 0)
 		(unit 1)
@@
 			)
 		)
-		(property "Description" "Germanium PNP Transistor"
+		(property "Description" "PNP BJT"
 			(at 53.34 41.91 0)
 			(hide yes)
@@
 			)
 		)
-		(property "Sim.Pins" "1=E 2=B 3=C"
+		(property "Sim.Pins" "1=B 2=E 3=C"
 			(at 53.34 41.91 0)
 			(hide yes)
@@
 			"201315d9-0c4a-4b5d-aaf8-a64f48f81597" "25a1d4c5-435f-427e-9a18-669169b64384"
 			"2bbcd01b-41e2-4fec-9ac4-256a58883156" "2c474328-e688-4daf-86b5-eccb654ed3ff"
-			"303191c9-896f-4229-a9f2-9898222e4f05" "380b751a-9709-41f7-a965-c97738731820"
-			"3a3cbf4c-41c0-4cf7-abfb-fe6790f1a0e2" "4ab5176f-3c0a-442b-9c91-e712eab4f9d5"
-			"575190ec-dd69-49bf-aeda-9965da5dde9b" "58e7f43d-9884-49ac-b71c-dfa3254176ab"
-			"5ae792fc-60ff-4895-beae-93c684ae89ab" "5bdc52cf-de97-4cfd-a000-336028979491"
-			"619b54a8-a1ac-4ab0-adad-2c8b1a0b7a8a" "62424de4-f5ed-48c3-b720-23802bf51cb0"
-			"62b69d7c-0d14-4a66-a6d7-218265729aef" "641a6762-5815-49e5-bce8-e4ad8aefa749"
-			"65b20e10-a6fe-4096-94bf-6c5a163e9b81" "6755bf6a-7e56-4896-be1f-2d2d0a8244cc"
-			"68f1b546-3a87-4897-9ee3-96d3faf5d6e3" "6e5500ba-b89d-4007-93bf-b4b469bb5abe"
-			"6f2fc8c7-a29d-4f72-8013-03f67e395064" "75a39b37-c77f-4d0e-a59c-261b7b545347"
-			"7e4fb2d0-4acd-4af6-bf99-a0d4890c28c6" "8217d20b-dae9-4e16-bf7b-15d751cfd1a7"
-			"85bfd106-1ca1-41c7-871b-25a04966d8f9" "85de43fb-0da9-49c0-9117-40137aa7a2bd"
-			"88bc5302-c981-4992-916d-510b2bb74577" "8dec0c9d-26eb-4274-9e43-c95d86e036f7"
-			"8e00735d-51bf-441d-b0f2-00b4d8f8ab17" "8f073495-a1d4-433d-a680-003f3751ea53"
-			"917101e5-f73d-4bb3-9035-cb123a9d99f0" "9387c127-9ee5-4c1d-9a55-02c4ed7500a6"
-			"a148e80e-f0bd-4d58-ad97-4885cbb16e92" "a53fa4e3-5e44-4b41-83bc-60257b4a72b4"
-			"a8a7bd4c-4078-4214-b83a-bdacb85ab65f" "aca422e2-4932-4482-9648-ac424ff0cccd"
-			"add4ebc8-a739-45aa-97e7-8d64e20c273f" "b059d0c5-87ed-4543-9bea-133927449165"
-			"b0c9674d-ddd5-4260-844c-bc81b4292e26" "b5ab4d50-a971-457a-b24f-b77dae1b5235"
-			"bd215ef0-fb09-45bb-b182-59b4ddff73fd" "be48a009-e01a-409d-848f-870d51faad8e"
-			"bf1961a9-28a8-4bc2-84e2-fc534fa2cc27" "bfe62c9c-816c-41d4-8c4e-7bd1e6d8eaae"
-			"c77282e7-b7e3-43e1-8d5b-e2a6478faebc" "d0f8438f-3233-4165-bcd4-b2ba5a89213c"
+			"303191c9-896f-4229-a9f2-9898222e4f05" "3a3cbf4c-41c0-4cf7-abfb-fe6790f1a0e2"
+			"4ab5176f-3c0a-442b-9c91-e712eab4f9d5" "575190ec-dd69-49bf-aeda-9965da5dde9b"
+			"58e7f43d-9884-49ac-b71c-dfa3254176ab" "5ae792fc-60ff-4895-beae-93c684ae89ab"
+			"5bdc52cf-de97-4cfd-a000-336028979491" "619b54a8-a1ac-4ab0-adad-2c8b1a0b7a8a"
+			"62424de4-f5ed-48c3-b720-23802bf51cb0" "62b69d7c-0d14-4a66-a6d7-218265729aef"
+			"641a6762-5815-49e5-bce8-e4ad8aefa749" "65b20e10-a6fe-4096-94bf-6c5a163e9b81"
+			"6755bf6a-7e56-4896-be1f-2d2d0a8244cc" "68f1b546-3a87-4897-9ee3-96d3faf5d6e3"
+			"6e5500ba-b89d-4007-93bf-b4b469bb5abe" "6f2fc8c7-a29d-4f72-8013-03f67e395064"
+			"75a39b37-c77f-4d0e-a59c-261b7b545347" "7e4fb2d0-4acd-4af6-bf99-a0d4890c28c6"
+			"8217d20b-dae9-4e16-bf7b-15d751cfd1a7" "85bfd106-1ca1-41c7-871b-25a04966d8f9"
+			"85de43fb-0da9-49c0-9117-40137aa7a2bd" "88bc5302-c981-4992-916d-510b2bb74577"
+			"8dec0c9d-26eb-4274-9e43-c95d86e036f7" "8e00735d-51bf-441d-b0f2-00b4d8f8ab17"
+			"8f073495-a1d4-433d-a680-003f3751ea53" "917101e5-f73d-4bb3-9035-cb123a9d99f0"
+			"9387c127-9ee5-4c1d-9a55-02c4ed7500a6" "a148e80e-f0bd-4d58-ad97-4885cbb16e92"
+			"a53fa4e3-5e44-4b41-83bc-60257b4a72b4" "a8a7bd4c-4078-4214-b83a-bdacb85ab65f"
+			"aca422e2-4932-4482-9648-ac424ff0cccd" "add4ebc8-a739-45aa-97e7-8d64e20c273f"
+			"b059d0c5-87ed-4543-9bea-133927449165" "b0c9674d-ddd5-4260-844c-bc81b4292e26"
+			"b5ab4d50-a971-457a-b24f-b77dae1b5235" "bd215ef0-fb09-45bb-b182-59b4ddff73fd"
+			"be48a009-e01a-409d-848f-870d51faad8e" "bf1961a9-28a8-4bc2-84e2-fc534fa2cc27"
+			"bfe62c9c-816c-41d4-8c4e-7bd1e6d8eaae" "d0f8438f-3233-4165-bcd4-b2ba5a89213c"
 			"d3489b2e-68ce-44a8-b583-29a524c5de48" "d7fe9955-b9fd-424f-94b9-7dc2f7b2b2b7"
 			"da9132e5-5474-4524-b030-c3a0713bfc83" "db5ed4bf-e455-40fe-86c3-85b7c6216fc3"

Commit message: Add script to export production files.
Parts:
- C5, C8: BOM Value (none) -> 120pF
- C6, C7: BOM Value (none) -> 680pF
- CR10, CR11, CR12, CR13, CR16, CR17, CR18, CR9: value 1N5819WS -> 1N4148WS; BOM Value (none) -> 1N4148WS; LCSC (none) -> C2128
- Q13, Q14, Q15, Q16, Q17, Q18, Q19, Q20, Q21, Q22, Q23, Q24, Q25, Q26, Q27: BOM Value (none) -> MMBT5401; LCSC (none) -> C8326
- R100, R101, R102, R103, R104, R105, R106, R107, R108, R109, R110, R111, R112, R113, R114, R115, R116, R117, R118, R119, R120, R121, R122, R123, R124, R125, R126, R127, R129, R130, R131, R132, R133, R134, R135, R136, R137, R138, R139, R140, R141, R142, R143, R144, R387, R388, R389, R390, R391, R392, R73, R74, R75, R76, R77, R78, R79, R80, R81, R82, R83, R84, R85, R86, R87, R88, R89, R90, R91, R92, R93, R94, R95, R96, R97, R98, R99: BOM Value (none) -> 15kΩ
- R128, R145: BOM Value (none) -> 2.4kΩ
- R146, R147: BOM Value (none) -> 2.4kΩ 250mW
- R186, R188, R190, R192, R194, R196, R200, R201, R22, R24, R26, R29, R31: BOM Value (none) -> 56kΩ
- R187, R189, R191, R193, R195, R197, R23, R25, R27, R30, R32: BOM Value (none) -> 2kΩ 500mW
- R198, R199: BOM Value (none) -> 33kΩ
- R28, R384: BOM Value (none) -> 300Ω 3W

Commit message: Rough layout for Phase Control.
Connections:
- net ~{G_{S}}: now reaches C5.2, Q25.3 (C), Q26.1 (B), R146.1, R384.2
- net G_{S}: now reaches C8.2, Q24.3 (C), Q27.1 (B), R147.2, R28.2
Changed lines of the file:
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@@
+		)
+	)
+	(label "G_{S}"
+		(at 224.79 46.99 180)
+		(effects
+			(font
+				(size 1.27 1.27)
+			)
+			(justify right bottom)
+		)
+	)
+	(label "~{G_{S}}"
+		(at 144.78 27.94 0)
+		(effects
+			(font
+				(size 1.27 1.27)
+			)
+			(justify left bottom)
 		)
 	)
