File: boards/phase-control/phase-control.kicad_pcb (KiCad board)
At the start: 2 copper layers, 114.3 x 118.7 mm, 6 parts, among them P1 Card Edge

Commit message: Start the Phase Control board.
Parts:
- added C1: 120p, Capacitor_SMD:C_0402_1005Metric, F.Cu at (116.8, 109.7)
- added C10: 120p, Capacitor_SMD:C_0402_1005Metric, F.Cu at (170.2, 255.5)
- added C11: 680p, Capacitor_SMD:C_0402_1005Metric, F.Cu at (170.2, 257.5)
- added C12: 680p, Capacitor_SMD:C_0402_1005Metric, F.Cu at (170.2, 259.5)
- added C13: 120p, Capacitor_SMD:C_0402_1005Metric, F.Cu at (170.2, 261.4)
- added C14: 120p, Capacitor_SMD:C_0402_1005Metric, F.Cu at (125.9, 342.5)
- added C15: 120p, Capacitor_SMD:C_0402_1005Metric, F.Cu at (125.9, 344.5)
- added C16: 120p, Capacitor_SMD:C_0402_1005Metric, F.Cu at (125.9, 346.5)
- added C17: 120p, Capacitor_SMD:C_0402_1005Metric, F.Cu at (125.9, 348.4)
- added C18: 120p, Capacitor_SMD:C_0402_1005Metric, F.Cu at (125.9, 350.4)
- added C19: 120p, Capacitor_SMD:C_0402_1005Metric, F.Cu at (130.5, 306.2)
- added C2: 680p, Capacitor_SMD:C_0402_1005Metric, F.Cu at (116.8, 111.6)
- added C20: 120p, Capacitor_SMD:C_0402_1005Metric, F.Cu at (130.5, 308.2)
- added C21: 120p, Capacitor_SMD:C_0402_1005Metric, F.Cu at (130.5, 310.1)
- added C3: 680p, Capacitor_SMD:C_0402_1005Metric, F.Cu at (116.8, 113.6)
- added C4: 120p, Capacitor_SMD:C_0402_1005Metric, F.Cu at (116.8, 115.6)
- added C5: 120p, Capacitor_SMD:C_0402_1005Metric, F.Cu at (138.5, 229.1)
- added C6: 680p, Capacitor_SMD:C_0402_1005Metric, F.Cu at (138.5, 231.1)
- added C7: 680p, Capacitor_SMD:C_0402_1005Metric, F.Cu at (138.5, 233.0)
- added C8: 120p, Capacitor_SMD:C_0402_1005Metric, F.Cu at (138.5, 235.0)
- added C9: 680p, Capacitor_SMD:C_0402_1005Metric, F.Cu at (179.6, 286.6)
- added C900: 680p, Capacitor_SMD:C_0402_1005Metric, F.Cu at (130.5, 312.1)
- added CR1: 1N5819WS, Diode_SMD:D_SOD-323, F.Cu at (123.2, 111.3)
- added CR10: 1N5819WS, Diode_SMD:D_SOD-323, F.Cu at (134.9, 232.5)
- added CR11: 1N5819WS, Diode_SMD:D_SOD-323, F.Cu at (134.9, 235.5)
- added CR12: 1N5819WS, Diode_SMD:D_SOD-323, F.Cu at (134.9, 238.4)
- added CR13: 1N5819WS, Diode_SMD:D_SOD-323, F.Cu at (134.9, 241.4)
- added CR16: 1N5819WS, Diode_SMD:D_SOD-323, F.Cu at (134.9, 244.3)
- added CR17: 1N5819WS, Diode_SMD:D_SOD-323, F.Cu at (134.9, 247.3)
- added CR18: 1N5819WS, Diode_SMD:D_SOD-323, F.Cu at (134.9, 250.2)
- added CR2: 1N5819WS, Diode_SMD:D_SOD-323, F.Cu at (123.2, 114.3)
- added CR20: 1N5819WS, Diode_SMD:D_SOD-323, F.Cu at (146.5, 242.7)
- added CR21: 1N5819WS, Diode_SMD:D_SOD-323, F.Cu at (146.5, 245.6)
- added CR22: 1N5819WS, Diode_SMD:D_SOD-323, F.Cu at (146.5, 248.6)
- added CR23: 1N5819WS, Diode_SMD:D_SOD-323, F.Cu at (146.5, 251.5)
- added CR24: 1N5819WS, Diode_SMD:D_SOD-323, F.Cu at (146.5, 254.5)
- added CR25: 1N5819WS, Diode_SMD:D_SOD-323, F.Cu at (146.5, 257.4)
- added CR26: 1N5819WS, Diode_SMD:D_SOD-323, F.Cu at (146.5, 260.4)
- added CR27: 1N5819WS, Diode_SMD:D_SOD-323, F.Cu at (146.5, 263.3)
- added CR28: 1N5819WS, Diode_SMD:D_SOD-323, F.Cu at (176.0, 272.3)
- added CR29: 1N5819WS, Diode_SMD:D_SOD-323, F.Cu at (176.0, 275.2)
- added CR3: 1N5819WS, Diode_SMD:D_SOD-323, F.Cu at (140.0, 335.6)
- added CR30: 1N5819WS, Diode_SMD:D_SOD-323, F.Cu at (113.8, 343.0)
- added CR31: 1N5819WS, Diode_SMD:D_SOD-323, F.Cu at (113.8, 346.0)
- added CR32: 1N5819WS, Diode_SMD:D_SOD-323, F.Cu at (113.8, 348.9)
- added CR33: 1N5819WS, Diode_SMD:D_SOD-323, F.Cu at (113.8, 351.9)
- added CR34: 1N5819WS, Diode_SMD:D_SOD-323, F.Cu at (113.8, 354.8)
- added CR35: 1N5819WS, Diode_SMD:D_SOD-323, F.Cu at (118.0, 343.0)
- added CR36: 1N5819WS, Diode_SMD:D_SOD-323, F.Cu at (118.0, 346.0)
- added CR37: 1N5819WS, Diode_SMD:D_SOD-323, F.Cu at (118.0, 348.9)
- added CR38: 1N5819WS, Diode_SMD:D_SOD-323, F.Cu at (118.0, 351.9)
- added CR39: 1N5819WS, Diode_SMD:D_SOD-323, F.Cu at (118.0, 354.8)
- added CR4: 1N5819WS, Diode_SMD:D_SOD-323, F.Cu at (140.0, 338.5)
- added CR40: 1N5819WS, Diode_SMD:D_SOD-323, F.Cu at (122.3, 343.0)
- added CR41: 1N5819WS, Diode_SMD:D_SOD-323, F.Cu at (122.3, 346.0)
- added CR42: 1N5819WS, Diode_SMD:D_SOD-323, F.Cu at (122.3, 348.9)
- added CR43: 1N5819WS, Diode_SMD:D_SOD-323, F.Cu at (131.2, 291.9)
- added CR44: 1N5819WS, Diode_SMD:D_SOD-323, F.Cu at (131.2, 294.9)
- added CR45: 1N5819WS, Diode_SMD:D_SOD-323, F.Cu at (131.2, 297.8)
- added CR46: 1N5819WS, Diode_SMD:D_SOD-323, F.Cu at (131.2, 300.8)
- added CR47: 1N5819WS, Diode_SMD:D_SOD-323, F.Cu at (131.2, 303.7)
- added CR48: 1N5819WS, Diode_SMD:D_SOD-323, F.Cu at (135.5, 291.9)
- added CR49: 1N5819WS, Diode_SMD:D_SOD-323, F.Cu at (135.5, 294.9)
- added CR5: 1N5819WS, Diode_SMD:D_SOD-323, F.Cu at (140.0, 341.5)
- added CR50: 1N5819WS, Diode_SMD:D_SOD-323, F.Cu at (135.5, 297.8)
- added CR51: 1N5819WS, Diode_SMD:D_SOD-323, F.Cu at (135.5, 300.8)
- added CR52: 1N5819WS, Diode_SMD:D_SOD-323, F.Cu at (135.5, 303.7)
- added CR53: 1N5819WS, Diode_SMD:D_SOD-323, F.Cu at (139.8, 291.9)
- added CR54: 1N5819WS, Diode_SMD:D_SOD-323, F.Cu at (139.8, 294.9)
- added CR55: 1N5819WS, Diode_SMD:D_SOD-323, F.Cu at (139.8, 297.8)
- added CR56: 1N5819WS, Diode_SMD:D_SOD-323, F.Cu at (176.0, 278.2)
- added CR57: 1N5819WS, Diode_SMD:D_SOD-323, F.Cu at (176.0, 281.1)
- added CR58: 1N5819WS, Diode_SMD:D_SOD-323, F.Cu at (176.0, 284.1)
- added CR59: 1N5819WS, Diode_SMD:D_SOD-323, F.Cu at (180.3, 272.3)
- added CR6: 1N5819WS, Diode_SMD:D_SOD-323, F.Cu at (186.4, 334.6)
- added CR60: 1N5819WS, Diode_SMD:D_SOD-323, F.Cu at (180.3, 275.2)
- added CR7: 1N5819WS, Diode_SMD:D_SOD-323, F.Cu at (186.4, 337.5)
- added CR8: 1N5819WS, Diode_SMD:D_SOD-323, F.Cu at (186.4, 340.5)
- added CR9: 1N5819WS, Diode_SMD:D_SOD-323, F.Cu at (134.9, 229.6)
- added CR90: 1N5819WS, Diode_SMD:D_SOD-323, F.Cu at (180.3, 278.2)
- added CR91: 1N5819WS, Diode_SMD:D_SOD-323, F.Cu at (180.3, 281.1)
- added CR92: 1N5819WS, Diode_SMD:D_SOD-323, F.Cu at (180.3, 284.1)
- added CR93: 1N5819WS, Diode_SMD:D_SOD-323, F.Cu at (139.8, 300.8)
- added Q1: MMBT5401, Package_TO_SOT_SMD:SOT-23, F.Cu at (144.6, 351.5)
- added Q10: MMBT5401, Package_TO_SOT_SMD:SOT-23, F.Cu at (105.4, 111.8)
- added Q11: MMBT5401, Package_TO_SOT_SMD:SOT-23, F.Cu at (159.3, 355.9)
- added Q12: MMBT5401, Package_TO_SOT_SMD:SOT-23, F.Cu at (205.7, 350.5)
- added Q13: MMBT5401, Package_TO_SOT_SMD:SOT-23, F.Cu at (120.5, 230.3)
- added Q14: MMBT5401, Package_TO_SOT_SMD:SOT-23, F.Cu at (120.5, 234.8)
- added Q15: MMBT5401, Package_TO_SOT_SMD:SOT-23, F.Cu at (120.5, 239.2)
- added Q16: MMBT5401, Package_TO_SOT_SMD:SOT-23, F.Cu at (120.5, 243.7)
- added Q17: MMBT5401, Package_TO_SOT_SMD:SOT-23, F.Cu at (120.5, 248.1)
- added Q18: MMBT5401, Package_TO_SOT_SMD:SOT-23, F.Cu at (120.5, 252.6)
- added Q19: MMBT5401, Package_TO_SOT_SMD:SOT-23, F.Cu at (125.4, 230.3)
- added Q2: MMBT5401, Package_TO_SOT_SMD:SOT-23, F.Cu at (144.6, 355.9)
- added Q20: MMBT5401, Package_TO_SOT_SMD:SOT-23, F.Cu at (125.4, 234.8)
- added Q21: MMBT5401, Package_TO_SOT_SMD:SOT-23, F.Cu at (125.4, 239.2)
- added Q22: MMBT5401, Package_TO_SOT_SMD:SOT-23, F.Cu at (125.4, 243.7)
- added Q23: MMBT5401, Package_TO_SOT_SMD:SOT-23, F.Cu at (125.4, 248.1)
- added Q24: MMBT5401, Package_TO_SOT_SMD:SOT-23, F.Cu at (125.4, 252.6)
- added Q25: MMBT5401, Package_TO_SOT_SMD:SOT-23, F.Cu at (130.3, 230.3)
- added Q26: MMBT5401, Package_TO_SOT_SMD:SOT-23, F.Cu at (130.3, 234.8)
- added Q27: MMBT5401, Package_TO_SOT_SMD:SOT-23, F.Cu at (130.3, 239.2)
- added Q28: MMBT5401, Package_TO_SOT_SMD:SOT-23, F.Cu at (121.5, 273.0)
- added Q29: MMBT5401, Package_TO_SOT_SMD:SOT-23, F.Cu at (121.5, 277.5)
- added Q3: MMBT5401, Package_TO_SOT_SMD:SOT-23, F.Cu at (144.6, 360.4)
- added Q30: MMBT5401, Package_TO_SOT_SMD:SOT-23, F.Cu at (121.5, 281.9)
- added Q31: MMBT5401, Package_TO_SOT_SMD:SOT-23, F.Cu at (121.5, 286.4)
- added Q32: MMBT5401, Package_TO_SOT_SMD:SOT-23, F.Cu at (126.4, 273.0)
- added Q33: MMBT5401, Package_TO_SOT_SMD:SOT-23, F.Cu at (126.4, 277.5)
- added Q34: MMBT5401, Package_TO_SOT_SMD:SOT-23, F.Cu at (126.4, 281.9)
- added Q35: MMBT5401, Package_TO_SOT_SMD:SOT-23, F.Cu at (126.4, 286.4)
- added Q36: MMBT5401, Package_TO_SOT_SMD:SOT-23, F.Cu at (131.3, 273.0)
- added Q37: MMBT5401, Package_TO_SOT_SMD:SOT-23, F.Cu at (131.3, 277.5)
- added Q38: MMBT5401, Package_TO_SOT_SMD:SOT-23, F.Cu at (131.3, 281.9)
- added Q39: MMBT5401, Package_TO_SOT_SMD:SOT-23, F.Cu at (131.3, 286.4)
- added Q4: MMBT5401, Package_TO_SOT_SMD:SOT-23, F.Cu at (149.5, 351.5)
- added Q40: MMBT5401, Package_TO_SOT_SMD:SOT-23, F.Cu at (152.0, 292.7)
- added Q41: MMBT5401, Package_TO_SOT_SMD:SOT-23, F.Cu at (152.0, 297.1)
- added Q42: MMBT5401, Package_TO_SOT_SMD:SOT-23, F.Cu at (152.0, 301.6)
- added Q43: MMBT5401, Package_TO_SOT_SMD:SOT-23, F.Cu at (156.9, 292.7)
- added Q44: MMBT5401, Package_TO_SOT_SMD:SOT-23, F.Cu at (156.9, 297.1)
- added Q45: MMBT5401, Package_TO_SOT_SMD:SOT-23, F.Cu at (156.9, 301.6)
- added Q46: MMBT5401, Package_TO_SOT_SMD:SOT-23, F.Cu at (161.8, 292.7)
- added Q47: MMBT5401, Package_TO_SOT_SMD:SOT-23, F.Cu at (161.8, 297.1)
- added Q48: MMBT5401, Package_TO_SOT_SMD:SOT-23, F.Cu at (161.8, 301.6)
- added Q49: MMBT5401, Package_TO_SOT_SMD:SOT-23, F.Cu at (166.7, 292.7)
- added Q5: MMBT5401, Package_TO_SOT_SMD:SOT-23, F.Cu at (149.5, 355.9)
- added Q50: MMBT5401, Package_TO_SOT_SMD:SOT-23, F.Cu at (156.7, 243.4)
- added Q51: MMBT5401, Package_TO_SOT_SMD:SOT-23, F.Cu at (156.7, 247.9)
- added Q52: MMBT5401, Package_TO_SOT_SMD:SOT-23, F.Cu at (156.7, 252.3)
- added Q53: MMBT5401, Package_TO_SOT_SMD:SOT-23, F.Cu at (161.6, 243.4)
- added Q54: MMBT5401, Package_TO_SOT_SMD:SOT-23, F.Cu at (161.6, 247.9)
- added Q55: MMBT5401, Package_TO_SOT_SMD:SOT-23, F.Cu at (161.6, 252.3)
- added Q56: MMBT5401, Package_TO_SOT_SMD:SOT-23, F.Cu at (166.5, 243.4)
- added Q57: MMBT5401, Package_TO_SOT_SMD:SOT-23, F.Cu at (166.5, 247.9)
- added Q58: MMBT5401, Package_TO_SOT_SMD:SOT-23, F.Cu at (166.5, 252.3)
- added Q59: MMBT5401, Package_TO_SOT_SMD:SOT-23, F.Cu at (166.7, 297.1)
- added Q6: MMBT5401, Package_TO_SOT_SMD:SOT-23, F.Cu at (149.5, 360.4)
- added Q60: MMBT5401, Package_TO_SOT_SMD:SOT-23, F.Cu at (166.7, 301.6)
- added Q61: MMBT5401, Package_TO_SOT_SMD:SOT-23, F.Cu at (97.2, 338.4)
- added Q62: MMBT5401, Package_TO_SOT_SMD:SOT-23, F.Cu at (97.2, 342.8)
- added Q63: MMBT5401, Package_TO_SOT_SMD:SOT-23, F.Cu at (97.2, 347.3)
- added Q64: MMBT5401, Package_TO_SOT_SMD:SOT-23, F.Cu at (97.2, 351.7)
- added Q65: MMBT5401, Package_TO_SOT_SMD:SOT-23, F.Cu at (97.2, 356.2)
- added Q66: MMBT5401, Package_TO_SOT_SMD:SOT-23, F.Cu at (102.1, 338.4)
- added Q67: MMBT5401, Package_TO_SOT_SMD:SOT-23, F.Cu at (102.1, 342.8)
- added Q68: MMBT5401, Package_TO_SOT_SMD:SOT-23, F.Cu at (102.1, 347.3)
- added Q69: MMBT5401, Package_TO_SOT_SMD:SOT-23, F.Cu at (102.1, 351.7)
- added Q7: MMBT5401, Package_TO_SOT_SMD:SOT-23, F.Cu at (154.4, 351.5)
- added Q70: MMBT5401, Package_TO_SOT_SMD:SOT-23, F.Cu at (102.1, 356.2)
- added Q71: MMBT5401, Package_TO_SOT_SMD:SOT-23, F.Cu at (107.0, 338.4)
- added Q72: MMBT5401, Package_TO_SOT_SMD:SOT-23, F.Cu at (107.0, 342.8)
- added Q73: MMBT5401, Package_TO_SOT_SMD:SOT-23, F.Cu at (107.0, 347.3)
- added Q74: MMBT5401, Package_TO_SOT_SMD:SOT-23, F.Cu at (136.2, 273.0)
- added Q75: MMBT5401, Package_TO_SOT_SMD:SOT-23, F.Cu at (136.2, 277.5)
- added Q76: MMBT5401, Package_TO_SOT_SMD:SOT-23, F.Cu at (136.2, 281.9)
- added Q77: MMBT5401, Package_TO_SOT_SMD:SOT-23, F.Cu at (136.2, 286.4)
- added Q8: MMBT5401, Package_TO_SOT_SMD:SOT-23, F.Cu at (154.4, 355.9)
- added Q9: MMBT5401, Package_TO_SOT_SMD:SOT-23, F.Cu at (105.4, 118.1)
- added R1: 56k, Resistor_SMD:R_0402_1005Metric, F.Cu at (154.8, 329.2)
- added R10: 2k ½W, Resistor_SMD:R_1210_3225Metric, F.Cu at (144.9, 347.1)
- added R100: 15k, Resistor_SMD:R_0402_1005Metric, F.Cu at (102.0, 245.0)
- added R101: 15k, Resistor_SMD:R_0402_1005Metric, F.Cu at (102.0, 247.0)
- added R102: 15k, Resistor_SMD:R_0402_1005Metric, F.Cu at (102.0, 249.0)
- added R103: 15k, Resistor_SMD:R_0402_1005Metric, F.Cu at (102.0, 251.0)
- added R104: 15k, Resistor_SMD:R_0402_1005Metric, F.Cu at (104.9, 229.1)
- added R105: 15k, Resistor_SMD:R_0402_1005Metric, F.Cu at (104.9, 231.1)
- added R106: 15k, Resistor_SMD:R_0402_1005Metric, F.Cu at (104.9, 233.1)
- added R107: 15k, Resistor_SMD:R_0402_1005Metric, F.Cu at (104.9, 235.1)
- added R108: 15k, Resistor_SMD:R_0402_1005Metric, F.Cu at (104.9, 237.1)
- added R109: 15k, Resistor_SMD:R_0402_1005Metric, F.Cu at (104.9, 239.0)
- added R11: 56k, Resistor_SMD:R_0402_1005Metric, F.Cu at (154.8, 339.1)
- added R110: 15k, Resistor_SMD:R_0402_1005Metric, F.Cu at (104.9, 241.0)
- added R111: 15k, Resistor_SMD:R_0402_1005Metric, F.Cu at (104.9, 243.0)
- added R112: 15k, Resistor_SMD:R_0402_1005Metric, F.Cu at (104.9, 245.0)
- added R113: 15k, Resistor_SMD:R_0402_1005Metric, F.Cu at (104.9, 247.0)
- added R114: 15k, Resistor_SMD:R_0402_1005Metric, F.Cu at (104.9, 249.0)
- added R115: 15k, Resistor_SMD:R_0402_1005Metric, F.Cu at (104.9, 251.0)
- added R116: 15k, Resistor_SMD:R_0402_1005Metric, F.Cu at (107.8, 229.1)
- added R117: 15k, Resistor_SMD:R_0402_1005Metric, F.Cu at (107.8, 231.1)
- added R118: 15k, Resistor_SMD:R_0402_1005Metric, F.Cu at (107.8, 233.1)
- added R119: 15k, Resistor_SMD:R_0402_1005Metric, F.Cu at (107.8, 235.1)
- added R12: 2k ½W, Resistor_SMD:R_1210_3225Metric, F.Cu at (150.6, 330.3)
- added R120: 15k, Resistor_SMD:R_0402_1005Metric, F.Cu at (107.8, 237.1)
- added R121: 15k, Resistor_SMD:R_0402_1005Metric, F.Cu at (107.8, 239.0)
- added R122: 15k, Resistor_SMD:R_0402_1005Metric, F.Cu at (107.8, 241.0)
- added R123: 15k, Resistor_SMD:R_0402_1005Metric, F.Cu at (107.8, 243.0)
- added R124: 15k, Resistor_SMD:R_0402_1005Metric, F.Cu at (107.8, 245.0)
- added R125: 15k, Resistor_SMD:R_0402_1005Metric, F.Cu at (107.8, 247.0)
- added R126: 15k, Resistor_SMD:R_0402_1005Metric, F.Cu at (107.8, 249.0)
- added R127: 15k, Resistor_SMD:R_0402_1005Metric, F.Cu at (107.8, 251.0)
- added R128: 2k4, Resistor_SMD:R_0402_1005Metric, F.Cu at (110.8, 229.1)
- added R129: 15k, Resistor_SMD:R_0402_1005Metric, F.Cu at (110.8, 231.1)
- added R13: 56k, Resistor_SMD:R_0402_1005Metric, F.Cu at (154.8, 341.1)
- added R130: 15k, Resistor_SMD:R_0402_1005Metric, F.Cu at (110.8, 233.1)
- added R131: 15k, Resistor_SMD:R_0402_1005Metric, F.Cu at (110.8, 235.1)
- added R132: 15k, Resistor_SMD:R_0402_1005Metric, F.Cu at (110.8, 237.1)
- added R133: 15k, Resistor_SMD:R_0402_1005Metric, F.Cu at (110.8, 239.0)
- added R134: 15k, Resistor_SMD:R_0402_1005Metric, F.Cu at (110.8, 241.0)
- added R135: 15k, Resistor_SMD:R_0402_1005Metric, F.Cu at (110.8, 243.0)
- added R136: 15k, Resistor_SMD:R_0402_1005Metric, F.Cu at (110.8, 245.0)
- added R137: 15k, Resistor_SMD:R_0402_1005Metric, F.Cu at (110.8, 247.0)
- added R138: 15k, Resistor_SMD:R_0402_1005Metric, F.Cu at (110.8, 249.0)
- added R139: 15k, Resistor_SMD:R_0402_1005Metric, F.Cu at (110.8, 251.0)
- added R14: 2k ½W, Resistor_SMD:R_1210_3225Metric, F.Cu at (150.6, 334.5)
- added R140: 15k, Resistor_SMD:R_0402_1005Metric, F.Cu at (113.7, 229.1)
- added R141: 15k, Resistor_SMD:R_0402_1005Metric, F.Cu at (113.7, 231.1)
- added R142: 15k, Resistor_SMD:R_0402_1005Metric, F.Cu at (113.7, 233.1)
- added R143: 15k, Resistor_SMD:R_0402_1005Metric, F.Cu at (113.7, 235.1)
- added R144: 15k, Resistor_SMD:R_0402_1005Metric, F.Cu at (113.7, 237.1)
- added R145: 2k4, Resistor_SMD:R_0402_1005Metric, F.Cu at (113.7, 239.0)
- added R146: 2k4 ¼W, Resistor_SMD:R_0603_1608Metric, F.Cu at (139.1, 237.2)
- added R147: 2k4 ¼W, Resistor_SMD:R_0603_1608Metric, F.Cu at (139.1, 239.7)
- added R148: 15k, Resistor_SMD:R_0402_1005Metric, F.Cu at (113.0, 291.5)
- added R149: 15k, Resistor_SMD:R_0402_1005Metric, F.Cu at (113.0, 293.5)
- added R15: 56k, Resistor_SMD:R_0402_1005Metric, F.Cu at (154.8, 343.1)
- added R150: 15k, Resistor_SMD:R_0402_1005Metric, F.Cu at (113.0, 295.4)
- added R151: 15k, Resistor_SMD:R_0402_1005Metric, F.Cu at (113.0, 297.4)
- added R152: 15k, Resistor_SMD:R_0402_1005Metric, F.Cu at (113.0, 299.4)
- added R153: 15k, Resistor_SMD:R_0402_1005Metric, F.Cu at (113.0, 301.4)
- added R154: 15k, Resistor_SMD:R_0402_1005Metric, F.Cu at (113.0, 303.4)
- added R155: 15k, Resistor_SMD:R_0402_1005Metric, F.Cu at (113.0, 305.4)
- added R156: 15k, Resistor_SMD:R_0402_1005Metric, F.Cu at (113.0, 307.4)
- added R157: 15k, Resistor_SMD:R_0402_1005Metric, F.Cu at (113.0, 309.4)
- added R158: 15k, Resistor_SMD:R_0402_1005Metric, F.Cu at (115.9, 291.5)
- added R159: 15k, Resistor_SMD:R_0402_1005Metric, F.Cu at (115.9, 293.5)
- added R16: 2k ½W, Resistor_SMD:R_1210_3225Metric, F.Cu at (150.6, 338.7)
- added R160: 15k, Resistor_SMD:R_0402_1005Metric, F.Cu at (115.9, 295.4)
- added R161: 15k, Resistor_SMD:R_0402_1005Metric, F.Cu at (115.9, 297.4)
- added R162: 15k, Resistor_SMD:R_0402_1005Metric, F.Cu at (115.9, 299.4)
- added R163: 15k, Resistor_SMD:R_0402_1005Metric, F.Cu at (115.9, 301.4)
- added R164: 15k, Resistor_SMD:R_0402_1005Metric, F.Cu at (115.9, 303.4)
- added R165: 15k, Resistor_SMD:R_0402_1005Metric, F.Cu at (115.9, 305.4)
- added R166: 15k, Resistor_SMD:R_0402_1005Metric, F.Cu at (115.9, 307.4)
- added R167: 15k, Resistor_SMD:R_0402_1005Metric, F.Cu at (115.9, 309.4)
- added R168: 15k, Resistor_SMD:R_0402_1005Metric, F.Cu at (118.9, 291.5)
- added R169: 15k, Resistor_SMD:R_0402_1005Metric, F.Cu at (118.9, 293.5)
- added R17: 33k, Resistor_SMD:R_0402_1005Metric, F.Cu at (112.2, 110.5)
- added R170: 15k, Resistor_SMD:R_0402_1005Metric, F.Cu at (118.9, 295.4)
- added R171: 15k, Resistor_SMD:R_0402_1005Metric, F.Cu at (118.9, 297.4)
- added R172: 15k, Resistor_SMD:R_0402_1005Metric, F.Cu at (118.9, 299.4)
- added R173: 15k, Resistor_SMD:R_0402_1005Metric, F.Cu at (118.9, 301.4)
- added R174: 15k, Resistor_SMD:R_0402_1005Metric, F.Cu at (118.9, 303.4)
- added R175: 15k, Resistor_SMD:R_0402_1005Metric, F.Cu at (118.9, 305.4)
- added R176: 15k, Resistor_SMD:R_0402_1005Metric, F.Cu at (118.9, 307.4)
- added R177: 15k, Resistor_SMD:R_0402_1005Metric, F.Cu at (118.9, 309.4)
- added R178: 15k, Resistor_SMD:R_0402_1005Metric, F.Cu at (121.8, 291.5)
- added R179: 15k, Resistor_SMD:R_0402_1005Metric, F.Cu at (121.8, 293.5)
- added R18: 33k, Resistor_SMD:R_0402_1005Metric, F.Cu at (112.2, 112.5)
- added R180: 15k, Resistor_SMD:R_0402_1005Metric, F.Cu at (121.8, 295.4)
- added R181: 15k, Resistor_SMD:R_0402_1005Metric, F.Cu at (121.8, 297.4)
- added R182: 15k, Resistor_SMD:R_0402_1005Metric, F.Cu at (170.6, 291.5)
- added R183: 15k, Resistor_SMD:R_0402_1005Metric, F.Cu at (170.6, 293.5)
- added R184: 6k8, Resistor_SMD:R_0402_1005Metric, F.Cu at (170.6, 295.4)
- added R185: 450R 2W, Resistor_THT:R_Axial_DIN0516_L15.5mm_D5.0mm_P20.32mm_Horizontal, F.Cu at (151.5, 274.1)
- added R186: 56k, Resistor_SMD:R_0402_1005Metric, F.Cu at (113.7, 241.0)
- added R187: 2k ½W, Resistor_SMD:R_1210_3225Metric, F.Cu at (103.2, 258.3)
- added R188: 56k, Resistor_SMD:R_0402_1005Metric, F.Cu at (113.7, 243.0)
- added R189: 2k ½W, Resistor_SMD:R_1210_3225Metric, F.Cu at (103.2, 262.5)
- added R19: 56k, Resistor_SMD:R_0402_1005Metric, F.Cu at (157.7, 329.2)
- added R190: 56k, Resistor_SMD:R_0402_1005Metric, F.Cu at (113.7, 245.0)
- added R191: 2k ½W, Resistor_SMD:R_1210_3225Metric, F.Cu at (103.2, 266.7)
- added R192: 56k, Resistor_SMD:R_0402_1005Metric, F.Cu at (113.7, 247.0)
- added R193: 2k ½W, Resistor_SMD:R_1210_3225Metric, F.Cu at (108.8, 254.1)
- added R194: 56k, Resistor_SMD:R_0402_1005Metric, F.Cu at (113.7, 249.0)
- added R195: 2k ½W, Resistor_SMD:R_1210_3225Metric, F.Cu at (108.8, 258.3)
- added R196: 56k, Resistor_SMD:R_0402_1005Metric, F.Cu at (113.7, 251.0)
- added R197: 2k ½W, Resistor_SMD:R_1210_3225Metric, F.Cu at (108.8, 262.5)
- added R198: 33k, Resistor_SMD:R_0402_1005Metric, F.Cu at (116.6, 229.1)
- added R199: 33k, Resistor_SMD:R_0402_1005Metric, F.Cu at (116.6, 231.1)
- added R2: 2k ½W, Resistor_SMD:R_1210_3225Metric, F.Cu at (144.9, 330.3)
- added R20: 56k, Resistor_SMD:R_0402_1005Metric, F.Cu at (204.1, 321.3)
- added R200: 56k, Resistor_SMD:R_0402_1005Metric, F.Cu at (116.6, 233.1)
- added R201: 56k, Resistor_SMD:R_0402_1005Metric, F.Cu at (116.6, 235.1)
- added R202: 56k, Resistor_SMD:R_0402_1005Metric, F.Cu at (121.8, 299.4)
- added R203: 2k ½W, Resistor_SMD:R_1210_3225Metric, F.Cu at (97.6, 292.6)
- added R204: 56k, Resistor_SMD:R_0402_1005Metric, F.Cu at (121.8, 301.4)
- added R205: 2k ½W, Resistor_SMD:R_1210_3225Metric, F.Cu at (97.6, 296.8)
- added R206: 56k, Resistor_SMD:R_0402_1005Metric, F.Cu at (121.8, 303.4)
- added R207: 2k ½W, Resistor_SMD:R_1210_3225Metric, F.Cu at (97.6, 301.0)
- added R208: 56k, Resistor_SMD:R_0402_1005Metric, F.Cu at (121.8, 305.4)
- added R209: 2k ½W, Resistor_SMD:R_1210_3225Metric, F.Cu at (97.6, 305.2)
- added R21: 300R 3W, Resistor_THT:R_Axial_DIN0516_L15.5mm_D5.0mm_P20.32mm_Horizontal, F.Cu at (139.8, 318.4)
- added R210: 56k, Resistor_SMD:R_0402_1005Metric, F.Cu at (121.8, 307.4)
- added R211: 2k ½W, Resistor_SMD:R_1210_3225Metric, F.Cu at (97.6, 309.4)
- added R212: 56k, Resistor_SMD:R_0402_1005Metric, F.Cu at (121.8, 309.4)
- added R213: 2k ½W, Resistor_SMD:R_1210_3225Metric, F.Cu at (103.2, 292.6)
- added R214: 56k, Resistor_SMD:R_0402_1005Metric, F.Cu at (124.7, 291.5)
- added R215: 2k ½W, Resistor_SMD:R_1210_3225Metric, F.Cu at (103.2, 296.8)
- added R216: 56k, Resistor_SMD:R_0402_1005Metric, F.Cu at (124.7, 293.5)
- added R217: 2k ½W, Resistor_SMD:R_1210_3225Metric, F.Cu at (103.2, 301.0)
- added R218: 56k, Resistor_SMD:R_0402_1005Metric, F.Cu at (124.7, 295.4)
- added R219: 2k ½W, Resistor_SMD:R_1210_3225Metric, F.Cu at (103.2, 305.2)
- added R22: 56k, Resistor_SMD:R_0402_1005Metric, F.Cu at (96.2, 229.1)
- added R220: 56k, Resistor_SMD:R_0402_1005Metric, F.Cu at (124.7, 297.4)
- added R221: 2k ½W, Resistor_SMD:R_1210_3225Metric, F.Cu at (103.2, 309.4)
- added R222: 56k, Resistor_SMD:R_0402_1005Metric, F.Cu at (124.7, 299.4)
- added R223: 2k ½W, Resistor_SMD:R_1210_3225Metric, F.Cu at (108.8, 292.6)
- added R224: 56k, Resistor_SMD:R_0402_1005Metric, F.Cu at (124.7, 301.4)
- added R225: 2k ½W, Resistor_SMD:R_1210_3225Metric, F.Cu at (108.8, 296.8)
- added R226: 56k, Resistor_SMD:R_0402_1005Metric, F.Cu at (170.6, 297.4)
- added R227: 800R 2W, Resistor_THT:R_Axial_DIN0516_L15.5mm_D5.0mm_P20.32mm_Horizontal, F.Cu at (151.5, 280.6)
- added R228: 56k, Resistor_SMD:R_0402_1005Metric, F.Cu at (170.6, 299.4)
- added R229: 2k ⅛W, Resistor_SMD:R_0805_2012Metric, F.Cu at (176.0, 287.0)
- added R23: 2k ½W, Resistor_SMD:R_1210_3225Metric, F.Cu at (97.6, 254.1)
- added R230: 56k, Resistor_SMD:R_0402_1005Metric, F.Cu at (170.6, 301.4)
- added R231: 2k ½W, Resistor_SMD:R_1210_3225Metric, F.Cu at (146.7, 272.9)
- added R232: 56k, Resistor_SMD:R_0402_1005Metric, F.Cu at (170.6, 303.4)
- added R233: 2k ½W, Resistor_SMD:R_1210_3225Metric, F.Cu at (146.7, 277.1)
- added R234: 56k, Resistor_SMD:R_0402_1005Metric, F.Cu at (173.5, 291.5)
- added R235: 56k, Resistor_SMD:R_0402_1005Metric, F.Cu at (173.5, 293.5)
- added R236: 2k ½W, Resistor_SMD:R_1210_3225Metric, F.Cu at (146.7, 281.3)
- added R237: 56k, Resistor_SMD:R_0402_1005Metric, F.Cu at (173.5, 295.4)
- added R238: 2k ½W, Resistor_SMD:R_1210_3225Metric, F.Cu at (146.7, 285.6)
- added R239: 56k, Resistor_SMD:R_0402_1005Metric, F.Cu at (173.5, 297.4)
- added R24: 56k, Resistor_SMD:R_0402_1005Metric, F.Cu at (96.2, 231.1)
- added R240: 2k ½W, Resistor_SMD:R_1210_3225Metric, F.Cu at (146.7, 289.8)
- added R241: 56k, Resistor_SMD:R_0402_1005Metric, F.Cu at (173.5, 299.4)
- added R242: 2k ½W, Resistor_SMD:R_1210_3225Metric, F.Cu at (146.7, 294.0)
- added R243: 56k, Resistor_SMD:R_0402_1005Metric, F.Cu at (155.7, 255.5)
- added R244: 2k ½W, Resistor_SMD:R_1210_3225Metric, F.Cu at (151.4, 243.3)
- added R245: 56k, Resistor_SMD:R_0402_1005Metric, F.Cu at (155.7, 257.5)
- added R246: 2k ½W, Resistor_SMD:R_1210_3225Metric, F.Cu at (151.4, 247.5)
- added R247: 56k, Resistor_SMD:R_0402_1005Metric, F.Cu at (155.7, 259.5)
- added R248: 2k ½W, Resistor_SMD:R_1210_3225Metric, F.Cu at (151.4, 251.7)
- added R249: 56k, Resistor_SMD:R_0402_1005Metric, F.Cu at (155.7, 261.5)
- added R25: 2k ½W, Resistor_SMD:R_1210_3225Metric, F.Cu at (97.6, 258.3)
- added R250: 2k ½W, Resistor_SMD:R_1210_3225Metric, F.Cu at (151.4, 255.9)
- added R251: 56k, Resistor_SMD:R_0402_1005Metric, F.Cu at (155.7, 263.5)
- added R252: 2k ½W, Resistor_SMD:R_1210_3225Metric, F.Cu at (151.4, 260.1)
- added R253: 33k, Resistor_SMD:R_0402_1005Metric, F.Cu at (155.7, 265.5)
- added R254: 33k, Resistor_SMD:R_0402_1005Metric, F.Cu at (158.6, 255.5)
- added R255: 56k, Resistor_SMD:R_0402_1005Metric, F.Cu at (158.6, 257.5)
- added R256: 56k, Resistor_SMD:R_0402_1005Metric, F.Cu at (158.6, 259.5)
- added R257: 56k, Resistor_SMD:R_0402_1005Metric, F.Cu at (173.5, 301.4)
- added R258: 800R 2W, Resistor_THT:R_Axial_DIN0516_L15.5mm_D5.0mm_P20.32mm_Horizontal, F.Cu at (151.5, 287.2)
- added R259: 56k, Resistor_SMD:R_0402_1005Metric, F.Cu at (173.5, 303.4)
- added R26: 56k, Resistor_SMD:R_0402_1005Metric, F.Cu at (96.2, 233.1)
- added R260: 2k ½W, Resistor_SMD:R_1210_3225Metric, F.Cu at (146.7, 298.2)
- added R261: 15k, Resistor_SMD:R_0402_1005Metric, F.Cu at (176.4, 291.5)
- added R262: 15k, Resistor_SMD:R_0402_1005Metric, F.Cu at (176.4, 293.5)
- added R263: 15k, Resistor_SMD:R_0402_1005Metric, F.Cu at (176.4, 295.4)
- added R264: 15k, Resistor_SMD:R_0402_1005Metric, F.Cu at (176.4, 297.4)
- added R265: 15k, Resistor_SMD:R_0402_1005Metric, F.Cu at (176.4, 299.4)
- added R266: 15k, Resistor_SMD:R_0402_1005Metric, F.Cu at (176.4, 301.4)
- added R267: 15k, Resistor_SMD:R_0402_1005Metric, F.Cu at (176.4, 303.4)
- added R268: 15k, Resistor_SMD:R_0402_1005Metric, F.Cu at (179.4, 291.5)
- added R269: 15k, Resistor_SMD:R_0402_1005Metric, F.Cu at (179.4, 293.5)
- added R27: 2k ½W, Resistor_SMD:R_1210_3225Metric, F.Cu at (97.6, 262.5)
- added R270: 15k, Resistor_SMD:R_0402_1005Metric, F.Cu at (179.4, 295.4)
- added R271: 15k, Resistor_SMD:R_0402_1005Metric, F.Cu at (179.4, 297.4)
- added R272: 15k, Resistor_SMD:R_0402_1005Metric, F.Cu at (179.4, 299.4)
- added R273: 15k, Resistor_SMD:R_0402_1005Metric, F.Cu at (179.4, 301.4)
- added R274: 15k, Resistor_SMD:R_0402_1005Metric, F.Cu at (179.4, 303.4)
- added R275: 15k, Resistor_SMD:R_0402_1005Metric, F.Cu at (182.3, 291.5)
- added R276: 15k, Resistor_SMD:R_0402_1005Metric, F.Cu at (182.3, 293.5)
- added R277: 15k, Resistor_SMD:R_0402_1005Metric, F.Cu at (182.3, 295.4)
- added R278: 15k, Resistor_SMD:R_0402_1005Metric, F.Cu at (182.3, 297.4)
- added R279: 15k, Resistor_SMD:R_0402_1005Metric, F.Cu at (182.3, 299.4)
- added R28: 300R 3W, Resistor_THT:R_Axial_DIN0516_L15.5mm_D5.0mm_P20.32mm_Horizontal, F.Cu at (120.0, 258.1)
- added R280: 15k, Resistor_SMD:R_0402_1005Metric, F.Cu at (182.3, 301.4)
- added R281: 15k, Resistor_SMD:R_0402_1005Metric, F.Cu at (182.3, 303.4)
- added R282: 15k, Resistor_SMD:R_0402_1005Metric, F.Cu at (185.2, 291.5)
- added R283: 15k, Resistor_SMD:R_0402_1005Metric, F.Cu at (185.2, 293.5)
- added R284: 15k, Resistor_SMD:R_0402_1005Metric, F.Cu at (158.6, 261.5)
- added R285: 15k, Resistor_SMD:R_0402_1005Metric, F.Cu at (158.6, 263.5)
- added R286: 15k, Resistor_SMD:R_0402_1005Metric, F.Cu at (158.6, 265.5)
- added R287: 15k, Resistor_SMD:R_0402_1005Metric, F.Cu at (161.5, 255.5)
- added R288: 15k, Resistor_SMD:R_0402_1005Metric, F.Cu at (161.5, 257.5)
- added R289: 15k, Resistor_SMD:R_0402_1005Metric, F.Cu at (161.5, 259.5)
- added R29: 56k, Resistor_SMD:R_0402_1005Metric, F.Cu at (96.2, 235.1)
- added R290: 15k, Resistor_SMD:R_0402_1005Metric, F.Cu at (161.5, 261.5)
- added R291: 15k, Resistor_SMD:R_0402_1005Metric, F.Cu at (161.5, 263.5)
- added R292: 2k4, Resistor_SMD:R_0402_1005Metric, F.Cu at (161.5, 265.5)
- added R293: 15k, Resistor_SMD:R_0402_1005Metric, F.Cu at (164.4, 255.5)
- added R294: 15k, Resistor_SMD:R_0402_1005Metric, F.Cu at (164.4, 257.5)
- added R295: 15k, Resistor_SMD:R_0402_1005Metric, F.Cu at (164.4, 259.5)
- added R296: 15k, Resistor_SMD:R_0402_1005Metric, F.Cu at (164.4, 261.5)
- added R297: 15k, Resistor_SMD:R_0402_1005Metric, F.Cu at (164.4, 263.5)
- added R298: 15k, Resistor_SMD:R_0402_1005Metric, F.Cu at (164.4, 265.5)
- added R299: 15k, Resistor_SMD:R_0402_1005Metric, F.Cu at (167.3, 255.5)
- added R3: 56k, Resistor_SMD:R_0402_1005Metric, F.Cu at (154.8, 331.2)
- added R30: 2k ½W, Resistor_SMD:R_1210_3225Metric, F.Cu at (97.6, 266.7)
- added R300: 15k, Resistor_SMD:R_0402_1005Metric, F.Cu at (167.3, 257.5)
- added R301: 15k, Resistor_SMD:R_0402_1005Metric, F.Cu at (167.3, 259.5)
- added R302: 15k, Resistor_SMD:R_0402_1005Metric, F.Cu at (167.3, 261.5)
- added R303: 300R 3W, Resistor_THT:R_Axial_DIN0516_L15.5mm_D5.0mm_P20.32mm_Horizontal, F.Cu at (146.3, 231.4)
- added R304: 15k, Resistor_SMD:R_0402_1005Metric, F.Cu at (167.3, 263.5)
- added R305: 2k4, Resistor_SMD:R_0402_1005Metric, F.Cu at (167.3, 265.5)
- added R306: 2k4 ¼W, Resistor_SMD:R_0603_1608Metric, F.Cu at (170.6, 229.4)
- added R307: 2k4 ¼W, Resistor_SMD:R_0603_1608Metric, F.Cu at (170.6, 231.9)
- added R308: 15k, Resistor_SMD:R_0402_1005Metric, F.Cu at (185.2, 295.4)
- added R309: 15k, Resistor_SMD:R_0402_1005Metric, F.Cu at (185.2, 297.4)
- added R31: 56k, Resistor_SMD:R_0402_1005Metric, F.Cu at (96.2, 237.1)
- added R310: 15k, Resistor_SMD:R_0402_1005Metric, F.Cu at (185.2, 299.4)
- added R311: 15k, Resistor_SMD:R_0402_1005Metric, F.Cu at (185.2, 301.4)
- added R312: 15k, Resistor_SMD:R_0402_1005Metric, F.Cu at (185.2, 303.4)
- added R313: 6k8, Resistor_SMD:R_0402_1005Metric, F.Cu at (113.0, 316.1)
- added R314: 6k8, Resistor_SMD:R_0402_1005Metric, F.Cu at (113.0, 318.1)
- added R315: 6k8, Resistor_SMD:R_0402_1005Metric, F.Cu at (113.0, 320.1)
- added R316: 6k8, Resistor_SMD:R_0402_1005Metric, F.Cu at (113.0, 322.1)
- added R317: 6k8, Resistor_SMD:R_0402_1005Metric, F.Cu at (113.0, 324.1)
- added R318: 15k, Resistor_SMD:R_0402_1005Metric, F.Cu at (113.0, 326.0)
- added R319: 15k, Resistor_SMD:R_0402_1005Metric, F.Cu at (113.0, 328.0)
- added R32: 2k ½W, Resistor_SMD:R_1210_3225Metric, F.Cu at (103.2, 254.1)
- added R320: 15k, Resistor_SMD:R_0402_1005Metric, F.Cu at (113.0, 330.0)
- added R321: 15k, Resistor_SMD:R_0402_1005Metric, F.Cu at (113.0, 332.0)
- added R322: 15k, Resistor_SMD:R_0402_1005Metric, F.Cu at (113.0, 334.0)
- added R323: 15k, Resistor_SMD:R_0402_1005Metric, F.Cu at (115.9, 316.1)
- added R324: 15k, Resistor_SMD:R_0402_1005Metric, F.Cu at (115.9, 318.1)
- added R325: 15k, Resistor_SMD:R_0402_1005Metric, F.Cu at (115.9, 320.1)
- added R326: 15k, Resistor_SMD:R_0402_1005Metric, F.Cu at (115.9, 322.1)
- added R327: 15k, Resistor_SMD:R_0402_1005Metric, F.Cu at (115.9, 324.1)
- added R328: 15k, Resistor_SMD:R_0402_1005Metric, F.Cu at (115.9, 326.0)
- added R329: 15k, Resistor_SMD:R_0402_1005Metric, F.Cu at (115.9, 328.0)
- added R33: 15k, Resistor_SMD:R_0402_1005Metric, F.Cu at (157.7, 333.2)
- added R330: 15k, Resistor_SMD:R_0402_1005Metric, F.Cu at (115.9, 330.0)
- added R331: 15k, Resistor_SMD:R_0402_1005Metric, F.Cu at (115.9, 332.0)
- added R332: 15k, Resistor_SMD:R_0402_1005Metric, F.Cu at (115.9, 334.0)
- added R333: 15k, Resistor_SMD:R_0402_1005Metric, F.Cu at (118.9, 316.1)
- added R334: 15k, Resistor_SMD:R_0402_1005Metric, F.Cu at (118.9, 318.1)
- added R335: 15k, Resistor_SMD:R_0402_1005Metric, F.Cu at (118.9, 320.1)
- added R336: 15k, Resistor_SMD:R_0402_1005Metric, F.Cu at (118.9, 322.1)
- added R337: 15k, Resistor_SMD:R_0402_1005Metric, F.Cu at (118.9, 324.1)
- added R338: 15k, Resistor_SMD:R_0402_1005Metric, F.Cu at (118.9, 326.0)
- added R339: 15k, Resistor_SMD:R_0402_1005Metric, F.Cu at (118.9, 328.0)
- added R34: 15k, Resistor_SMD:R_0402_1005Metric, F.Cu at (157.7, 335.2)
- added R340: 15k, Resistor_SMD:R_0402_1005Metric, F.Cu at (118.9, 330.0)
- added R341: 15k, Resistor_SMD:R_0402_1005Metric, F.Cu at (118.9, 332.0)
- added R342: 15k, Resistor_SMD:R_0402_1005Metric, F.Cu at (118.9, 334.0)
- added R343: 15k, Resistor_SMD:R_0402_1005Metric, F.Cu at (121.8, 316.1)
- added R344: 15k, Resistor_SMD:R_0402_1005Metric, F.Cu at (121.8, 318.1)
- added R345: 6k8, Resistor_SMD:R_0402_1005Metric, F.Cu at (124.7, 303.4)
- added R346: 6k8, Resistor_SMD:R_0402_1005Metric, F.Cu at (124.7, 305.4)
- added R347: 6k8, Resistor_SMD:R_0402_1005Metric, F.Cu at (124.7, 307.4)
- added R348: 10k ½W, Resistor_SMD:R_1210_3225Metric, F.Cu at (97.6, 317.2)
- added R349: 33k, Resistor_SMD:R_0402_1005Metric, F.Cu at (121.8, 320.1)
- added R35: 15k, Resistor_SMD:R_0402_1005Metric, F.Cu at (157.7, 337.2)
- added R350: 2k ½W, Resistor_SMD:R_1210_3225Metric, F.Cu at (97.6, 321.4)
- added R351: 10k ½W, Resistor_SMD:R_1210_3225Metric, F.Cu at (97.6, 325.6)
- added R352: 33k, Resistor_SMD:R_0402_1005Metric, F.Cu at (121.8, 322.1)
- added R353: 10k ½W, Resistor_SMD:R_1210_3225Metric, F.Cu at (97.6, 329.8)
- added R354: 33k, Resistor_SMD:R_0402_1005Metric, F.Cu at (121.8, 324.1)
- added R355: 10k ½W, Resistor_SMD:R_1210_3225Metric, F.Cu at (97.6, 334.0)
- added R356: 33k, Resistor_SMD:R_0402_1005Metric, F.Cu at (121.8, 326.0)
- added R357: 33k, Resistor_SMD:R_0402_1005Metric, F.Cu at (121.8, 328.0)
- added R358: 800R 2W, Resistor_THT:R_Axial_DIN0516_L15.5mm_D5.0mm_P20.32mm_Horizontal, F.Cu at (113.6, 338.3)
- added R359: 56k, Resistor_SMD:R_0402_1005Metric, F.Cu at (121.8, 330.0)
- added R36: 15k, Resistor_SMD:R_0402_1005Metric, F.Cu at (157.7, 339.1)
- added R360: 2k ½W, Resistor_SMD:R_1210_3225Metric, F.Cu at (103.2, 317.2)
- added R361: 56k, Resistor_SMD:R_0402_1005Metric, F.Cu at (121.8, 332.0)
- added R362: 2k ½W, Resistor_SMD:R_1210_3225Metric, F.Cu at (103.2, 321.4)
- added R363: 56k, Resistor_SMD:R_0402_1005Metric, F.Cu at (121.8, 334.0)
- added R364: 2k ½W, Resistor_SMD:R_1210_3225Metric, F.Cu at (103.2, 325.6)
- added R365: 56k, Resistor_SMD:R_0402_1005Metric, F.Cu at (124.7, 316.1)
- added R366: 2k ½W, Resistor_SMD:R_1210_3225Metric, F.Cu at (103.2, 329.8)
- added R367: 56k, Resistor_SMD:R_0402_1005Metric, F.Cu at (124.7, 318.1)
- added R368: 2k ½W, Resistor_SMD:R_1210_3225Metric, F.Cu at (103.2, 334.0)
- added R369: 56k, Resistor_SMD:R_0402_1005Metric, F.Cu at (124.7, 320.1)
- added R37: 15k, Resistor_SMD:R_0402_1005Metric, F.Cu at (157.7, 341.1)
- added R370: 2k ½W, Resistor_SMD:R_1210_3225Metric, F.Cu at (108.8, 317.2)
- added R371: 56k, Resistor_SMD:R_0402_1005Metric, F.Cu at (124.7, 322.1)
- added R372: 2k ½W, Resistor_SMD:R_1210_3225Metric, F.Cu at (108.8, 321.4)
- added R373: 56k, Resistor_SMD:R_0402_1005Metric, F.Cu at (124.7, 324.1)
- added R374: 2k ½W, Resistor_SMD:R_1210_3225Metric, F.Cu at (108.8, 325.6)
- added R375: 10k ½W, Resistor_SMD:R_1210_3225Metric, F.Cu at (108.8, 301.0)
- added R376: 33k, Resistor_SMD:R_0402_1005Metric, F.Cu at (124.7, 309.4)
- added R377: 800R 2W, Resistor_THT:R_Axial_DIN0516_L15.5mm_D5.0mm_P20.32mm_Horizontal, F.Cu at (96.7, 274.1)
- added R378: 10k ½W, Resistor_SMD:R_1210_3225Metric, F.Cu at (108.8, 305.2)
- added R379: 33k, Resistor_SMD:R_0402_1005Metric, F.Cu at (127.6, 291.5)
- added R38: 15k, Resistor_SMD:R_0402_1005Metric, F.Cu at (157.7, 343.1)
- added R380: 33k, Resistor_SMD:R_0402_1005Metric, F.Cu at (127.6, 293.5)
- added R381: 800R 2W, Resistor_THT:R_Axial_DIN0516_L15.5mm_D5.0mm_P20.32mm_Horizontal, F.Cu at (96.7, 280.6)
- added R382: 300R 3W, Resistor_THT:R_Axial_DIN0516_L15.5mm_D5.0mm_P20.32mm_Horizontal, F.Cu at (96.7, 287.2)
- added R383: 300R 3W, Resistor_THT:R_Axial_DIN0516_L15.5mm_D5.0mm_P20.32mm_Horizontal, F.Cu at (146.3, 237.9)
- added R384: 300R 3W, Resistor_THT:R_Axial_DIN0516_L15.5mm_D5.0mm_P20.32mm_Horizontal, F.Cu at (120.0, 264.6)
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Connections:
- P1 pad A10: ~{rl} -> unconnected-(P1-~{r1}-PadA10)
- P1 pad A12: ~{P2c} -> unconnected-(P1-~{P2c}-PadA12)
- P1 pad A14: ~{P3c} -> unconnected-(P1-~{P3c}-PadA14)
- P1 pad A16: ~{P4c} -> unconnected-(P1-~{P4c}-PadA16)
- P1 pad A20: ~{P5c} -> unconnected-(P1-~{P5c}-PadA20)
- P1 pad A22: ~{V} -> unconnected-(P1-~{V}-PadA22)
- P1 pad A24: ~{P6c} -> unconnected-(P1-~{P6c}-PadA24)
- P1 pad A27: S2 -> unconnected-(P1-S2-PadA27)
- P1 pad A31: ~{Tb2} -> unconnected-(P1-~{Tb2}-PadA31)
- P1 pad A32: ~{Tb1} -> unconnected-(P1-~{Tb1}-PadA32)
- P1 pad A34: ~{Tb3} -> unconnected-(P1-~{Tb3}-PadA34)
- P1 pad A35: ~{Tb4} -> unconnected-(P1-~{Tb4}-PadA35)
- P1 pad A36: Tc -> unconnected-(P1-Tc-PadA36)
- P1 pad A38: Q1b -> unconnected-(P1-Q1b-PadA38)
- P1 pad A39: ~{Q1d} -> unconnected-(P1-~{Q1d}-PadA39)
- P1 pad A40: ~{Q2a} -> unconnected-(P1-Q2a-PadA40)
- P1 pad A41: ~{O1} -> unconnected-(P1-~{O1}-PadA41)
- P1 pad A43: ~{Q2c} -> unconnected-(P1-~{Q2c}-PadA43)
- P1 pad A44: O1 -> unconnected-(P1-O1-PadA44)
- P1 pad A45: ~{Q2d} -> unconnected-(P1-~{Q2d}-PadA45)
- P1 pad A46: ~{S1} -> unconnected-(P1-~{S1}-PadA46)
- P1 pad A48: ~{P2} -> unconnected-(P1-~{P2}-PadA48)
- P1 pad A49: ~{P3} -> unconnected-(P1-~{P3}-PadA49)
- P1 pad A52: ~{P4} -> unconnected-(P1-~{P4}-PadA52)
- P1 pad A55: ~{P5} -> unconnected-(P1-~{P5}-PadA55)
- P1 pad A56: unconnected-(P1-W-PadA56) -> W
- P1 pad A60: unconnected-(P1-~{W}-PadA60) -> ~{W}
- P1 pad A8: rl -> unconnected-(P1-r1-PadA8)
- P1 pad A9: ~{P1c} -> unconnected-(P1-~{P1c}-PadA9)
- P1 pad B10: unconnected-(P1-Gb-PadB10) -> Gb
- P1 pad B11: unconnected-(P1-~{Gd}-PadB11) -> ~{Gd}
- P1 pad B13: ~{A} -> unconnected-(P1-~{A}-PadB13)
- P1 pad B14: A* -> unconnected-(P1-A*-PadB14)
- P1 pad B15: ~{A*} -> unconnected-(P1-~{A*}-PadB15)
- P1 pad B18: unconnected-(P1-~{T3}-PadB18) -> ~{T3}
- P1 pad B19: P5 -> unconnected-(P1-P5-PadB19)
- P1 pad B20: unconnected-(P1-~{brc}-PadB20) -> ~{brc}
- P1 pad B22: unconnected-(P1-~{be}-PadB22) -> ~{be}
- P1 pad B23: unconnected-(P1-brc-PadB23) -> brc
- P1 pad B24: unconnected-(P1-~{Ac1}-PadB24) -> ~{Ac1}
- P1 pad B29: P2 -> unconnected-(P1-P2-PadB29)
- P1 pad B3: unconnected-(P1-Fa-PadB3) -> Fa
- P1 pad B30: bs -> unconnected-(P1-bs-PadB30)
- P1 pad B32: P3 -> unconnected-(P1-P3-PadB32)
- P1 pad B35: unconnected-(P1-~{K}-PadB35) -> ~{K}
- P1 pad B36: unconnected-(P1-K'-PadB36) -> K'
- P1 pad B38: unconnected-(P1-C-PadB38) -> C
- P1 pad B39: B1 -> Bl
- P1 pad B4: unconnected-(P1-~{Fc}-PadB4) -> ~{Fc}
- P1 pad B45: ~{P6} -> unconnected-(P1-~{P6}-PadB45)
- P1 pad B49: ~{To} -> unconnected-(P1-~{To}-PadB49)
- P1 pad B5: unconnected-(P1-Fb-PadB5) -> Fb
- P1 pad B53: unconnected-(P1-S1-PadB53) -> S1
- P1 pad B54: unconnected-(P1-Vw'-PadB54) -> Vw'
- P1 pad B55: unconnected-(P1-Rw'-PadB55) -> Rw'
- P1 pad B57: unconnected-(P1-~{L}-PadB57) -> ~{L}
- P1 pad B59: unconnected-(P1-Kc-PadB59) -> Kc
- P1 pad B6: unconnected-(P1-~{Fd}-PadB6) -> ~{Fd}
- P1 pad B7: unconnected-(P1-Ga-PadB7) -> Ga
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
Commit message: Rough layout for Phase Control.
Parts:
- CR1, CR10, CR11, CR12, CR13, CR16, CR17, CR18, CR2, CR20, CR21, CR22, CR23, CR24, CR25, CR26, CR27, CR28, CR29, CR3, CR30, CR31, CR32, CR33, CR34, CR35, CR36, CR37, CR38, CR39, CR4, CR40, CR41, CR42, CR43, CR44, CR45, CR46, CR47, CR48, CR49, CR5, CR50, CR51, CR52, CR53, CR54, CR55, CR56, CR57, CR58, CR59, CR6, CR60, CR7, CR8, CR9, CR90, CR91, CR92, CR93: value 1N5819WS -> 1N4148WS
- moved Q65 278.1 mm to (179.3, 90.4)
- moved Q12 271.1 mm to (87.4, 106.6), turned to 180 degrees
- moved C18 265.0 mm to (174.5, 89.9), turned to -90 degrees
- moved Q70 259.2 mm to (179.3, 108.7)
- moved Q69 258.4 mm to (179.3, 105.2)
- moved Q68 257.5 mm to (179.3, 101.6)
- moved Q67 256.7 mm to (179.3, 98.0)
- moved Q11 256.1 mm to (87.4, 110.2), turned to 180 degrees
- moved Q66 255.8 mm to (179.3, 94.5)
- moved CR8 252.8 mm to (90.4, 106.6), turned to -90 degrees
- moved CR7 249.3 mm to (92.5, 106.6), turned to -90 degrees
- moved R70 246.8 mm to (91.2, 119.6)
- moved R350 246.7 mm to (184.2, 90.4), turned to 180 degrees
- moved R357 246.6 mm to (181.1, 88.6), turned to 90 degrees
- moved CR6 245.8 mm to (94.5, 106.6), turned to -90 degrees
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Connections:
- net Net-(Q10-C) renamed /F Flip-Flop/~{F_{S}}
- net Net-(Q12-B) renamed /F Flip-Flop/F_{S}
- net Net-(Q24-C) renamed /G Flip-Flop/G_{S}
- net Net-(Q25-C) renamed /G Flip-Flop/~{G_{S}}
- net Net-(Q55-C) renamed /H Flip-Flop/H_{S}
- net Net-(Q56-C) renamed /H Flip-Flop/~{H_{S}}
- P1 pad A10: unconnected-(P1-~{r1}-PadA10) -> ~{r1}
- P1 pad A8: unconnected-(P1-r1-PadA8) -> r1
- Q38 pad 3: rl -> r1
- Q39 pad 3: ~{rl} -> ~{r1}
- R181 pad 1: rl -> r1
- R223 pad 2: rl -> r1
- R225 pad 2: ~{rl} -> ~{r1}
Routing:
- net +15V: track 0.00 -> 745.8 mm, vias 0 -> 6
- net GND: track 0.00 -> 608.6 mm, vias 0 -> 66
- net -20V: track 0.00 -> 330.7 mm, vias 0 -> 2
- net Net-(Q18-B): track 0.00 -> 17.1 mm
- net Net-(CR2-K): track 0.00 -> 15.4 mm
- net Net-(CR56-K): track 0.00 -> 13.9 mm
- net Net-(Q22-B): track 0.00 -> 12.3 mm
- net /F Flip-Flop/~{F_{S}}: track 0.00 -> 12.2 mm, vias 0 -> 2
- net /G Flip-Flop/~{G_{S}}: track 0.00 -> 12.2 mm, vias 0 -> 2
- net /H Flip-Flop/~{H_{S}}: track 0.00 -> 12.2 mm, vias 0 -> 2
- net Net-(Q20-B): track 0.00 -> 11.6 mm
- net Net-(Q31-B): track 0.00 -> 11.2 mm
- net Net-(Q20-C): track 0.00 -> 10.5 mm
- net Net-(Q21-C): track 0.00 -> 9.98 mm
- net Net-(Q33-B): track 0.00 -> 9.23 mm
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- added copper zone on F.Cu, net -20V
Other:
- board text added: "F"
- board text added: "G"
- board text added: "~{F}"
- board text added: "~{G}"
