File: boards/phase-control/phase-control.kicad_sch (KiCad schematic)
At the start: 77 parts, among them P1 Card Edge, Q40 MMBT5401, Q41 MMBT5401, Q42 MMBT5401, Q43 MMBT5401, Q44 MMBT5401, Q45 MMBT5401, Q46 MMBT5401, Q47 MMBT5401, Q48 MMBT5401, Q49 MMBT5401, Q59 MMBT5401, Q60 MMBT5401

Commit message: Create diode coupled inverter block.
Parts:
- R229: value 2k -> 2k ⅛W; footprint (none) -> Resistor_SMD:R_0805_2012Metric
- renumbered CR17 to CR90, CR18 to CR91, CR19 to CR92
Changed lines of the file:
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@@
 		(in_pos_files yes)
 		(dnp no)
-		(property "Reference" "CR18"
+		(property "Reference" "CR91"
 			(at 244.602 48.26 90)
 			(show_name no)
@@
 			(project "phase-control"
 				(path "/d5da316c-1ec9-4d99-8330-1c4a3f6c3ba4"
-					(reference "CR18")
+					(reference "CR91")
 					(unit 1)
 				)
@@
 			)
 		)
-		(property "Value" "2k"
+		(property "Value" "2k ⅛W"
 			(at 146.304 39.37 0)
 			(show_name no)
@@
 			)
 		)
-		(property "Footprint" ""
+		(property "Footprint" "Resistor_SMD:R_0805_2012Metric"
 			(at 145.796 38.354 90)
 			(hide yes)
@@
 		(in_pos_files yes)
 		(dnp no)
-		(property "Reference" "CR17"
+		(property "Reference" "CR90"
 			(at 244.348 57.15 90)
 			(show_name no)
@@
 			(project "phase-control"
 				(path "/d5da316c-1ec9-4d99-8330-1c4a3f6c3ba4"
-					(reference "CR17")
+					(reference "CR90")
 					(unit 1)
 				)
@@
 		(in_pos_files yes)
 		(dnp no)
-		(property "Reference" "CR19"
+		(property "Reference" "CR92"
 			(at 244.348 43.18 90)
 			(show_name no)
@@
 			(project "phase-control"
 				(path "/d5da316c-1ec9-4d99-8330-1c4a3f6c3ba4"
-					(reference "CR19")
+					(reference "CR92")
 					(unit 1)
 				)

Commit message: Start the Phase Control board.
Parts:
- Q40, Q41, Q42, Q43, Q44, Q45, Q46, Q47, Q48, Q49, Q59, Q60: symbol Transistor_BJT:Q_PNP_EBC -> Transistor_BJT:Q_PNP_BEC
Connections:
- net CP: now also Q42.1 (B); no longer Q42.2 (B)
- net GND: now also Q40.2 (E), Q41.2 (E), Q43.2 (E), Q44.2 (E), Q46.2 (E), Q47.2 (E), Q48.2 (E), Q49.2 (E), Q59.2 (E), Q60.2 (E); no longer Q40.1 (E), Q41.1 (E), Q43.1 (E), Q44.1 (E), Q46.1 (E), Q47.1 (E), Q48.1 (E), Q49.1 (E), Q59.1 (E), Q60.1 (E)
- net at R239.1, R271.2, R279.2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: now also Q48.1 (B); no longer Q48.2 (B)
- net at C9.1, R184.1: now also Q42.2 (E); no longer Q42.1 (E)
- net at R235.1, R264.2, R265.2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: now also Q46.1 (B); no longer Q46.2 (B)
- net at R257.1, R308.2: now also Q59.1 (B); no longer Q59.2 (B)
- net at R259.1, R310.2, R311.2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: now also Q60.1 (B); no longer Q60.2 (B)
- net at R182.2, R183.2, R226.1: now also Q40.1 (B); no longer Q40.2 (B)
- net at R232.1, R263.2: now also Q44.1 (B); no longer Q44.2 (B)
- net at R230.1, R261.2, R262.2: now also Q43.1 (B); no longer Q43.2 (B)
- net at R237.1, R272.2, R273.2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: now also Q47.1 (B); no longer Q47.2 (B)
- net at C9.2, R184.2, R228.1: now also Q41.1 (B); no longer Q41.2 (B)
- net at R241.1, R282.2, R283.2: now also Q49.1 (B); no longer Q49.2 (B)
- net at CR92.1 (K): now also Q45.2 (E); no longer Q45.1 (E)
- net at Q44.3 (C), R233.2: now also Q45.1 (B); no longer Q45.2 (B)
Changed lines of the file:
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@@
 	)
 	(symbol
-		(lib_id "Transistor_BJT:Q_PNP_EBC")
+		(lib_id "Transistor_BJT:Q_PNP_BEC")
 		(at 110.49 31.75 0)
 		(unit 1)
@@
 			)
 		)
-		(property "Description" "Germanium PNP Transistor"
+		(property "Description" "PNP BJT"
 			(at 110.49 31.75 0)
 			(hide yes)
@@
 			)
 		)
-		(property "Sim.Pins" "1=E 2=B 3=C"
+		(property "Sim.Pins" "1=B 2=E 3=C"
 			(at 110.49 31.75 0)
 			(hide yes)
@@
 	)
 	(symbol
-		(lib_id "Transistor_BJT:Q_PNP_EBC")
+		(lib_id "Transistor_BJT:Q_PNP_BEC")
 		(at 218.44 91.44 0)
 		(unit 1)
@@
 			)
 		)
-		(property "Description" "Germanium PNP Transistor"
+		(property "Description" "PNP BJT"
 			(at 218.44 91.44 0)
 			(hide yes)
@@
 			)
 		)
-		(property "Sim.Pins" "1=E 2=B 3=C"
+		(property "Sim.Pins" "1=B 2=E 3=C"
 			(at 218.44 91.44 0)
 			(hide yes)
@@
 	)
 	(symbol
-		(lib_id "Transistor_BJT:Q_PNP_EBC")
+		(lib_id "Transistor_BJT:Q_PNP_BEC")
 		(at 204.47 175.26 0)
 		(unit 1)
@@
 			)
 		)
-		(property "Description" "Germanium PNP Transistor"
+		(property "Description" "PNP BJT"
 			(at 204.47 175.26 0)
 			(hide yes)
@@
 			)
 		)
-		(property "Sim.Pins" "1=E 2=B 3=C"
+		(property "Sim.Pins" "1=B 2=E 3=C"
 			(at 204.47 175.26 0)
 			(hide yes)
@@
 	)
 	(symbol
-		(lib_id "Transistor_BJT:Q_PNP_EBC")
+		(lib_id "Transistor_BJT:Q_PNP_BEC")
 		(at 134.62 91.44 0)
 		(unit 1)
@@
 			)
 		)
-		(property "Description" "Germanium PNP Transistor"
+		(property "Description" "PNP BJT"
 			(at 134.62 91.44 0)
 			(hide yes)
@@
 			)
 		)
-		(property "Sim.Pins" "1=E 2=B 3=C"
+		(property "Sim.Pins" "1=B 2=E 3=C"
 			(at 134.62 91.44 0)
 			(hide yes)
@@
 	)
 	(symbol
-		(lib_id "Transistor_BJT:Q_PNP_EBC")
+		(lib_id "Transistor_BJT:Q_PNP_BEC")
 		(at 184.15 135.89 0)
 		(unit 1)
@@
 			)
 		)
-		(property "Description" "Germanium PNP Transistor"
+		(property "Description" "PNP BJT"
 			(at 184.15 135.89 0)
 			(hide yes)
@@
 			)
 		)
-		(property "Sim.Pins" "1=E 2=B 3=C"
+		(property "Sim.Pins" "1=B 2=E 3=C"
 			(at 184.15 135.89 0)
 			(hide yes)
@@
 	)
 	(symbol
-		(lib_id "Transistor_BJT:Q_PNP_EBC")
+		(lib_id "Transistor_BJT:Q_PNP_BEC")
 		(at 189.23 48.26 0)
 		(unit 1)
@@
 			)
 		)
-		(property "Description" "Germanium PNP Transistor"
+		(property "Description" "PNP BJT"
 			(at 189.23 48.26 0)
 			(hide yes)
@@
 			)
 		)
-		(property "Sim.Pins" "1=E 2=B 3=C"
+		(property "Sim.Pins" "1=B 2=E 3=C"
 			(at 189.23 48.26 0)
 			(hide yes)
@@
 	)
 	(symbol
-		(lib_id "Transistor_BJT:Q_PNP_EBC")
+		(lib_id "Transistor_BJT:Q_PNP_BEC")
 		(at 226.06 132.08 0)
 		(unit 1)
@@
 			)
 		)
-		(property "Description" "Germanium PNP Transistor"
+		(property "Description" "PNP BJT"
 			(at 226.06 132.08 0)
 			(hide yes)
@@
 			)
 		)
-		(property "Sim.Pins" "1=E 2=B 3=C"
+		(property "Sim.Pins" "1=B 2=E 3=C"
 			(at 226.06 132.08 0)
 			(hide yes)
@@
 	)
 	(symbol
-		(lib_id "Transistor_BJT:Q_PNP_EBC")
+		(lib_id "Transistor_BJT:Q_PNP_BEC")
 		(at 134.62 134.62 0)
 		(unit 1)
@@
 			)
 		)
-		(property "Description" "Germanium PNP Transistor"
+		(property "Description" "PNP BJT"
 			(at 134.62 134.62 0)
 			(hide yes)
@@
 			)
 		)
-		(property "Sim.Pins" "1=E 2=B 3=C"
+		(property "Sim.Pins" "1=B 2=E 3=C"
 			(at 134.62 134.62 0)
 			(hide yes)
@@
 	)
 	(symbol
-		(lib_id "Transistor_BJT:Q_PNP_EBC")
+		(lib_id "Transistor_BJT:Q_PNP_BEC")
 		(at 240.03 35.56 0)
 		(unit 1)
@@
 			)
 		)
-		(property "Description" "Germanium PNP Transistor"
+		(property "Description" "PNP BJT"
 			(at 240.03 35.56 0)
 			(hide yes)
@@
 			)
 		)
-		(property "Sim.Pins" "1=E 2=B 3=C"
+		(property "Sim.Pins" "1=B 2=E 3=C"
 			(at 240.03 35.56 0)
 			(hide yes)
@@
 	)
 	(symbol
-		(lib_id "Transistor_BJT:Q_PNP_EBC")
+		(lib_id "Transistor_BJT:Q_PNP_BEC")
 		(at 134.62 173.99 0)
 		(unit 1)
@@
 			)
 		)
-		(property "Description" "Germanium PNP Transistor"
+		(property "Description" "PNP BJT"
 			(at 134.62 173.99 0)
 			(hide yes)
@@
 			)
 		)
-		(property "Sim.Pins" "1=E 2=B 3=C"
+		(property "Sim.Pins" "1=B 2=E 3=C"
 			(at 134.62 173.99 0)
 			(hide yes)
@@
 	)
 	(symbol
-		(lib_id "Transistor_BJT:Q_PNP_EBC")
+		(lib_id "Transistor_BJT:Q_PNP_BEC")
 		(at 132.08 39.37 0)
 		(unit 1)
@@
 			)
 		)
-		(property "Description" "Germanium PNP Transistor"
+		(property "Description" "PNP BJT"
 			(at 132.08 39.37 0)
 			(hide yes)
@@
 			)
 		)
-		(property "Sim.Pins" "1=E 2=B 3=C"
+		(property "Sim.Pins" "1=B 2=E 3=C"
 			(at 132.08 39.37 0)
 			(hide yes)
@@
 	)
 	(symbol
-		(lib_id "Transistor_BJT:Q_PNP_EBC")
+		(lib_id "Transistor_BJT:Q_PNP_BEC")
 		(at 223.52 41.91 0)
 		(unit 1)
@@
 			)
 		)
-		(property "Description" "Germanium PNP Transistor"
+		(property "Description" "PNP BJT"
 			(at 223.52 41.91 0)
 			(hide yes)
@@
 			)
 		)
-		(property "Sim.Pins" "1=E 2=B 3=C"
+		(property "Sim.Pins" "1=B 2=E 3=C"
 			(at 223.52 41.91 0)
 			(hide yes)

Commit message: Add script to export production files.
Parts:
- C9: BOM Value (none) -> 680pF
- CR28, CR29, CR56, CR57, CR58, CR59, CR60, CR90, CR91, CR92: value 1N5819WS -> 1N4148WS; BOM Value (none) -> 1N4148WS; LCSC (none) -> C2128
- P1: now left out of the parts list
- Q40, Q41, Q42, Q43, Q44, Q45, Q46, Q47, Q48, Q49, Q59, Q60: BOM Value (none) -> MMBT5401; LCSC (none) -> C8326
- R182, R183, R261, R262, R263, R264, R265, R266, R267, R268, R269, R270, R271, R272, R273, R274, R275, R276, R277, R278, R279, R280, R281, R282, R283, R308, R309, R310, R311, R312: BOM Value (none) -> 15kΩ
- R184: BOM Value (none) -> 6.8kΩ
- R185: BOM Value (none) -> 450Ω 2W
- R226, R228, R230, R232, R234, R235, R237, R239, R241, R257, R259: BOM Value (none) -> 56kΩ
- R227, R258: BOM Value (none) -> 800Ω 2W
- R229: BOM Value (none) -> 2kΩ 125mW
- R231, R233, R236, R238, R240, R242, R260: BOM Value (none) -> 2kΩ 500mW

Commit message: Rough layout for Phase Control.
Connections:
- net ~{r1}: now reaches P1.A10 (~{r1})
- net r1: now reaches P1.A8 (r1)
- no-connect marks 46 -> 44
Changed lines of the file:
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@@
 	)
 	(no_connect
-		(at 66.04 165.1)
-	)
-	(no_connect
 		(at 38.1 109.22)
 	)
@@
 		(at 66.04 78.74)
 	)
-	(no_connect
-		(at 66.04 160.02)
-	)
 	(wire
 		(pts
@@
 	(wire
 		(pts
-			(xy 62.23 165.1) (xy 66.04 165.1)
+			(xy 62.23 165.1) (xy 73.66 165.1)
 		)
 		(stroke
@@
 	(wire
 		(pts
-			(xy 62.23 160.02) (xy 66.04 160.02)
+			(xy 62.23 160.02) (xy 73.66 160.02)
 		)
 		(stroke
@@
 		)
 	)
+	(global_label "~{r1}"
+		(shape input)
+		(at 73.66 160.02 0)
+		(fields_autoplaced yes)
+		(effects
+			(font
+				(size 1.27 1.27)
+			)
+			(justify left)
+		)
+		(property "Intersheetrefs" "${INTERSHEET_REFS}"
+			(at 78.6409 160.02 0)
+			(show_name no)
+			(do_not_autoplace no)
+			(effects
+				(font
+					(size 1.27 1.27)
+				)
+				(justify left)
+			)
+		)
+	)
 	(global_label "Bl"
 		(shape output)
@@
 			(show_name no)
 			(do_not_autoplace no)
+			(effects
+				(font
+					(size 1.27 1.27)
+				)
+				(justify left)
+			)
+		)
+	)
+	(global_label "r1"
+		(shape input)
+		(at 73.66 165.1 0)
+		(fields_autoplaced yes)
+		(effects
+			(font
+				(size 1.27 1.27)
+			)
+			(justify left)
+		)
+		(property "Intersheetrefs" "${INTERSHEET_REFS}"
+			(at 78.6409 165.1 0)
+			(show_name no)
+			(do_not_autoplace no)
