File: boards/phase-control/terms.kicad_sch (KiCad schematic)
At the start: 105 parts, among them Q28 MMBT5401, Q29 MMBT5401, Q30 MMBT5401, Q31 MMBT5401, Q32 MMBT5401, Q33 MMBT5401, Q34 MMBT5401, Q35 MMBT5401, Q36 MMBT5401, Q37 MMBT5401, Q38 MMBT5401, Q39 MMBT5401, Q74 MMBT5401, Q75 MMBT5401, Q76 MMBT5401, Q77 MMBT5401

Commit message: Create diode coupled inverter block.
Parts:
- R375, R378: value 10k -> 10k ½W; footprint (none) -> Resistor_SMD:R_1210_3225Metric
- gave numbers to parts that had none: 3
Changed lines of the file:
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@@
 	)
 	(junction
-		(at 171.45 185.42)
-		(diameter 0)
-		(color 0 0 0 0)
-	)
-	(junction
 		(at 156.21 66.04)
 		(diameter 0)
@@
 	)
 	(junction
+		(at 171.45 185.42)
+		(diameter 0)
+		(color 0 0 0 0)
+	)
+	(junction
 		(at 133.35 111.76)
 		(diameter 0)
@@
 	(wire
 		(pts
+			(xy 171.45 185.42) (xy 176.53 185.42)
+		)
+		(stroke
+			(width 0)
+			(type default)
+		)
+	)
+	(wire
+		(pts
 			(xy 196.85 157.48) (xy 199.39 157.48)
 		)
@@
 	(wire
 		(pts
-			(xy 166.37 185.42) (xy 171.45 185.42)
-		)
-		(stroke
-			(width 0)
-			(type default)
-		)
-	)
-	(wire
-		(pts
 			(xy 101.6 118.11) (xy 101.6 119.38)
 		)
@@
 	(wire
 		(pts
+			(xy 166.37 185.42) (xy 166.37 186.69)
+		)
+		(stroke
+			(width 0)
+			(type default)
+		)
+	)
+	(wire
+		(pts
 			(xy 100.33 30.48) (xy 165.1 30.48)
 		)
@@
 	(wire
 		(pts
-			(xy 176.53 185.42) (xy 171.45 185.42)
+			(xy 166.37 185.42) (xy 171.45 185.42)
 		)
 		(stroke
@@
 	(wire
 		(pts
+			(xy 171.45 185.42) (xy 171.45 187.96)
+		)
+		(stroke
+			(width 0)
+			(type default)
+		)
+	)
+	(wire
+		(pts
 			(xy 236.22 158.75) (xy 231.14 158.75)
 		)
@@
 	(wire
 		(pts
-			(xy 166.37 185.42) (xy 166.37 186.69)
-		)
-		(stroke
-			(width 0)
-			(type default)
-		)
-	)
-	(wire
-		(pts
 			(xy 102.87 77.47) (xy 104.14 77.47)
 		)
@@
 	(wire
 		(pts
-			(xy 171.45 187.96) (xy 171.45 185.42)
-		)
-		(stroke
-			(width 0)
-			(type default)
-		)
-	)
-	(wire
-		(pts
 			(xy 77.47 39.37) (xy 74.93 39.37)
 		)
@@
 		(in_pos_files yes)
 		(dnp no)
-		(property "Reference" "R?"
+		(property "Reference" "R900"
 			(at 164.846 189.23 0)
 			(show_name no)
@@
 			(project "phase-control"
 				(path "/d5da316c-1ec9-4d99-8330-1c4a3f6c3ba4/d8e0bdbb-d4a7-44ba-8f1b-a0e3a02bb0c0"
-					(reference "R?")
+					(reference "R900")
 					(unit 1)
 				)
@@
 		(in_pos_files yes)
 		(dnp no)
-		(property "Reference" "C?"
+		(property "Reference" "C900"
 			(at 173.228 189.23 0)
 			(show_name no)
@@
 			(project "phase-control"
 				(path "/d5da316c-1ec9-4d99-8330-1c4a3f6c3ba4/d8e0bdbb-d4a7-44ba-8f1b-a0e3a02bb0c0"
-					(reference "C?")
+					(reference "C900")
 					(unit 1)
 				)
@@
 			)
 		)
-		(property "Value" "10k"
+		(property "Value" "10k ½W"
 			(at 183.896 102.87 0)
 			(show_name no)
@@
 			)
 		)
-		(property "Footprint" ""
+		(property "Footprint" "Resistor_SMD:R_1210_3225Metric"
 			(at 186.436 101.854 90)
 			(hide yes)
@@
 		(in_pos_files yes)
 		(dnp no)
-		(property "Reference" "CR?"
+		(property "Reference" "CR93"
 			(at 180.34 182.88 0)
 			(show_name no)
@@
 			(project "phase-control"
 				(path "/d5da316c-1ec9-4d99-8330-1c4a3f6c3ba4/d8e0bdbb-d4a7-44ba-8f1b-a0e3a02bb0c0"
-					(reference "CR?")
+					(reference "CR93")
 					(unit 1)
 				)
@@
 			)
 		)
-		(property "Value" "10k"
+		(property "Value" "10k ½W"
 			(at 183.896 148.59 0)
 			(show_name no)
@@
 			)
 		)
-		(property "Footprint" ""
+		(property "Footprint" "Resistor_SMD:R_1210_3225Metric"
 			(at 186.436 147.574 90)
 			(hide yes)
@@
 	)
 	(group ""
+		(lib_id "Project:diode-inverter")
+		(members "0015785b-a96f-4629-bef5-14c4434ecc91" "001c58b1-5fad-4d05-9b5f-dfc400fed6bd"
+			"003cf61b-7fb0-4ccb-a1d1-e24ee09c34aa" "0d0cd723-e577-4989-8097-fd3607c05180"
+			"1cbbe984-6b4c-4725-889d-b4f6cb2f0631" "3837bbb7-d374-4a2a-9f2b-d9829e4f4417"
+			"5ebb3683-7a79-4834-bb01-30339c4f9f6a" "62ffe6df-854f-455a-8602-ecffd9d05146"
+			"6d2a2d7e-cb09-4530-8708-7e9d81e50db7" "82af8f89-ca36-474f-8b34-caa4324fef47"
+			"91c380ec-998b-43fd-b16e-077190f7eb0f" "991a20f2-3291-4596-8654-1209998c9cf2"
+			"9ce114b7-c480-41d6-b3f7-51ea0967ccf6" "a58becb9-0522-4d57-9ef4-065acd160d51"
+			"acc062ea-12bc-4af4-bf68-d959dbc2c6eb" "aea8e449-dac7-4747-a141-cdc66f638668"
+			"b0ff2f28-5417-4c5c-a0bf-5b3e8dbea5f7" "bae85d6a-3c01-4db5-ad18-0fbd03fc1c34"
+			"c1fb7815-dcad-42f1-a229-731183fe986c" "cf804a68-f03f-450d-9730-1b907b35a5ee"
+			"e208e9bb-ae7a-4fb3-a96a-a8925ab44a2e" "ff46b247-5bb3-48a4-bfab-e9de3dcfced4"
+		)
+	)
+	(group ""
 		(lib_id "Project:nor")
 		(members "0021ec18-a54d-41ec-ba31-7dca9c6eb146" "164e9b57-a37e-418d-8d84-000b6c8b5566"
@@
 	)
 	(group ""
+		(lib_id "Project:diode-inverter")
+		(members "01f5fa6c-9c7d-4a3c-8fd3-ee86d4faff37" "0402ba7e-63cb-4daa-8591-8e5c01a2d09f"
+			"0ba439b4-1b66-4cf0-813d-9f0f7b8b0e14" "0f8c5b0e-333f-4de5-8c99-7a37dcfcbf46"
+			"186dfb79-fb08-491c-971c-d81574c15170" "18ef2b66-51dd-415a-b0f4-575b8609fc2d"
+			"21916fc2-bbd2-42c8-9970-6c3747b93d87" "25355833-b0f8-4cef-9f08-a86bc465d14f"
+			"3875c930-a091-4822-b044-b09cf938d15c" "3d726489-a481-4590-9cb3-820198fbc4e6"
+			"3eb3937c-c043-43d1-a550-0fc3f0f07ccc" "458c2dbe-68ea-42e9-a8be-cb3c315bc79d"
+			"6e595713-1b9d-44be-b378-4863c4fa0cdb" "70750090-a3d2-42e8-b295-6f96d16bed95"
+			"7206b996-4368-450a-94bb-1459afe284bf" "86f45b42-26d6-4dd9-86a0-d574fc3b6d72"
+			"87ca36ed-7903-46cb-a3c8-20f9dc8d6bf3" "91f881f9-870c-48c9-8684-37b800228570"
+			"a57609e0-9e89-4993-a75e-bf6ff19d5f73" "b37d5b70-5eb0-463f-a706-dec52a53abd6"
+			"c1c6df6a-1ed8-4515-bc1a-dcffa03f488b" "c3bc85e0-dc50-4040-a5f1-c83b441e8938"
+			"cd86d2da-8e9e-4b56-ae05-9ea02cded8df" "ce888a0e-0383-4c3f-944e-654202cbfb2b"
+		)
+	)
+	(group ""
 		(lib_id "Project:nor")
 		(members "0d514b4d-1ab6-4588-be68-97976a6e7973" "18b71015-6191-4796-a85b-d019bae202d6"
@@
 		)
 	)
+	(group ""
+		(lib_id "Project:diode-inverter")
+		(members "1105647f-f572-4295-9bd0-9f476ea3ec47" "211d76ff-0d76-4039-aa7d-7c9b1d5ea664"
+			"2899eca2-bfbe-466c-9714-812bd2222891" "3d916724-9f70-42a7-9075-9114018b8b2d"
+			"3ff3a0c6-e8e6-4941-9ac5-db65400cfb0f" "48201187-eed7-4dd7-b717-cb91cf827791"
+			"49690052-3de2-4b20-b9d6-b80e9678c838" "572a56fa-1131-464e-97be-b6a688e8f669"
+			"721f7409-730a-47ba-b8cf-343a5627d982" "7488cd99-13ca-4d06-8c17-d2bda5402347"
+			"7d772f4b-c0e6-4076-944c-d523f6c2b415" "816c10b8-90b9-4921-9846-71f87061369a"
+			"89e40c5c-8af1-4845-94ee-4a915422ab6c" "9275c77c-bdef-4335-8d3e-ee9a4a8836fb"
+			"c6a6ddf9-752f-4add-9cc6-e7e65313c494" "ce39b239-33ed-4516-a320-0539fcbfb773"
+			"e72b459e-22d2-433a-a339-737be7eada27" "e8320575-5dfb-429c-b876-4393b9a24f70"
+			"ef7a4fc0-adda-4dfd-9ad3-0178d904a067" "f9c312b4-9ffc-4454-af31-3f840d2e7c1d"
+			"fdebbbb4-fed5-4289-8fab-588b2b26da8d"
+		)
+	)

Commit message: Start the Phase Control board.
Parts:
- Q28, Q29, Q30, Q31, Q32, Q33, Q34, Q35, Q36, Q37, Q38, Q39, Q74, Q75, Q76, Q77: symbol Transistor_BJT:Q_PNP_EBC -> Transistor_BJT:Q_PNP_BEC
Connections:
- net GND: now also Q28.2 (E), Q29.2 (E), Q30.2 (E), Q31.2 (E), Q32.2 (E), Q33.2 (E), Q34.2 (E), Q35.2 (E), Q36.2 (E), Q37.2 (E), Q38.2 (E), Q39.2 (E), Q74.2 (E), Q75.2 (E), Q76.2 (E); no longer Q28.1 (E), Q29.1 (E), Q30.1 (E), Q31.1 (E), Q32.1 (E), Q33.1 (E), Q34.1 (E), Q35.1 (E), Q36.1 (E), Q37.1 (E), Q38.1 (E), Q39.1 (E), Q74.1 (E), Q75.1 (E), Q76.1 (E)
- net W: now also Q77.2 (E); no longer Q77.1 (E)
- net at C21.1, R347.2, R380.1: now also Q76.1 (B); no longer Q76.2 (B)
- net at R154.2, R162.2, R163.2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: now also Q33.1 (B); no longer Q33.2 (B)
- net at R171.2, R172.2, R216.1: now also Q35.1 (B); no longer Q35.2 (B)
- net at C20.1, R346.2, R379.1: now also Q75.1 (B); no longer Q75.2 (B)
- net at R148.2, R149.2, R202.1: now also Q28.1 (B); no longer Q28.2 (B)
- net at R155.2, R156.2, R157.2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: now also Q31.1 (B); no longer Q31.2 (B)
- net at C19.1, R345.2, R376.1: now also Q74.1 (B); no longer Q74.2 (B)
- net at C21.2, CR55.2 (A), Q74.3 (C)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: now also Q77.1 (B); no longer Q77.2 (B)
- net at R151.2, R152.2, R204.1: now also Q29.1 (B); no longer Q29.2 (B)
- net at R177.2, R178.2, R179.2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: now also Q37.1 (B); no longer Q37.2 (B)
- net at R161.2, R167.2, R168.2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: now also Q34.1 (B); no longer Q34.2 (B)
- net at R181.2, R224.1: now also Q39.1 (B); no longer Q39.2 (B)
- net at R150.2, R153.2, R206.1: now also Q30.1 (B); no longer Q30.2 (B)
- net at R173.2, R176.2, R180.2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: now also Q38.1 (B); no longer Q38.2 (B)
- net at R174.2, R175.2, R218.1: now also Q36.1 (B); no longer Q36.2 (B)
- net at R159.2, R160.2, R210.1: now also Q32.1 (B); no longer Q32.2 (B)
Changed lines of the file:
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@@
 	)
 	(symbol
-		(lib_id "Transistor_BJT:Q_PNP_EBC")
+		(lib_id "Transistor_BJT:Q_PNP_BEC")
 		(at 217.17 35.56 0)
 		(unit 1)
@@
 			)
 		)
-		(property "Description" "Germanium PNP Transistor"
+		(property "Description" "PNP BJT"
 			(at 217.17 35.56 0)
 			(hide yes)
@@
 			)
 		)
-		(property "Sim.Pins" "1=E 2=B 3=C"
+		(property "Sim.Pins" "1=B 2=E 3=C"
 			(at 217.17 35.56 0)
 			(hide yes)
@@
 	)
 	(symbol
-		(lib_id "Transistor_BJT:Q_PNP_EBC")
+		(lib_id "Transistor_BJT:Q_PNP_BEC")
 		(at 58.42 73.66 0)
 		(unit 1)
@@
 			)
 		)
-		(property "Description" "Germanium PNP Transistor"
+		(property "Description" "PNP BJT"
 			(at 58.42 73.66 0)
 			(hide yes)
@@
 			)
 		)
-		(property "Sim.Pins" "1=E 2=B 3=C"
+		(property "Sim.Pins" "1=B 2=E 3=C"
 			(at 58.42 73.66 0)
 			(hide yes)
@@
 	)
 	(symbol
-		(lib_id "Transistor_BJT:Q_PNP_EBC")
+		(lib_id "Transistor_BJT:Q_PNP_BEC")
 		(at 53.34 186.69 0)
 		(unit 1)
@@
 			)
 		)
-		(property "Description" "Germanium PNP Transistor"
+		(property "Description" "PNP BJT"
 			(at 53.34 186.69 0)
 			(hide yes)
@@
 			)
 		)
-		(property "Sim.Pins" "1=E 2=B 3=C"
+		(property "Sim.Pins" "1=B 2=E 3=C"
 			(at 53.34 186.69 0)
 			(hide yes)
@@
 	)
 	(symbol
-		(lib_id "Transistor_BJT:Q_PNP_EBC")
+		(lib_id "Transistor_BJT:Q_PNP_BEC")
 		(at 208.28 157.48 0)
 		(unit 1)
@@
 			)
 		)
-		(property "Description" "Germanium PNP Transistor"
+		(property "Description" "PNP BJT"
 			(at 208.28 157.48 0)
 			(hide yes)
@@
 			)
 		)
-		(property "Sim.Pins" "1=E 2=B 3=C"
+		(property "Sim.Pins" "1=B 2=E 3=C"
 			(at 208.28 157.48 0)
 			(hide yes)
@@
 	)
 	(symbol
-		(lib_id "Transistor_BJT:Q_PNP_EBC")
+		(lib_id "Transistor_BJT:Q_PNP_BEC")
 		(at 217.17 67.31 0)
 		(unit 1)
@@
 			)
 		)
-		(property "Description" "Germanium PNP Transistor"
+		(property "Description" "PNP BJT"
 			(at 217.17 67.31 0)
 			(hide yes)
@@
 			)
 		)
-		(property "Sim.Pins" "1=E 2=B 3=C"
+		(property "Sim.Pins" "1=B 2=E 3=C"
 			(at 217.17 67.31 0)
 			(hide yes)
@@
 	)
 	(symbol
-		(lib_id "Transistor_BJT:Q_PNP_EBC")
+		(lib_id "Transistor_BJT:Q_PNP_BEC")
 		(at 130.81 118.11 0)
 		(unit 1)
@@
 			)
 		)
-		(property "Description" "Germanium PNP Transistor"
+		(property "Description" "PNP BJT"
 			(at 130.81 118.11 0)
 			(hide yes)
@@
 			)
 		)
-		(property "Sim.Pins" "1=E 2=B 3=C"
+		(property "Sim.Pins" "1=B 2=E 3=C"
 			(at 130.81 118.11 0)
 			(hide yes)
@@
 	)
 	(symbol
-		(lib_id "Transistor_BJT:Q_PNP_EBC")
+		(lib_id "Transistor_BJT:Q_PNP_BEC")
 		(at 99.06 124.46 0)
 		(unit 1)
@@
 			)
 		)
-		(property "Description" "Germanium PNP Transistor"
+		(property "Description" "PNP BJT"
 			(at 99.06 124.46 0)
 			(hide yes)
@@
 			)
 		)
-		(property "Sim.Pins" "1=E 2=B 3=C"
+		(property "Sim.Pins" "1=B 2=E 3=C"
 			(at 99.06 124.46 0)
 			(hide yes)
@@
 	)
 	(symbol
-		(lib_id "Transistor_BJT:Q_PNP_EBC")
+		(lib_id "Transistor_BJT:Q_PNP_BEC")
 		(at 97.79 36.83 0)
 		(unit 1)
@@
 			)
 		)
-		(property "Description" "Germanium PNP Transistor"
+		(property "Description" "PNP BJT"
 			(at 97.79 36.83 0)
 			(hide yes)
@@
 			)
 		)
-		(property "Sim.Pins" "1=E 2=B 3=C"
+		(property "Sim.Pins" "1=B 2=E 3=C"
 			(at 97.79 36.83 0)
 			(hide yes)
@@
 	)
 	(symbol
-		(lib_id "Transistor_BJT:Q_PNP_EBC")
+		(lib_id "Transistor_BJT:Q_PNP_BEC")
 		(at 53.34 152.4 0)
 		(unit 1)
@@
 			)
 		)
-		(property "Description" "Germanium PNP Transistor"
+		(property "Description" "PNP BJT"
 			(at 53.34 152.4 0)
 			(hide yes)
@@
 			)
 		)
-		(property "Sim.Pins" "1=E 2=B 3=C"
+		(property "Sim.Pins" "1=B 2=E 3=C"
 			(at 53.34 152.4 0)
 			(hide yes)
@@
 	)
 	(symbol
-		(lib_id "Transistor_BJT:Q_PNP_EBC")
+		(lib_id "Transistor_BJT:Q_PNP_BEC")
 		(at 243.84 151.13 0)
 		(unit 1)
@@
 			)
 		)
-		(property "Description" "Germanium PNP Transistor"
+		(property "Description" "PNP BJT"
 			(at 243.84 151.13 0)
 			(hide yes)
@@
 			)
 		)
-		(property "Sim.Pins" "1=E 2=B 3=C"
+		(property "Sim.Pins" "1=B 2=E 3=C"
 			(at 243.84 151.13 0)
 			(hide yes)
@@
 	)
 	(symbol
-		(lib_id "Transistor_BJT:Q_PNP_EBC")
+		(lib_id "Transistor_BJT:Q_PNP_BEC")
 		(at 53.34 118.11 0)
 		(unit 1)
@@
 			)
 		)
-		(property "Description" "Germanium PNP Transistor"
+		(property "Description" "PNP BJT"
 			(at 53.34 118.11 0)
 			(hide yes)
@@
 			)
 		)
-		(property "Sim.Pins" "1=E 2=B 3=C"
+		(property "Sim.Pins" "1=B 2=E 3=C"
 			(at 53.34 118.11 0)
 			(hide yes)
@@
 	)
 	(symbol
-		(lib_id "Transistor_BJT:Q_PNP_EBC")
+		(lib_id "Transistor_BJT:Q_PNP_BEC")
 		(at 115.57 74.93 0)
 		(unit 1)
@@
 			)
 		)
-		(property "Description" "Germanium PNP Transistor"
+		(property "Description" "PNP BJT"
 			(at 115.57 74.93 0)
 			(hide yes)
@@
 			)
 		)
-		(property "Sim.Pins" "1=E 2=B 3=C"
+		(property "Sim.Pins" "1=B 2=E 3=C"
 			(at 115.57 74.93 0)
 			(hide yes)
@@
 	)
 	(symbol
-		(lib_id "Transistor_BJT:Q_PNP_EBC")
+		(lib_id "Transistor_BJT:Q_PNP_BEC")
 		(at 208.28 111.76 0)
 		(unit 1)
@@
 			)
 		)
-		(property "Description" "Germanium PNP Transistor"
+		(property "Description" "PNP BJT"
 			(at 208.28 111.76 0)
 			(hide yes)
@@
 			)
 		)
-		(property "Sim.Pins" "1=E 2=B 3=C"
+		(property "Sim.Pins" "1=B 2=E 3=C"
 			(at 208.28 111.76 0)
 			(hide yes)
@@
 	)
 	(symbol
-		(lib_id "Transistor_BJT:Q_PNP_EBC")
+		(lib_id "Transistor_BJT:Q_PNP_BEC")
 		(at 243.84 116.84 0)
 		(unit 1)
@@
 			)
 		)
-		(property "Description" "Germanium PNP Transistor"
+		(property "Description" "PNP BJT"
 			(at 243.84 116.84 0)
 			(hide yes)
@@
 			)
 		)
-		(property "Sim.Pins" "1=E 2=B 3=C"
+		(property "Sim.Pins" "1=B 2=E 3=C"
 			(at 243.84 116.84 0)
 			(hide yes)
@@
 	)
 	(symbol
-		(lib_id "Transistor_BJT:Q_PNP_EBC")
+		(lib_id "Transistor_BJT:Q_PNP_BEC")
 		(at 163.83 66.04 0)
 		(unit 1)
@@
 			)
 		)
-		(property "Description" "Germanium PNP Transistor"
+		(property "Description" "PNP BJT"
 			(at 163.83 66.04 0)
 			(hide yes)
@@
 			)
 		)
-		(property "Sim.Pins" "1=E 2=B 3=C"
+		(property "Sim.Pins" "1=B 2=E 3=C"
 			(at 163.83 66.04 0)
 			(hide yes)
@@
 	)
 	(symbol
-		(lib_id "Transistor_BJT:Q_PNP_EBC")
+		(lib_id "Transistor_BJT:Q_PNP_BEC")
 		(at 58.42 38.1 0)
 		(unit 1)
@@
 			)
 		)
-		(property "Description" "Germanium PNP Transistor"
+		(property "Description" "PNP BJT"
 			(at 58.42 38.1 0)
 			(hide yes)
@@
 			)
 		)
-		(property "Sim.Pins" "1=E 2=B 3=C"
+		(property "Sim.Pins" "1=B 2=E 3=C"
 			(at 58.42 38.1 0)
 			(hide yes)

Commit message: Add script to export production files.
Parts:
- C19, C20, C21: BOM Value (none) -> 120pF
- C900: BOM Value (none) -> 680pF
- CR43, CR44, CR45, CR46, CR47, CR48, CR49, CR50, CR51, CR52, CR53, CR54, CR55, CR93: value 1N5819WS -> 1N4148WS; BOM Value (none) -> 1N4148WS; LCSC (none) -> C2128
- Q28, Q29, Q30, Q31, Q32, Q33, Q34, Q35, Q36, Q37, Q38, Q39, Q74, Q75, Q76, Q77: BOM Value (none) -> MMBT5401; LCSC (none) -> C8326
- R148, R149, R150, R151, R152, R153, R154, R155, R156, R157, R158, R159, R160, R161, R162, R163, R164, R165, R166, R167, R168, R169, R170, R171, R172, R173, R174, R175, R176, R177, R178, R179, R180, R181, R386, R900: BOM Value (none) -> 15kΩ
- R202, R204, R206, R208, R210, R212, R214, R216, R218, R220, R222, R224: BOM Value (none) -> 56kΩ
- R203, R205, R207, R209, R211, R213, R215, R217, R219, R221, R223, R225: BOM Value (none) -> 2kΩ 500mW
- R345, R346, R347: BOM Value (none) -> 6.8kΩ
- R375, R378: BOM Value (none) -> 10kΩ 500mW
- R376, R379, R380: BOM Value (none) -> 33kΩ
- R377, R381: BOM Value (none) -> 800Ω 2W
- R382: BOM Value (none) -> 300Ω 3W

Commit message: Rough layout for Phase Control.
Connections:
- net rl renamed r1
- net ~{rl} renamed ~{r1}
Changed lines of the file:
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@@
 		)
 	)
-	(global_label "~{rl}"
+	(global_label "~{r1}"
 		(shape output)
 		(at 140.97 111.76 0)
@@
 		)
 	)
-	(global_label "rl"
+	(global_label "r1"
 		(shape output)
 		(at 140.97 135.89 0)
