File: boards/project.kicad_blocks/flip-flop.kicad_block/flip-flop.kicad_sch (KiCad schematic)
At the start: 12 parts, among them Q10 MMBT5401, Q11 MMBT5401

Commit message: Rough layout for Phase Control.
Parts:
- removed Q10, Q11: MMBT5401, Package_TO_SOT_SMD:SOT-23, symbol Transistor_BJT:Q_PNP_BEC
- removed R19, R20: 33k, Resistor_SMD:R_0402_1005Metric, symbol Device:R_US
- removed R85, R86: 2k4 ¼W, Resistor_SMD:R_0603_1608Metric, symbol Device:R_US
- added Q1, Q2: MMBT5401, Package_TO_SOT_SMD:SOT-23, symbol Transistor_BJT:Q_PNP_BEC
- added R1, R4: 2k4 ¼W, Resistor_SMD:R_0603_1608Metric, symbol Device:R_US
- added R2, R3: 33k, Resistor_SMD:R_0402_1005Metric, symbol Device:R_US
- C1, C4: BOM Value (none) -> 120pF
- C2, C3: BOM Value (none) -> 680pF
- CR1, CR2: value 1N5819WS -> 1N4148WS; BOM Value (none) -> 1N4148WS; LCSC (none) -> C2128
Connections:
- net +15V: now also R2.2, R3.2
- net GND: now also Q1.2 (E), Q2.2 (E)
- net at C1.1, CR1.1 (K): now also Q2.1 (B), R1.2, R2.1
- net at C4.1: now also CR2.1 (K), Q1.1 (B), R3.1, R4.1
- net at C1.2: now also Q1.3 (C), R1.1
- net at C4.2: now also Q2.3 (C), R4.2; no longer CR2.1 (K)
Other:
- note added: "A"
